Commit message: Automatic build. Travis build:229
icub-model-generator commit:7cc507ecede34ae987c9dec384d2d7910e8c5296

urdf_parser_py commit:31474b9baaf7c3845b40e5a9aa87d5900a2282c3

simmechanics-to-urdf commit:1bd48b2d02b1d155a782f35d96865753c2e49706

yarp commit:131bb8c022c3bcec2e00c7d6c93cf14951383a56

icub-main commit:c3698cb14ee3c0228fbebecd4f49756e630f75c2

idyntree commit:96f5c366ba02d5a62fd57c1f3fc2ddd6f2f9eb28

File: iCub/robots/iCubGazeboV2_5_plus/model.urdf (robot description, URDF)
Before this commit: robot iCub, 140 links, 139 joints
Joints:
- joint l_hip_yaw: origin xyz=0 0 0.0144 rpy=-3.14159265359 0 -1.57079632679 -> xyz=0 0 0.0144 rpy=-3.14159265359 0 0
- joint l_leg_ft_sensor: origin xyz=-0.0008575 0 -0.0743 rpy=-3.14159265359 0 -1.57079632679 -> xyz=-0.0008575 0 -0.0743 rpy=3.14159265359 0 0

File: iCub/robots/iCubGenova04_plus/model.urdf (robot description, URDF)
Before this commit: robot iCub, 140 links, 139 joints
Joints:
- joint l_hip_yaw: origin xyz=0 0 0.0144 rpy=-3.14159265359 0 -1.57079632679 -> xyz=0 0 0.0144 rpy=-3.14159265359 0 0
- joint l_leg_ft_sensor: origin xyz=-0.0008575 0 -0.0743 rpy=-3.14159265359 0 -1.57079632679 -> xyz=-0.0008575 0 -0.0743 rpy=3.14159265359 0 0
