Commit message: Updated models after icub-model-generator PR 49

File: iCub/robots/iCubGenova02/model.urdf (robot description, URDF)
Before this commit: robot ICUB_2-5_BB_SIM_MODEL, 163 links, 162 joints
Links:
- removed link chest_ems_acc_eb1
- removed link chest_ems_acc_eb2
- removed link chest_ems_acc_eb3
- removed link chest_ems_acc_eb4
- removed link chest_ems_gyro_eb1
- removed link chest_ems_gyro_eb2
- removed link chest_ems_gyro_eb3
- removed link chest_ems_gyro_eb4
- removed link chest_mtb_acc_0b10
- removed link chest_mtb_acc_0b7
- removed link chest_mtb_acc_0b8
- removed link chest_mtb_acc_0b9
- removed link l_foot_mtb_acc_10b12
- removed link l_foot_mtb_acc_10b13
- removed link l_forearm_mtb_acc_1b7
- removed link l_forearm_mtb_acc_1b8
- removed link l_forearm_mtb_acc_1b9
- removed link l_lower_leg_ems_acc_eb7
- removed link l_lower_leg_ems_gyro_eb7
- removed link l_lower_leg_mtb_acc_10b10
- removed link l_lower_leg_mtb_acc_10b11
- removed link l_lower_leg_mtb_acc_10b8
- removed link l_lower_leg_mtb_acc_10b9
- removed link l_upper_arm_mtb_acc_1b10
- removed link l_upper_arm_mtb_acc_1b11
- removed link l_upper_arm_mtb_acc_1b12
- removed link l_upper_arm_mtb_acc_1b13
- removed link l_upper_leg_ems_acc_eb10
- removed link l_upper_leg_ems_acc_eb6
- removed link l_upper_leg_ems_gyro_eb10
- removed link l_upper_leg_ems_gyro_eb6
- removed link l_upper_leg_mtb_acc_10b1
- removed link l_upper_leg_mtb_acc_10b2
- removed link l_upper_leg_mtb_acc_10b3
- removed link l_upper_leg_mtb_acc_10b4
- removed link l_upper_leg_mtb_acc_10b5
- removed link l_upper_leg_mtb_acc_10b6
- removed link l_upper_leg_mtb_acc_10b7
- removed link r_foot_mtb_acc_11b12
- removed link r_foot_mtb_acc_11b13
- removed link r_forearm_mtb_acc_2b7
- removed link r_forearm_mtb_acc_2b8
- removed link r_forearm_mtb_acc_2b9
- removed link r_lower_leg_ems_acc_eb9
- removed link r_lower_leg_ems_gyro_eb9
- removed link r_lower_leg_mtb_acc_11b10
- removed link r_lower_leg_mtb_acc_11b11
- removed link r_lower_leg_mtb_acc_11b8
- removed link r_lower_leg_mtb_acc_11b9
- removed link r_upper_arm_mtb_acc_2b10
- removed link r_upper_arm_mtb_acc_2b11
- removed link r_upper_arm_mtb_acc_2b12
- removed link r_upper_arm_mtb_acc_2b13
- removed link r_upper_leg_ems_acc_eb11
- removed link r_upper_leg_ems_acc_eb8
- removed link r_upper_leg_ems_gyro_eb11
- removed link r_upper_leg_ems_gyro_eb8
- removed link r_upper_leg_mtb_acc_11b1
- removed link r_upper_leg_mtb_acc_11b2
- removed link r_upper_leg_mtb_acc_11b3
- removed link r_upper_leg_mtb_acc_11b4
- removed link r_upper_leg_mtb_acc_11b5
- removed link r_upper_leg_mtb_acc_11b6
- removed link r_upper_leg_mtb_acc_11b7
- removed link root_link_ems_acc_eb5
- removed link root_link_ems_gyro_eb5
Joints:
- removed joint chest_ems_acc_eb1_fixed_joint
- removed joint chest_ems_acc_eb2_fixed_joint
- removed joint chest_ems_acc_eb3_fixed_joint
- removed joint chest_ems_acc_eb4_fixed_joint
- removed joint chest_ems_gyro_eb1_fixed_joint
- removed joint chest_ems_gyro_eb2_fixed_joint
- removed joint chest_ems_gyro_eb3_fixed_joint
- removed joint chest_ems_gyro_eb4_fixed_joint
- removed joint chest_mtb_acc_0b10_fixed_joint
- removed joint chest_mtb_acc_0b7_fixed_joint
- removed joint chest_mtb_acc_0b8_fixed_joint
- removed joint chest_mtb_acc_0b9_fixed_joint
- removed joint l_foot_mtb_acc_10b12_fixed_joint
- removed joint l_foot_mtb_acc_10b13_fixed_joint
- removed joint l_forearm_mtb_acc_1b7_fixed_joint
- removed joint l_forearm_mtb_acc_1b8_fixed_joint
- removed joint l_forearm_mtb_acc_1b9_fixed_joint
- removed joint l_lower_leg_ems_acc_eb7_fixed_joint
- removed joint l_lower_leg_ems_gyro_eb7_fixed_joint
- removed joint l_lower_leg_mtb_acc_10b10_fixed_joint
- removed joint l_lower_leg_mtb_acc_10b11_fixed_joint
- removed joint l_lower_leg_mtb_acc_10b8_fixed_joint
- removed joint l_lower_leg_mtb_acc_10b9_fixed_joint
- removed joint l_upper_arm_mtb_acc_1b10_fixed_joint
- removed joint l_upper_arm_mtb_acc_1b11_fixed_joint
- removed joint l_upper_arm_mtb_acc_1b12_fixed_joint
- removed joint l_upper_arm_mtb_acc_1b13_fixed_joint
- removed joint l_upper_leg_ems_acc_eb10_fixed_joint
- removed joint l_upper_leg_ems_acc_eb6_fixed_joint
- removed joint l_upper_leg_ems_gyro_eb10_fixed_joint
- removed joint l_upper_leg_ems_gyro_eb6_fixed_joint
- removed joint l_upper_leg_mtb_acc_10b1_fixed_joint
- removed joint l_upper_leg_mtb_acc_10b2_fixed_joint
- removed joint l_upper_leg_mtb_acc_10b3_fixed_joint
- removed joint l_upper_leg_mtb_acc_10b4_fixed_joint
- removed joint l_upper_leg_mtb_acc_10b5_fixed_joint
- removed joint l_upper_leg_mtb_acc_10b6_fixed_joint
- removed joint l_upper_leg_mtb_acc_10b7_fixed_joint
- removed joint r_foot_mtb_acc_11b12_fixed_joint
- removed joint r_foot_mtb_acc_11b13_fixed_joint
- removed joint r_forearm_mtb_acc_2b7_fixed_joint
- removed joint r_forearm_mtb_acc_2b8_fixed_joint
- removed joint r_forearm_mtb_acc_2b9_fixed_joint
- removed joint r_lower_leg_ems_acc_eb9_fixed_joint
- removed joint r_lower_leg_ems_gyro_eb9_fixed_joint
- removed joint r_lower_leg_mtb_acc_11b10_fixed_joint
- removed joint r_lower_leg_mtb_acc_11b11_fixed_joint
- removed joint r_lower_leg_mtb_acc_11b8_fixed_joint
- removed joint r_lower_leg_mtb_acc_11b9_fixed_joint
- removed joint r_upper_arm_mtb_acc_2b10_fixed_joint
- removed joint r_upper_arm_mtb_acc_2b11_fixed_joint
- removed joint r_upper_arm_mtb_acc_2b12_fixed_joint
- removed joint r_upper_arm_mtb_acc_2b13_fixed_joint
- removed joint r_upper_leg_ems_acc_eb11_fixed_joint
- removed joint r_upper_leg_ems_acc_eb8_fixed_joint
- removed joint r_upper_leg_ems_gyro_eb11_fixed_joint
- removed joint r_upper_leg_ems_gyro_eb8_fixed_joint
- removed joint r_upper_leg_mtb_acc_11b1_fixed_joint
- removed joint r_upper_leg_mtb_acc_11b2_fixed_joint
- removed joint r_upper_leg_mtb_acc_11b3_fixed_joint
- removed joint r_upper_leg_mtb_acc_11b4_fixed_joint
- removed joint r_upper_leg_mtb_acc_11b5_fixed_joint
- removed joint r_upper_leg_mtb_acc_11b6_fixed_joint
- removed joint r_upper_leg_mtb_acc_11b7_fixed_joint
- removed joint root_link_ems_acc_eb5_fixed_joint
- removed joint root_link_ems_gyro_eb5_fixed_joint

Commit message: Automatic build. Travis build:234
icub-model-generator commit:bada6e53f0c874d80812a0b3cd146145d1ea85c9

urdf_parser_py commit:31474b9baaf7c3845b40e5a9aa87d5900a2282c3

simmechanics-to-urdf commit:1bd48b2d02b1d155a782f35d96865753c2e49706

yarp commit:2aa5e018e8ed8751fbca8b5ce9f97e5b97c05876

icub-main commit:4fc21383a376b807fee1c16660929a740f95b32b

idyntree commit:6f98701123e66b8fbb274e8e0ae657d7688f7501

File: iCub/robots/iCubGenova02/model.urdf (robot description, URDF)
Before this commit: robot iCub, 189 links, 188 joints
Links:
- removed link l_sole_skin_0
- removed link l_sole_skin_1
- removed link l_sole_skin_10
- removed link l_sole_skin_11
- removed link l_sole_skin_12
- removed link l_sole_skin_13
- removed link l_sole_skin_14
- removed link l_sole_skin_15
- removed link l_sole_skin_17
- removed link l_sole_skin_18
- removed link l_sole_skin_19
- removed link l_sole_skin_2
- removed link l_sole_skin_20
- removed link l_sole_skin_21
- removed link l_sole_skin_22
- removed link l_sole_skin_24
- removed link l_sole_skin_25
- removed link l_sole_skin_26
- removed link l_sole_skin_27
- removed link l_sole_skin_28
- removed link l_sole_skin_29
- removed link l_sole_skin_3
- removed link l_sole_skin_4
- removed link l_sole_skin_8
- removed link l_sole_skin_9
- removed link r_sole_skin_0
- removed link r_sole_skin_1
- removed link r_sole_skin_10
- removed link r_sole_skin_11
- removed link r_sole_skin_12
- removed link r_sole_skin_13
- removed link r_sole_skin_14
- removed link r_sole_skin_15
- removed link r_sole_skin_17
- removed link r_sole_skin_18
- removed link r_sole_skin_19
- removed link r_sole_skin_2
- removed link r_sole_skin_20
- removed link r_sole_skin_21
- removed link r_sole_skin_22
- removed link r_sole_skin_24
- removed link r_sole_skin_25
- removed link r_sole_skin_26
- removed link r_sole_skin_27
- removed link r_sole_skin_28
- removed link r_sole_skin_29
- removed link r_sole_skin_3
- removed link r_sole_skin_4
- removed link r_sole_skin_8
- removed link r_sole_skin_9
- added link root_link_imu_frame
- link chest: geometry collision mesh filename=package://iCub/meshes/simmechanics/2-5_plus/sim_sea_2-5_che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 scale=0.001 0.001 0.001; visual mesh filename=package://iCub/meshes/simmechanics/2-5_plus/sim_sea_2-5_che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 scale=0.001 0.001 0.001
- link head: geometry collision mesh filename=package://iCub/meshes/simmechanics/2-5_plus/sim_sea_2-5_hea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 scale=0.001 0.001 0.001; visual mesh filename=package://iCub/meshes/simmechanics/2-5_plus/sim_sea_2-5_hea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 scale=0.001 0.001 0.001
- link l_ankle_1: geometry collision mesh filename=package://iCub/meshes/simmechanics/2-5_plus/sim_sea_2-5_l_a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 scale=0.001 0.001 0.001; visual mesh filename=package://iCub/meshes/simmechanics/2-5_plus/sim_sea_2-5_l_a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 scale=0.001 0.001 0.001
- link l_ankle_2: mass 0.267485 -> 0.265337; geometry collision mesh filename=package://iCub/meshes/simmechanics/2-5_plus/sim_sea_2-5_l_f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 scale=0.001 0.001 0.001; visual mesh filename=package://iCub/meshes/simmechanics/2-5_plus/sim_sea_2-5_l_f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 scale=0.001 0.001 0.001
- link l_elbow_1: geometry collision mesh filename=package://iCub/meshes/simmechanics/2-5_plus/sim_sea_2-5_l_e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 scale=0.001 0.001 0.001; visual mesh filename=package://iCub/meshes/simmechanics/2-5_plus/sim_sea_2-5_l_e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 scale=0.001 0.001 0.001
- link l_foot: mass 0.382968 -> 0.357881; geometry collision mesh filename=package://iCub/meshes/simmechanics/2-5_plus/sim_sea_2-5_l_s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 scale=0.001 0.001 0.001; visual mesh filename=package://iCub/meshes/simmechanics/2-5_plus/sim_sea_2-5_l_s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 scale=0.001 0.001 0.001
- link l_forearm: geometry collision mesh filename=package://iCub/meshes/simmechanics/2-5_plus/sim_sea_2-5_l_f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 scale=0.001 0.001 0.001; visual mesh filename=package://iCub/meshes/simmechanics/2-5_plus/sim_sea_2-5_l_f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 scale=0.001 0.001 0.001
- link l_hand: geometry collision mesh filename=package://iCub/meshes/simmechanics/2-5_plus/sim_sea_2-5_l_h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 scale=0.001 0.001 0.001; visual mesh filename=package://iCub/meshes/simmechanics/2-5_plus/sim_sea_2-5_l_h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 scale=0.001 0.001 0.001
- link l_hip_1: geometry collision mesh filename=package://iCub/meshes/simmechanics/2-5_plus/sim_sea_2-5_l_h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 scale=0.001 0.001 0.001; visual mesh filename=package://iCub/meshes/simmechanics/2-5_plus/sim_sea_2-5_l_h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 scale=0.001 0.001 0.001
- link l_hip_2: geometry collision mesh filename=package://iCub/meshes/simmechanics/2-5_plus/sim_sea_2-5_l_h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 scale=0.001 0.001 0.001; visual mesh filename=package://iCub/meshes/simmechanics/2-5_plus/sim_sea_2-5_l_h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 scale=0.001 0.001 0.001
- link l_hip_3: geometry collision mesh filename=package://iCub/meshes/simmechanics/2-5_plus/sim_sea_2-5_l_u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 scale=0.001 0.001 0.001; visual mesh filename=package://iCub/meshes/simmechanics/2-5_plus/sim_sea_2-5_l_u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 scale=0.001 0.001 0.001
- link l_lower_leg: geometry collision mesh filename=package://iCub/meshes/simmechanics/2-5_plus/sim_sea_2-5_l_s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 scale=0.001 0.001 0.001; visual mesh filename=package://iCub/meshes/simmechanics/2-5_plus/sim_sea_2-5_l_s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 scale=0.001 0.001 0.001
- link l_shoulder_1: geometry collision mesh filename=package://iCub/meshes/simmechanics/2-5_plus/sim_sea_2-5_l_s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 scale=0.001 0.001 0.001; visual mesh filename=package://iCub/meshes/simmechanics/2-5_plus/sim_sea_2-5_l_s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 scale=0.001 0.001 0.001
- link l_shoulder_2: geometry collision mesh filename=package://iCub/meshes/simmechanics/2-5_plus/sim_sea_2-5_l_s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 scale=0.001 0.001 0.001; visual mesh filename=package://iCub/meshes/simmechanics/2-5_plus/sim_sea_2-5_l_s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 scale=0.001 0.001 0.001
- link l_shoulder_3: geometry collision mesh filename=package://iCub/meshes/simmechanics/2-5_plus/sim_sea_2-5_l_u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 scale=0.001 0.001 0.001; visual mesh filename=package://iCub/meshes/simmechanics/2-5_plus/sim_sea_2-5_l_u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 scale=0.001 0.001 0.001
- link l_upper_arm: geometry collision mesh filename=package://iCub/meshes/simmechanics/2-5_plus/sim_sea_2-5_l_e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 scale=0.001 0.001 0.001; visual mesh filename=package://iCub/meshes/simmechanics/2-5_plus/sim_sea_2-5_l_e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 scale=0.001 0.001 0.001
- link l_upper_leg: geometry collision mesh filename=package://iCub/meshes/simmechanics/2-5_plus/sim_sea_2-5_l_t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 scale=0.001 0.001 0.001; visual mesh filename=package://iCub/meshes/simmechanics/2-5_plus/sim_sea_2-5_l_t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 scale=0.001 0.001 0.001
- link l_wrist_1: geometry collision mesh filename=package://iCub/meshes/simmechanics/2-5_plus/sim_sea_2-5_l_w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 scale=0.001 0.001 0.001; visual mesh filename=package://iCub/meshes/simmechanics/2-5_plus/sim_sea_2-5_l_w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 scale=0.001 0.001 0.001
- link neck_1: geometry collision mesh filename=package://iCub/meshes/simmechanics/2-5_plus/sim_sea_2-5_nec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 scale=0.001 0.001 0.001; visual mesh filename=package://iCub/meshes/simmechanics/2-5_plus/sim_sea_2-5_nec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 scale=0.001 0.001 0.001
- link neck_2: geometry collision mesh filename=package://iCub/meshes/simmechanics/2-5_plus/sim_sea_2-5_nec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 scale=0.001 0.001 0.001; visual mesh filename=package://iCub/meshes/simmechanics/2-5_plus/sim_sea_2-5_nec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 scale=0.001 0.001 0.001
- link r_ankle_1: geometry collision mesh filename=package://iCub/meshes/simmechanics/2-5_plus/sim_sea_2-5_r_a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 scale=0.001 0.001 0.001; visual mesh filename=package://iCub/meshes/simmechanics/2-5_plus/sim_sea_2-5_r_a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 scale=0.001 0.001 0.001
- link r_ankle_2: mass 0.267485 -> 0.265337; geometry collision mesh filename=package://iCub/meshes/simmechanics/2-5_plus/sim_sea_2-5_r_f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 scale=0.001 0.001 0.001; visual mesh filename=package://iCub/meshes/simmechanics/2-5_plus/sim_sea_2-5_r_f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 scale=0.001 0.001 0.001
- link r_elbow_1: geometry collision mesh filename=package://iCub/meshes/simmechanics/2-5_plus/sim_sea_2-5_r_e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 scale=0.001 0.001 0.001; visual mesh filename=package://iCub/meshes/simmechanics/2-5_plus/sim_sea_2-5_r_e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 scale=0.001 0.001 0.001
- link r_foot: mass 0.382866 -> 0.357881; geometry collision mesh filename=package://iCub/meshes/simmechanics/2-5_plus/sim_sea_2-5_r_s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 scale=0.001 0.001 0.001; visual mesh filename=package://iCub/meshes/simmechanics/2-5_plus/sim_sea_2-5_r_s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 scale=0.001 0.001 0.001
- link r_forearm: geometry collision mesh filename=package://iCub/meshes/simmechanics/2-5_plus/sim_sea_2-5_r_f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 scale=0.001 0.001 0.001; visual mesh filename=package://iCub/meshes/simmechanics/2-5_plus/sim_sea_2-5_r_f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 scale=0.001 0.001 0.001
- link r_hand: geometry collision mesh filename=package://iCub/meshes/simmechanics/2-5_plus/sim_sea_2-5_r_h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 scale=0.001 0.001 0.001; visual mesh filename=package://iCub/meshes/simmechanics/2-5_plus/sim_sea_2-5_r_h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 scale=0.001 0.001 0.001
- link r_hip_1: geometry collision mesh filename=package://iCub/meshes/simmechanics/2-5_plus/sim_sea_2-5_r_h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 scale=0.001 0.001 0.001; visual mesh filename=package://iCub/meshes/simmechanics/2-5_plus/sim_sea_2-5_r_h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 scale=0.001 0.001 0.001
- link r_hip_2: geometry collision mesh filename=package://iCub/meshes/simmechanics/2-5_plus/sim_sea_2-5_r_h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 scale=0.001 0.001 0.001; visual mesh filename=package://iCub/meshes/simmechanics/2-5_plus/sim_sea_2-5_r_h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 scale=0.001 0.001 0.001
- link r_hip_3: geometry collision mesh filename=package://iCub/meshes/simmechanics/2-5_plus/sim_sea_2-5_r_u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 scale=0.001 0.001 0.001; visual mesh filename=package://iCub/meshes/simmechanics/2-5_plus/sim_sea_2-5_r_u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 scale=0.001 0.001 0.001
- link r_lower_leg: geometry collision mesh filename=package://iCub/meshes/simmechanics/2-5_plus/sim_sea_2-5_r_s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 scale=0.001 0.001 0.001; visual mesh filename=package://iCub/meshes/simmechanics/2-5_plus/sim_sea_2-5_r_s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 scale=0.001 0.001 0.001
- link r_shoulder_1: geometry collision mesh filename=package://iCub/meshes/simmechanics/2-5_plus/sim_sea_2-5_r_s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 scale=0.001 0.001 0.001; visual mesh filename=package://iCub/meshes/simmechanics/2-5_plus/sim_sea_2-5_r_s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 scale=0.001 0.001 0.001
- link r_shoulder_2: geometry collision mesh filename=package://iCub/meshes/simmechanics/2-5_plus/sim_sea_2-5_r_s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 scale=0.001 0.001 0.001; visual mesh filename=package://iCub/meshes/simmechanics/2-5_plus/sim_sea_2-5_r_s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 scale=0.001 0.001 0.001
- link r_shoulder_3: geometry collision mesh filename=package://iCub/meshes/simmechanics/2-5_plus/sim_sea_2-5_r_u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 scale=0.001 0.001 0.001; visual mesh filename=package://iCub/meshes/simmechanics/2-5_plus/sim_sea_2-5_r_u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 scale=0.001 0.001 0.001
- link r_upper_arm: geometry collision mesh filename=package://iCub/meshes/simmechanics/2-5_plus/sim_sea_2-5_r_e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 scale=0.001 0.001 0.001; visual mesh filename=package://iCub/meshes/simmechanics/2-5_plus/sim_sea_2-5_r_e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 scale=0.001 0.001 0.001
- link r_upper_leg: geometry collision mesh filename=package://iCub/meshes/simmechanics/2-5_plus/sim_sea_2-5_r_t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 scale=0.001 0.001 0.001; visual mesh filename=package://iCub/meshes/simmechanics/2-5_plus/sim_sea_2-5_r_t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 scale=0.001 0.001 0.001
- link r_wrist_1: geometry collision mesh filename=package://iCub/meshes/simmechanics/2-5_plus/sim_sea_2-5_r_w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 scale=0.001 0.001 0.001; visual mesh filename=package://iCub/meshes/simmechanics/2-5_plus/sim_sea_2-5_r_w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 scale=0.001 0.001 0.001
- link root_link: mass 5.09143 -> 5.12739; geometry collision mesh filename=package://iCub/meshes/simmechanics/2-5_plus/sim_sea_2-5_roo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 scale=0.001 0.001 0.001; visual mesh filename=package://iCub/meshes/simmechanics/2-5_plus/sim_sea_2-5_roo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 scale=0.001 0.001 0.001
- link torso_1: geometry collision mesh filename=package://iCub/meshes/simmechanics/2-5_plus/sim_sea_2-5_lap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 scale=0.001 0.001 0.001; visual mesh filename=package://iCub/meshes/simmechanics/2-5_plus/sim_sea_2-5_lap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 scale=0.001 0.001 0.001
- link torso_2: geometry collision mesh filename=package://iCub/meshes/simmechanics/2-5_plus/sim_sea_2-5_lap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 scale=0.001 0.001 0.001; visual mesh filename=package://iCub/meshes/simmechanics/2-5_plus/sim_sea_2-5_lap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 scale=0.001 0.001 0.001
Joints:
- removed joint l_sole_skin_0_fixed_joint
- removed joint l_sole_skin_10_fixed_joint
- removed joint l_sole_skin_11_fixed_joint
- removed joint l_sole_skin_12_fixed_joint
- removed joint l_sole_skin_13_fixed_joint
- removed joint l_sole_skin_14_fixed_joint
- removed joint l_sole_skin_15_fixed_joint
- removed joint l_sole_skin_17_fixed_joint
- removed joint l_sole_skin_18_fixed_joint
- removed joint l_sole_skin_19_fixed_joint
- removed joint l_sole_skin_1_fixed_joint
- removed joint l_sole_skin_20_fixed_joint
- removed joint l_sole_skin_21_fixed_joint
- removed joint l_sole_skin_22_fixed_joint
- removed joint l_sole_skin_24_fixed_joint
- removed joint l_sole_skin_25_fixed_joint
- removed joint l_sole_skin_26_fixed_joint
- removed joint l_sole_skin_27_fixed_joint
- removed joint l_sole_skin_28_fixed_joint
- removed joint l_sole_skin_29_fixed_joint
- removed joint l_sole_skin_2_fixed_joint
- removed joint l_sole_skin_3_fixed_joint
- removed joint l_sole_skin_4_fixed_joint
- removed joint l_sole_skin_8_fixed_joint
- removed joint l_sole_skin_9_fixed_joint
- removed joint r_sole_skin_0_fixed_joint
- removed joint r_sole_skin_10_fixed_joint
- removed joint r_sole_skin_11_fixed_joint
- removed joint r_sole_skin_12_fixed_joint
- removed joint r_sole_skin_13_fixed_joint
- removed joint r_sole_skin_14_fixed_joint
- removed joint r_sole_skin_15_fixed_joint
- removed joint r_sole_skin_17_fixed_joint
- removed joint r_sole_skin_18_fixed_joint
- removed joint r_sole_skin_19_fixed_joint
- removed joint r_sole_skin_1_fixed_joint
- removed joint r_sole_skin_20_fixed_joint
- removed joint r_sole_skin_21_fixed_joint
- removed joint r_sole_skin_22_fixed_joint
- removed joint r_sole_skin_24_fixed_joint
- removed joint r_sole_skin_25_fixed_joint
- removed joint r_sole_skin_26_fixed_joint
- removed joint r_sole_skin_27_fixed_joint
- removed joint r_sole_skin_28_fixed_joint
- removed joint r_sole_skin_29_fixed_joint
- removed joint r_sole_skin_2_fixed_joint
- removed joint r_sole_skin_3_fixed_joint
- removed joint r_sole_skin_4_fixed_joint
- removed joint r_sole_skin_8_fixed_joint
- removed joint r_sole_skin_9_fixed_joint
- added joint root_link_imu_frame_fixed_joint: type fixed, parent root_link, child root_link_imu_frame, origin xyz=0.085155 -0.011 -0.112309 rpy=-2.09439521059 0 -1.57079632679
- joint l_ankle_pitch: axis 2.22044604925e-16 1.0 0.0 -> -6.66133814775e-16 1.0 4.4408920985e-16; limit lower=-0.610865238198 upper=0.610865238198 effort=37.0 velocity=7.64 -> lower=-0.872664625997 upper=0.349065850399 effort=37.0 velocity=7.64; origin xyz=0 0 -0.2005 rpy=0 0 0 -> xyz=0 0 -0.2005 rpy=0 0.26179917948 0
- joint l_ankle_roll: axis 1.0 0.0 2.22044604925e-16 -> 1.00000015612 6.0136540192e-16 -1.19793949732e-07
- joint l_foot_ft_sensor: origin xyz=-0.0035 0 -0.0605 rpy=3.14159265359 0 0 -> xyz=-0.00349992806597 0 -0.0605003432802 rpy=-3.14159264324 0 0
- joint l_sole_fixed_joint: origin xyz=0.0035 0 0.004 rpy=-3.14159265359 0 0 -> xyz=0.0214502260596 0 0.00669127665248 rpy=-3.14159265359 0.261799192098 0
- joint r_ankle_pitch: axis 2.22044604925e-16 1.0 0.0 -> -6.66133814775e-16 1.0 4.4408920985e-16; limit lower=-0.610865238198 upper=0.610865238198 effort=37.0 velocity=7.64 -> lower=-0.872664625997 upper=0.349065850399 effort=37.0 velocity=7.64; origin xyz=0 0 -0.2005 rpy=0 0 0 -> xyz=0 0 -0.2005 rpy=0 0.26179917948 0
- joint r_ankle_roll: axis -1.0 0.0 -2.22044604925e-16 -> -1.00000015612 -6.0136540192e-16 1.19793949732e-07
- joint r_foot_ft_sensor: origin xyz=-0.0035 0 -0.0605 rpy=3.14159265359 0 0 -> xyz=-0.00349992806597 0 -0.0605003432802 rpy=3.14159265242 0 0
- joint r_sole_fixed_joint: origin xyz=0.0035 0 0.004 rpy=-3.14159265359 0 0 -> xyz=0.0214502260596 0 0.00669127665248 rpy=-3.14159265359 0.261799181028 0
- joint torso_pitch: origin xyz=0 0.0270463 0 rpy=1.57079632679 0 -1.57079632679 -> xyz=0 0.0269348 0 rpy=1.57079632679 0 -1.57079632679
- joint torso_roll: origin xyz=0.0270462998093 0.032 -0.0573446 rpy=0 0 0 -> xyz=0.0269347998093 0.032 -0.0573446 rpy=0 0 0
