Commit message: Automatic build. Travis build:505
icub-model-generator commit:bd5033f1664009c9a89d23162d1b8b8462958454

urdf_parser_py commit:31474b9baaf7c3845b40e5a9aa87d5900a2282c3

simmechanics-to-urdf commit:386e2c9c809d8d95e8e6c169cc23747de58ebae3

yarp commit:fdd9c2157c150b6e617dc8bb55515d8b66ae4640

icub-main commit:7baee55743fef19fa163f12231bc0aa65354fb0b

idyntree commit:40ba1b919b5f730faf597cc4237b492d03f45708

File: iCub/robots/iCubGazeboV2_5/model.urdf (robot description, URDF)
Before this commit: robot iCub, 189 links, 188 joints
Links:
- link l_foot: geometry collision mesh filename=package://iCub/meshes/simmechanics/sim_sea_2-5_l_sole_prt-b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 scale=0.001 0.001 0.001; visual mesh filename=package://iCub/meshes/simmechanics/sim_sea_2-5_l_sole_prt-b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 scale=0.001 0.001 0.001
- link r_foot: geometry collision mesh filename=package://iCub/meshes/simmechanics/sim_sea_2-5_r_sole_prt-b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 scale=0.001 0.001 0.001; visual mesh filename=package://iCub/meshes/simmechanics/sim_sea_2-5_r_sole_prt-b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 scale=0.001 0.001 0.001

File: iCub/robots/iCubGazeboV2_5_plus/model.urdf (robot description, URDF)
Before this commit: robot iCub, 140 links, 139 joints
Links:
- link l_foot: geometry collision mesh filename=package://iCub/meshes/simmechanics/2-5_plus/sim_sea_2-5_l_s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 scale=0.001 0.001 0.001; visual mesh filename=package://iCub/meshes/simmechanics/2-5_plus/sim_sea_2-5_l_s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 scale=0.001 0.001 0.001
- link r_foot: geometry collision mesh filename=package://iCub/meshes/simmechanics/2-5_plus/sim_sea_2-5_r_s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 scale=0.001 0.001 0.001; visual mesh filename=package://iCub/meshes/simmechanics/2-5_plus/sim_sea_2-5_r_s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 scale=0.001 0.001 0.001

File: iCub/robots/iCubGazeboV2_6/model.urdf (robot description, URDF)
Before this commit: robot iCub, 189 links, 188 joints
Links:
- link l_foot: geometry collision mesh filename=package://iCub/meshes/simmechanics/sim_sea_2-5_l_sole_prt-b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 scale=0.001 0.001 0.001; visual mesh filename=package://iCub/meshes/simmechanics/sim_sea_2-5_l_sole_prt-b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 scale=0.001 0.001 0.001
- link r_foot: geometry collision mesh filename=package://iCub/meshes/simmechanics/sim_sea_2-5_r_sole_prt-b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 scale=0.001 0.001 0.001; visual mesh filename=package://iCub/meshes/simmechanics/sim_sea_2-5_r_sole_prt-b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 scale=0.001 0.001 0.001

File: iCub/robots/iCubGazeboV3/model.urdf (robot description, URDF)
Before this commit: robot iCub, 45 links, 44 joints
Links:
- link l_foot_front: geometry collision box size=0.117 0.1 0.006; visual mesh filename=package://iCub/meshes/simmechanics/sim_icub3_l_foot_front_p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 scale=0.001 0.001 0.001
- link l_foot_rear: geometry collision box size=0.117 0.1 0.006; visual mesh filename=package://iCub/meshes/simmechanics/sim_icub3_l_foot_rear_pr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 scale=0.001 0.001 0.001
- link r_foot_front: geometry collision box size=0.117 0.1 0.006; visual mesh filename=package://iCub/meshes/simmechanics/sim_icub3_r_foot_front_p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 scale=0.001 0.001 0.001
- link r_foot_rear: geometry collision box size=0.117 0.1 0.006; visual mesh filename=package://iCub/meshes/simmechanics/sim_icub3_r_foot_rear_pr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 scale=0.001 0.001 0.001

Commit message: Automatic build. GitHub Actions build: 372103414 icub-model-generator commit:29dc0d90e75baf7027241fba0c3d0fd2ecdf141e urdf_parser_py commit:31474b9baaf7c3845b40e5a9aa87d5900a2282c3 simmechanics-to-urdf commit:386e2c9c809d8d95e8e6c169cc23747de58ebae3

File: iCub/robots/iCubGazeboV2_5/model.urdf (robot description, URDF)
Before this commit: robot iCub, 189 links, 188 joints
Links:
- link l_foot: geometry collision box size=0.16 0.072 0.001; visual mesh filename=package://iCub/meshes/simmechanics/sim_sea_2-5_l_sole_prt-b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 scale=0.001 0.001 0.001
- link r_foot: geometry collision box size=0.16 0.072 0.001; visual mesh filename=package://iCub/meshes/simmechanics/sim_sea_2-5_r_sole_prt-b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 scale=0.001 0.001 0.001

File: iCub/robots/iCubGazeboV2_5_plus/model.urdf (robot description, URDF)
Before this commit: robot iCub, 140 links, 139 joints
Links:
- link l_foot: geometry collision box size=0.16 0.072 0.001; visual mesh filename=package://iCub/meshes/simmechanics/2-5_plus/sim_sea_2-5_l_s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 scale=0.001 0.001 0.001
- link r_foot: geometry collision box size=0.16 0.072 0.001; visual mesh filename=package://iCub/meshes/simmechanics/2-5_plus/sim_sea_2-5_r_s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 scale=0.001 0.001 0.001

File: iCub/robots/iCubGazeboV2_6/model.urdf (robot description, URDF)
Before this commit: robot iCub, 189 links, 188 joints
Links:
- link l_foot: geometry collision box size=0.16 0.072 0.001; visual mesh filename=package://iCub/meshes/simmechanics/sim_sea_2-5_l_sole_prt-b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 scale=0.001 0.001 0.001
- link r_foot: geometry collision box size=0.16 0.072 0.001; visual mesh filename=package://iCub/meshes/simmechanics/sim_sea_2-5_r_sole_prt-b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 scale=0.001 0.001 0.001

File: iCub/robots/iCubGazeboV2_7/model.urdf (robot description, URDF)
Before this commit: robot iCub, 190 links, 189 joints
Links:
- link l_foot: geometry collision box size=0.16 0.072 0.001; visual mesh filename=package://iCub/meshes/simmechanics/sim_sea_2-5_l_sole_prt-b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 scale=0.001 0.001 0.001
- link r_foot: geometry collision box size=0.16 0.072 0.001; visual mesh filename=package://iCub/meshes/simmechanics/sim_sea_2-5_r_sole_prt-b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 scale=0.001 0.001 0.001
