Commit message: Automatic build. Travis build:398
icub-model-generator commit:e2a5b13c70b36be982fe9cc2b09f1d6a885ace79

urdf_parser_py commit:31474b9baaf7c3845b40e5a9aa87d5900a2282c3

simmechanics-to-urdf commit:1bd48b2d02b1d155a782f35d96865753c2e49706

yarp commit:fdd9c2157c150b6e617dc8bb55515d8b66ae4640

icub-main commit:7baee55743fef19fa163f12231bc0aa65354fb0b

idyntree commit:40ba1b919b5f730faf597cc4237b492d03f45708

File: iCub/robots/iCubGenova09/model.urdf (robot description, URDF)
Before this commit: robot iCub, 13 links, 12 joints
Links:
- added link head, mass 1.955; collision mesh filename=package://iCub/meshes/simmechanics/sim_icub3_head_prt.stl scale=0.001 0.001 0.001; visual mesh filename=package://iCub/meshes/simmechanics/sim_icub3_head_prt.stl scale=0.001 0.001 0.001
- added link l_ankle_1, mass 1.80595; collision mesh filename=package://iCub/meshes/simmechanics/sim_icub3_l_ankle_1_prt.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 scale=0.001 0.001 0.001; visual mesh filename=package://iCub/meshes/simmechanics/sim_icub3_l_ankle_1_prt.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 scale=0.001 0.001 0.001
- added link l_ankle_2, mass 1.06976; collision mesh filename=package://iCub/meshes/simmechanics/sim_icub3_l_ankle_2_prt.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 scale=0.001 0.001 0.001; visual mesh filename=package://iCub/meshes/simmechanics/sim_icub3_l_ankle_2_prt.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 scale=0.001 0.001 0.001
- added link l_foot_front, mass 0.723938; collision mesh filename=package://iCub/meshes/simmechanics/sim_icub3_l_foot_front_p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 scale=0.001 0.001 0.001; visual mesh filename=package://iCub/meshes/simmechanics/sim_icub3_l_foot_front_p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 scale=0.001 0.001 0.001
- added link l_foot_rear, mass 0.728095; collision mesh filename=package://iCub/meshes/simmechanics/sim_icub3_l_foot_rear_pr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 scale=0.001 0.001 0.001; visual mesh filename=package://iCub/meshes/simmechanics/sim_icub3_l_foot_rear_pr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 scale=0.001 0.001 0.001
- added link l_hip_1, mass 2.48546; collision mesh filename=package://iCub/meshes/simmechanics/sim_icub3_l_hip_1_prt.stl scale=0.001 0.001 0.001; visual mesh filename=package://iCub/meshes/simmechanics/sim_icub3_l_hip_1_prt.stl scale=0.001 0.001 0.001
- added link l_hip_2, mass 1.8834; collision mesh filename=package://iCub/meshes/simmechanics/sim_icub3_l_hip_2_prt.stl scale=0.001 0.001 0.001; visual mesh filename=package://iCub/meshes/simmechanics/sim_icub3_l_hip_2_prt.stl scale=0.001 0.001 0.001
- added link l_hip_3, mass 2.29352; collision mesh filename=package://iCub/meshes/simmechanics/sim_icub3_l_hip_3_prt.stl scale=0.001 0.001 0.001; visual mesh filename=package://iCub/meshes/simmechanics/sim_icub3_l_hip_3_prt.stl scale=0.001 0.001 0.001
- added link l_lower_leg, mass 4.59072; collision mesh filename=package://iCub/meshes/simmechanics/sim_icub3_l_lower_leg_pr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 scale=0.001 0.001 0.001; visual mesh filename=package://iCub/meshes/simmechanics/sim_icub3_l_lower_leg_pr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 scale=0.001 0.001 0.001
- added link l_sole
- added link l_upper_leg, mass 2.24396; collision mesh filename=package://iCub/meshes/simmechanics/sim_icub3_l_upper_leg_pr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 scale=0.001 0.001 0.001; visual mesh filename=package://iCub/meshes/simmechanics/sim_icub3_l_upper_leg_pr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 scale=0.001 0.001 0.001
- added link neck_1, mass 0.380522; collision mesh filename=package://iCub/meshes/simmechanics/sim_icub3_neck_1_prt.stl scale=0.001 0.001 0.001; visual mesh filename=package://iCub/meshes/simmechanics/sim_icub3_neck_1_prt.stl scale=0.001 0.001 0.001
- added link neck_2, mass 0.125914; collision mesh filename=package://iCub/meshes/simmechanics/sim_icub3_neck_2_prt.stl scale=0.001 0.001 0.001; visual mesh filename=package://iCub/meshes/simmechanics/sim_icub3_neck_2_prt.stl scale=0.001 0.001 0.001
- added link neck_3, mass 0.15881; collision mesh filename=package://iCub/meshes/simmechanics/sim_icub3_neck_3_prt.stl scale=0.001 0.001 0.001; visual mesh filename=package://iCub/meshes/simmechanics/sim_icub3_neck_3_prt.stl scale=0.001 0.001 0.001
- added link r_ankle_1, mass 1.80595; collision mesh filename=package://iCub/meshes/simmechanics/sim_icub3_r_ankle_1_prt.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 scale=0.001 0.001 0.001; visual mesh filename=package://iCub/meshes/simmechanics/sim_icub3_r_ankle_1_prt.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 scale=0.001 0.001 0.001
- added link r_ankle_2, mass 1.06976; collision mesh filename=package://iCub/meshes/simmechanics/sim_icub3_r_ankle_2_prt.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 scale=0.001 0.001 0.001; visual mesh filename=package://iCub/meshes/simmechanics/sim_icub3_r_ankle_2_prt.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 scale=0.001 0.001 0.001
- added link r_foot_front, mass 0.723938; collision mesh filename=package://iCub/meshes/simmechanics/sim_icub3_r_foot_front_p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 scale=0.001 0.001 0.001; visual mesh filename=package://iCub/meshes/simmechanics/sim_icub3_r_foot_front_p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 scale=0.001 0.001 0.001
- added link r_foot_rear, mass 0.728095; collision mesh filename=package://iCub/meshes/simmechanics/sim_icub3_r_foot_rear_pr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 scale=0.001 0.001 0.001; visual mesh filename=package://iCub/meshes/simmechanics/sim_icub3_r_foot_rear_pr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 scale=0.001 0.001 0.001
- added link r_hip_1, mass 2.48546; collision mesh filename=package://iCub/meshes/simmechanics/sim_icub3_r_hip_1_prt.stl scale=0.001 0.001 0.001; visual mesh filename=package://iCub/meshes/simmechanics/sim_icub3_r_hip_1_prt.stl scale=0.001 0.001 0.001
- added link r_hip_2, mass 1.8834; collision mesh filename=package://iCub/meshes/simmechanics/sim_icub3_r_hip_2_prt.stl scale=0.001 0.001 0.001; visual mesh filename=package://iCub/meshes/simmechanics/sim_icub3_r_hip_2_prt.stl scale=0.001 0.001 0.001
- added link r_hip_3, mass 2.29352; collision mesh filename=package://iCub/meshes/simmechanics/sim_icub3_r_hip_3_prt.stl scale=0.001 0.001 0.001; visual mesh filename=package://iCub/meshes/simmechanics/sim_icub3_r_hip_3_prt.stl scale=0.001 0.001 0.001
- added link r_lower_leg, mass 4.59072; collision mesh filename=package://iCub/meshes/simmechanics/sim_icub3_r_lower_leg_pr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 scale=0.001 0.001 0.001; visual mesh filename=package://iCub/meshes/simmechanics/sim_icub3_r_lower_leg_pr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 scale=0.001 0.001 0.001
- added link r_sole
- added link r_upper_leg, mass 2.24396; collision mesh filename=package://iCub/meshes/simmechanics/sim_icub3_r_upper_leg_pr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 scale=0.001 0.001 0.001; visual mesh filename=package://iCub/meshes/simmechanics/sim_icub3_r_upper_leg_pr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 scale=0.001 0.001 0.001
Joints:
- added joint l_ankle_pitch: type revolute, parent l_lower_leg, child l_ankle_1, origin xyz=0 -0.0005000000000000004 -0.255989 rpy=0 0 0, axis 0.0 -1.0 0.0, limit lower=-0.7853981633974483 upper=0.7853981633974483 effort=50000 velocity=120.0
- added joint l_ankle_roll: type revolute, parent l_ankle_1, child l_ankle_2, origin xyz=-0.052750000000000005 -0.018200000000000008 -0.03500000000000003 rpy=0 0 0, axis 1.0 0.0 0.0, limit lower=-0.4363323129985824 upper=0.4363323129985824 effort=50000 velocity=120.0
- added joint l_foot_front_ft_sensor: type fixed, parent l_ankle_2, child l_foot_front, origin xyz=0.13524999999999998 0 -0.06579999999999997 rpy=0 0 0
- added joint l_foot_rear_ft_sensor: type fixed, parent l_ankle_2, child l_foot_rear, origin xyz=0.016 0 -0.06579999999999997 rpy=0 0 0
- added joint l_hip_pitch: type revolute, parent root_link, child l_hip_1, origin xyz=0.0216 0.04045000000000001 0 rpy=0 0 0, axis 0.0 -1.0 0.0, limit lower=-0.7853981633974483 upper=2.007128639793479 effort=50000 velocity=120.0
- added joint l_hip_roll: type revolute, parent l_hip_1, child l_hip_2, origin xyz=-0.04725 0.0331 -0.009000000000000008 rpy=0 0 0, axis 1.0 0.0 0.0, limit lower=-0.17453292519943295 upper=2.007128639793479 effort=50000 velocity=120.0
- added joint l_hip_yaw: type revolute, parent l_hip_3, child l_upper_leg, origin xyz=0 -0.015000000000000006 -0.07090000000000007 rpy=0 0 0, axis 0.0 0.0 1.0, limit lower=-1.3962634015954636 upper=1.3962634015954636 effort=50000 velocity=120.0
- added joint l_knee: type revolute, parent l_upper_leg, child l_lower_leg, origin xyz=0.015 0.024900000000000012 -0.10619999999999996 rpy=0 0 0, axis 0.0 -1.0 0.0, limit lower=-1.2217304763960306 upper=0.08726646259971647 effort=50000 velocity=120.0
- added joint l_leg_ft_sensor: type fixed, parent l_hip_2, child l_hip_3, origin xyz=0.036699999999999997 0 -0.08969999999999995 rpy=0 0 0
- added joint l_sole_fixed_joint: type fixed, parent l_foot_rear, child l_sole, origin xyz=0.05963 0 0 rpy=0 0 0
- added joint neck_fixed_joint: type fixed, parent chest, child neck_1, origin xyz=-0.00378849 0 0.1652995 rpy=0 0 0
- added joint neck_pitch: type revolute, parent neck_1, child neck_2, origin xyz=0.00865 0 0.049000000000000016 rpy=0 0 0, axis 0.0 -1.0 0.0, limit lower=-0.5235987755982988 upper=0.3839724354387525 effort=50000 velocity=120.0
- added joint neck_roll: type revolute, parent neck_2, child neck_3, origin xyz=0 0 0.009500499999999995 rpy=0 0 0, axis 1.0 0.0 0.0, limit lower=-0.3490658503988659 upper=0.3490658503988659 effort=50000 velocity=120.0
- added joint neck_yaw: type revolute, parent neck_3, child head, origin xyz=0 0 0.06915000000000002 rpy=0 0 0, axis 0.0 0.0 -1.0, limit lower=-0.7853981633974483 upper=0.7853981633974483 effort=50000 velocity=120.0
- added joint r_ankle_pitch: type revolute, parent r_lower_leg, child r_ankle_1, origin xyz=0 0.0005000000000000004 -0.255989 rpy=0 0 0, axis 0.0 1.0 0.0, limit lower=-0.7853981633974483 upper=0.7853981633974483 effort=50000 velocity=120.0
- added joint r_ankle_roll: type revolute, parent r_ankle_1, child r_ankle_2, origin xyz=-0.052750000000000005 0.018200000000000008 -0.03500000000000003 rpy=0 0 0, axis 1.0 0.0 0.0, limit lower=-0.4363323129985824 upper=0.4363323129985824 effort=50000 velocity=120.0
- added joint r_foot_front_ft_sensor: type fixed, parent r_ankle_2, child r_foot_front, origin xyz=0.13525 0 -0.06579999999999997 rpy=0 0 0
- added joint r_foot_rear_ft_sensor: type fixed, parent r_ankle_2, child r_foot_rear, origin xyz=0.016 0 -0.06579999999999997 rpy=0 0 0
- added joint r_hip_pitch: type revolute, parent root_link, child r_hip_1, origin xyz=0.0216 -0.040549999999999996 0 rpy=0 0 0, axis 0.0 -1.0 0.0, limit lower=-0.7853981633974483 upper=2.007128639793479 effort=50000 velocity=120.0
- added joint r_hip_roll: type revolute, parent r_hip_1, child r_hip_2, origin xyz=-0.0473 -0.03310000000000001 -0.009000000000000008 rpy=0 0 0, axis 1.0 0.0 0.0, limit lower=-0.17453292519943295 upper=2.007128639793479 effort=50000 velocity=120.0
- added joint r_hip_yaw: type revolute, parent r_hip_3, child r_upper_leg, origin xyz=0 0.015000000000000006 -0.07090000000000007 rpy=0 0 0, axis 0.0 0.0 1.0, limit lower=-1.3962634015954636 upper=1.3962634015954636 effort=50000 velocity=120.0
- added joint r_knee: type revolute, parent r_upper_leg, child r_lower_leg, origin xyz=0.015000000000000003 -0.0249 -0.10619999999999996 rpy=0 0 0, axis 0.0 -1.0 0.0, limit lower=-1.2217304763960306 upper=0.08726646259971647 effort=50000 velocity=120.0
- added joint r_leg_ft_sensor: type fixed, parent r_hip_2, child r_hip_3, origin xyz=0.036699999999999997 0 -0.08969999999999995 rpy=0 0 0
- added joint r_sole_fixed_joint: type fixed, parent r_foot_rear, child r_sole, origin xyz=0.05963000000000001 0 0 rpy=0 0 0

Commit message: Add FT sensor on right upper leg with model generation

File: iCub/robots/iCubGenova09/model.urdf (robot description, URDF)
Before this commit: robot iCub, 48 links, 47 joints
Joints:
- joint l_elbow: origin xyz=0.009999930234919404 -0.001499647423428896 -0.12370033753758375 rpy=0 0 0 -> xyz=0.009999930234919404 -0.001499647423428896 -0.12370033753758372 rpy=0 0 0
- joint r_arm_ft_sensor: origin xyz=-0.006849946385389875 2.1904996055921444e-07 -0.05429998157789099 rpy=0 0 0 -> xyz=-0.006849946385389879 2.1904996055921444e-07 -0.054299981577890996 rpy=0 0 0
- joint r_shoulder_roll: origin xyz=0.007489008185044645 -0.11150041046657978 0.0004027858966975245 rpy=0.17453306234069357 -0.053747792579130614 -6.132332688812785e-07 -> xyz=0.007489008185044648 -0.11150041046657978 0.0004027858966975245 rpy=0.1745330623406936 -0.05374779257913062 -6.132332688847529e-07
- joint r_wrist_pitch: origin xyz=0.016299953353948633 -0.002007442890811839 -0.10750007971210637 rpy=0 0 0 -> xyz=0.016299953353948637 -0.002007442890811839 -0.10750007971210643 rpy=0 0 0
- joint r_wrist_yaw: origin xyz=-0.016300122874272734 0.0069993900510918194 0 rpy=0 0 0 -> xyz=-0.016300122874272727 0.0069993900510918194 0 rpy=0 0 0
