Commit message: Fix wrong collision of 'l_hand_little_1' in iCub_manual/iCubGazeboV2_5

File: iCub_manual/robots/iCubGazeboV2_5_visuomanip/model.urdf (robot description, URDF)
Before this commit: robot iCub, 102 links, 101 joints
Links:
- link l_hand_little_1: geometry collision mesh filename=package://iCub/meshes/col_LeftLittle1.dae scale=1.0 1.0 1.0; visual mesh filename=package://iCub/meshes/full_LeftLittle1.dae scale=1.0 1.0 1.0
