Commit message: rebase on top of upstream master parent 530d01711a919361163b3d7b2c54b701f2e27170 author mebbaid <mohd-b-mohd@hotmail.com> 1669978606 +0100 committer mebbaid <mohd-b-mohd@hotmail.com> 1669978616 +0100
fix rebase conflict

restore current version

added missing velocityControlImplementationType  param in config variables

delete un-used config files

add arm_no_hand config files to conf_manual

Fix Hands weird position

hand location fix

fix r_hand collision group

fix r_wrist_axis, play with camera sensors

correct file name in l_eye sensor

fix flipped pose of rgb sensors

fix l_eye and r_eye pan axis

Fix to make sure that ROS2 can find the iCub package (#178)

File: iCub_manual/robots/iCubGazeboV3_visuomanip/model.urdf (robot description, URDF)
Before this commit: robot iCub, 101 links, 100 joints
Links:
- link chest: mass 5.771074695 -> 7.5231
- link head: mass 1.831737118 -> 1.8728
- link l_elbow_1: mass 0.217768231 -> 0.22161
- link l_forearm: mass 0.858696525 -> 0.87311
- link l_shoulder_1: mass 1.376687449 -> 0.78644
- link l_shoulder_2: mass 0.304658373 -> 0.42492
- link l_shoulder_3: mass 0.242239185 -> 0.2625
- link l_upper_arm: mass 2.07285 -> 1.67729
- link l_wrist_1: mass 0.032535096 -> 0.033183
- link neck_1: mass 0.359964395 -> 0.36804
- link neck_2: mass 0.118740971 -> 0.1214
- link neck_3: mass 0.179822835 -> 0.18386
- link r_ankle_1: mass 0.346176903 -> 0.36569
- link r_ankle_2: mass 1.00828013 -> 1.3771
- link r_elbow_1: mass 0.217609341 -> 0.22157
- link r_foot_front: mass 0.17569926 -> 0.17964
- link r_forearm: mass 0.854281652 -> 0.8686
- link r_hand: mass 0.2499009 -> 0.25705; geometry collision mesh filename=package://iCub/meshes/col_RightHandPalm.dae scale=1.0 1.0 1.0; visual mesh filename=package://iCub/meshes/full_RightHandPalm.dae scale=1.0 1.0 1.0
- link r_hip_1: mass 2.134290199 -> 2.1623
- link r_hip_2: mass 1.779000764 -> 1.7731
- link r_hip_3: mass 2.1678368 -> 2.1635
- link r_lower_leg: mass 5.074105512 -> 5.0761
- link r_shoulder_1: mass 1.380716446 -> 0.78697
- link r_shoulder_2: mass 0.304658373 -> 0.42492
- link r_shoulder_3: mass 0.24467077 -> 0.2625
- link r_upper_arm: mass 1.960447492 -> 1.6219
- link r_upper_leg: mass 0.980691904 -> 0.90926
- link r_wrist_1: mass 0.032535096 -> 0.033183
- link root_link: mass 2.52649319 -> 2.5751
Joints:
- joint imu_frame_fixed_joint: origin xyz=0.0034999999997785457 0.0054999999863750895 0.1013340000004441 rpy=-3.141592653589793 0 -1.570796326794897 -> xyz=0.0035000000000000005 0.0055 0.10133400000000001 rpy=3.141592653589793 0 -1.5707963267948966
- joint l_eye_pan_joint: axis 0.0 1.0 0.0 -> 0.0 -1.0 0.0; origin xyz=0.0 0.0 -0.034 rpy=0.0 -1.5707963267949 0.0 -> xyz=0.0 0.0 0.034 rpy=0.0 -1.57 0.0
- joint l_shoulder_pitch: limit lower=-1.53588974175501 upper=0.22689280275926285 effort=50000 velocity=120.0 -> lower=-3.0543261909900767 upper=0.3490658503988659 effort=50000 velocity=120.0
- joint neck_yaw: axis -1.6255499221370677e-21 -1.0999983743979075e-15 1.0 -> 0.0 0.0 1.0
- joint r_eye_pan_joint: axis 0.0 1.0 0.0 -> 0.0 -1.0 0.0; origin xyz=0.0 0.0 0.034 rpy=0.0 -1.5707963267949 0.0 -> xyz=0.0 0.0 -0.034 rpy=0.0 -1.57 0.0
- joint r_hip_roll: limit lower=-0.17453292519943295 upper=2.007128639793479 effort=50000 velocity=120.0 -> lower=-0.17453292519943295 upper=1.9547687622336491 effort=50000 velocity=120.0
- joint r_shoulder_pitch: limit lower=-1.53588974175501 upper=0.22689280275926285 effort=50000 velocity=120.0 -> lower=-3.0543261909900767 upper=0.3490658503988659 effort=50000 velocity=120.0
- joint r_wrist_yaw: axis -2.4949582807394525e-07 1.0000002733514362 -2.7942487010105877e-08 -> -2.4949582807394525e-07 -1.0000002733514362 -2.7942487010105877e-08
