Commit message: Automatic build. Travis build:416
icub-model-generator commit:869ad5fe70e72bb7a5f274753c45823a31c4c82a

urdf_parser_py commit:31474b9baaf7c3845b40e5a9aa87d5900a2282c3

simmechanics-to-urdf commit:1bd48b2d02b1d155a782f35d96865753c2e49706

yarp commit:fdd9c2157c150b6e617dc8bb55515d8b66ae4640

icub-main commit:7baee55743fef19fa163f12231bc0aa65354fb0b

idyntree commit:40ba1b919b5f730faf597cc4237b492d03f45708

File: iCub/robots/iCubGazeboV3/model.urdf (robot description, URDF)
Before this commit: robot iCub, 45 links, 44 joints
Joints:
- joint torso_yaw: axis 0.0 0.0 1.0 -> 0.0 0.0 -1.0

File: iCub/robots/iCubGenova09/model.urdf (robot description, URDF)
Before this commit: robot iCub, 45 links, 44 joints
Joints:
- joint torso_yaw: axis 0.0 0.0 1.0 -> 0.0 0.0 -1.0

Commit message: Automatic build. Travis build:423
icub-model-generator commit:49a4e0a4d11a09895c207baba1b29c5395ecc662

urdf_parser_py commit:31474b9baaf7c3845b40e5a9aa87d5900a2282c3

simmechanics-to-urdf commit:1bd48b2d02b1d155a782f35d96865753c2e49706

yarp commit:fdd9c2157c150b6e617dc8bb55515d8b66ae4640

icub-main commit:7baee55743fef19fa163f12231bc0aa65354fb0b

idyntree commit:40ba1b919b5f730faf597cc4237b492d03f45708

File: iCub/robots/iCubGazeboV3/model.urdf (robot description, URDF)
Before this commit: robot iCub, 45 links, 44 joints
Joints:
- joint torso_pitch: axis 0.0 -1.0 0.0 -> 0.0 1.0 0.0

File: iCub/robots/iCubGenova09/model.urdf (robot description, URDF)
Before this commit: robot iCub, 45 links, 44 joints
Joints:
- joint torso_pitch: axis 0.0 -1.0 0.0 -> 0.0 1.0 0.0

Commit message: Automatic build. Travis build:425
icub-model-generator commit:e2a3dbb331cdde57f881b2017d58ae21156c9135

urdf_parser_py commit:31474b9baaf7c3845b40e5a9aa87d5900a2282c3

simmechanics-to-urdf commit:1bd48b2d02b1d155a782f35d96865753c2e49706

yarp commit:fdd9c2157c150b6e617dc8bb55515d8b66ae4640

icub-main commit:7baee55743fef19fa163f12231bc0aa65354fb0b

idyntree commit:40ba1b919b5f730faf597cc4237b492d03f45708

File: iCub/robots/iCubGazeboV3/model.urdf (robot description, URDF)
Before this commit: robot iCub, 45 links, 44 joints
Joints:
- joint r_hip_roll: axis 1.0 0.0 0.0 -> -1.0 0.0 0.0

File: iCub/robots/iCubGenova09/model.urdf (robot description, URDF)
Before this commit: robot iCub, 45 links, 44 joints
Joints:
- joint r_hip_roll: axis 1.0 0.0 0.0 -> -1.0 0.0 0.0

Commit message: Automatic build. Travis build:429
icub-model-generator commit:4a17a2be57e98823084dd4d2c669ba572d633cf8

urdf_parser_py commit:31474b9baaf7c3845b40e5a9aa87d5900a2282c3

simmechanics-to-urdf commit:1bd48b2d02b1d155a782f35d96865753c2e49706

yarp commit:fdd9c2157c150b6e617dc8bb55515d8b66ae4640

icub-main commit:7baee55743fef19fa163f12231bc0aa65354fb0b

idyntree commit:40ba1b919b5f730faf597cc4237b492d03f45708

File: iCub/robots/iCubGazeboV3/model.urdf (robot description, URDF)
Before this commit: robot iCub, 45 links, 44 joints
Joints:
- joint l_ankle_pitch: axis 0.0 -1.0 0.0 -> 0.0 1.0 0.0
- joint r_ankle_roll: axis 1.0 0.0 0.0 -> -1.0 0.0 0.0
- joint r_hip_yaw: axis 0.0 0.0 1.0 -> 0.0 0.0 -1.0
- joint torso_roll: axis 1.0 0.0 0.0 -> -1.0 0.0 0.0

File: iCub/robots/iCubGenova09/model.urdf (robot description, URDF)
Before this commit: robot iCub, 45 links, 44 joints
Joints:
- joint l_ankle_pitch: axis 0.0 -1.0 0.0 -> 0.0 1.0 0.0
- joint r_ankle_roll: axis 1.0 0.0 0.0 -> -1.0 0.0 0.0
- joint r_hip_yaw: axis 0.0 0.0 1.0 -> 0.0 0.0 -1.0
- joint torso_roll: axis 1.0 0.0 0.0 -> -1.0 0.0 0.0

Commit message: Automatic build. Travis build:498
icub-model-generator commit:5f1ccfe8031fa2bbcd341c83fd85a10a93b381bf

urdf_parser_py commit:31474b9baaf7c3845b40e5a9aa87d5900a2282c3

simmechanics-to-urdf commit:386e2c9c809d8d95e8e6c169cc23747de58ebae3

yarp commit:fdd9c2157c150b6e617dc8bb55515d8b66ae4640

icub-main commit:7baee55743fef19fa163f12231bc0aa65354fb0b

idyntree commit:40ba1b919b5f730faf597cc4237b492d03f45708

File: iCub/robots/iCubGazeboV3/model.urdf (robot description, URDF)
Before this commit: robot iCub, 45 links, 44 joints
Links:
- link l_foot_front: mass 0.723938 -> 0.18507432
- link l_foot_rear: mass 0.728095 -> 0.18460842
- link r_foot_front: mass 0.723938 -> 0.184375
- link r_foot_rear: mass 0.728095 -> 0.18484137

File: iCub/robots/iCubGenova09/model.urdf (robot description, URDF)
Before this commit: robot iCub, 45 links, 44 joints
Links:
- link l_foot_front: mass 0.723938 -> 0.18507432
- link l_foot_rear: mass 0.728095 -> 0.18460842
- link r_foot_front: mass 0.723938 -> 0.184375
- link r_foot_rear: mass 0.728095 -> 0.18484137

Commit message: Automatic build. GitHub Actions build: 372318540 icub-model-generator commit:f82b2fcaf5608b4da6495cd5433f970d76b3d425 urdf_parser_py commit:31474b9baaf7c3845b40e5a9aa87d5900a2282c3 simmechanics-to-urdf commit:386e2c9c809d8d95e8e6c169cc23747de58ebae3

File: iCub/robots/iCubGazeboV3/model.urdf (robot description, URDF)
Before this commit: robot iCub, 45 links, 44 joints
Links:
- added link chest_depth_frame
- added link chest_rgb_frame
- added link imu_frame
- link head: mass 1.955 -> 1.94302; geometry collision mesh filename=package://iCub/meshes/simmechanics/sim_head_head_prt.stl scale=0.001 0.001 0.001; visual mesh filename=package://iCub/meshes/simmechanics/sim_head_head_prt.stl scale=0.001 0.001 0.001
- link l_ankle_2: mass 1.06976 -> 1.06953
- link neck_1: mass 0.380522 -> 0.380603; geometry collision mesh filename=package://iCub/meshes/simmechanics/sim_head_neck_1_prt.stl scale=0.001 0.001 0.001; visual mesh filename=package://iCub/meshes/simmechanics/sim_head_neck_1_prt.stl scale=0.001 0.001 0.001
- link neck_2: mass 0.125914 -> 0.125549; geometry collision mesh filename=package://iCub/meshes/simmechanics/sim_head_neck_2_prt.stl scale=0.001 0.001 0.001; visual mesh filename=package://iCub/meshes/simmechanics/sim_head_neck_2_prt.stl scale=0.001 0.001 0.001
- link neck_3: mass 0.15881 -> 0.190133; geometry collision mesh filename=package://iCub/meshes/simmechanics/sim_head_neck_3_prt.stl scale=0.001 0.001 0.001; visual mesh filename=package://iCub/meshes/simmechanics/sim_head_neck_3_prt.stl scale=0.001 0.001 0.001
Joints:
- added joint chest_depth_frame_fixed_joint: type fixed, parent chest, child chest_depth_frame, origin xyz=0.0894115 0.0175 0.09929950000000001 rpy=-1.5707963267948968 0 -1.5707963267948968
- added joint chest_rgb_frame_fixed_joint: type fixed, parent chest, child chest_rgb_frame, origin xyz=0.0894115 -0.0115 0.09929950000000001 rpy=-1.5707963267948968 0 -1.5707963267948968
- added joint imu_frame_fixed_joint: type fixed, parent head, child imu_frame, origin xyz=0.0034999999997785457 0.0054999999863750895 0.1013340000004441 rpy=-3.141592653589793 0 -1.570796326794897
- joint l_hip_roll: limit lower=-0.17453292519943295 upper=2.007128639793479 effort=50000 velocity=120.0 -> lower=-10.0 upper=115.0 effort=50000 velocity=120.0; type revolute -> prismatic
- joint l_shoulder_pitch: axis 3.3231509266596455e-07 0.9999999783534343 1.4456511512603564e-07 -> 3.323079797554136e-07 0.9999999783534342 1.4452224303420037e-07; origin xyz=-0.020835100000000002 0.0397423 0.1052029 rpy=0.2532616237670649 -1.1982921379466467e-07 -0.26179930185680106 -> xyz=-0.020835100000000002 0.0397423 0.1052029 rpy=0.25326162380993705 -1.1977334179319483e-07 -0.26179930184968747
- joint l_shoulder_roll: origin xyz=0.004992849332498911 0.11149983845605199 0.00026865023223796025 rpy=-0.17453296136691587 -0.05374759926346641 0 -> xyz=0.004992849331690818 0.111499838456099 0.00026865022773668243 rpy=-0.17453296140985003 -0.05374759931933849 0
- joint neck_yaw: axis 0.0 0.0 -1.0 -> 1.6255499221370677e-21 1.0999983743979075e-15 -1.0

File: iCub/robots/iCubGenova09/model.urdf (robot description, URDF)
Before this commit: robot iCub, 45 links, 44 joints
Links:
- added link chest_depth_frame
- added link chest_rgb_frame
- added link imu_frame
- link head: mass 1.955 -> 1.94302; geometry collision mesh filename=package://iCub/meshes/simmechanics/sim_head_head_prt.stl scale=0.001 0.001 0.001; visual mesh filename=package://iCub/meshes/simmechanics/sim_head_head_prt.stl scale=0.001 0.001 0.001
- link l_ankle_2: mass 1.06976 -> 1.06953
- link neck_1: mass 0.380522 -> 0.380603; geometry collision mesh filename=package://iCub/meshes/simmechanics/sim_head_neck_1_prt.stl scale=0.001 0.001 0.001; visual mesh filename=package://iCub/meshes/simmechanics/sim_head_neck_1_prt.stl scale=0.001 0.001 0.001
- link neck_2: mass 0.125914 -> 0.125549; geometry collision mesh filename=package://iCub/meshes/simmechanics/sim_head_neck_2_prt.stl scale=0.001 0.001 0.001; visual mesh filename=package://iCub/meshes/simmechanics/sim_head_neck_2_prt.stl scale=0.001 0.001 0.001
- link neck_3: mass 0.15881 -> 0.190133; geometry collision mesh filename=package://iCub/meshes/simmechanics/sim_head_neck_3_prt.stl scale=0.001 0.001 0.001; visual mesh filename=package://iCub/meshes/simmechanics/sim_head_neck_3_prt.stl scale=0.001 0.001 0.001
Joints:
- added joint chest_depth_frame_fixed_joint: type fixed, parent chest, child chest_depth_frame, origin xyz=0.0894115 0.0175 0.09929950000000001 rpy=-1.5707963267948968 0 -1.5707963267948968
- added joint chest_rgb_frame_fixed_joint: type fixed, parent chest, child chest_rgb_frame, origin xyz=0.0894115 -0.0115 0.09929950000000001 rpy=-1.5707963267948968 0 -1.5707963267948968
- added joint imu_frame_fixed_joint: type fixed, parent head, child imu_frame, origin xyz=0.0034999999997785457 0.0054999999863750895 0.1013340000004441 rpy=-3.141592653589793 0 -1.570796326794897
- joint l_hip_roll: limit lower=-0.17453292519943295 upper=2.007128639793479 effort=50000 velocity=120.0 -> lower=-10.0 upper=115.0 effort=50000 velocity=120.0; type revolute -> prismatic
- joint l_shoulder_pitch: axis 3.3231509266596455e-07 0.9999999783534343 1.4456511512603564e-07 -> 3.323079797554136e-07 0.9999999783534342 1.4452224303420037e-07; origin xyz=-0.020835100000000002 0.0397423 0.1052029 rpy=0.2532616237670649 -1.1982921379466467e-07 -0.26179930185680106 -> xyz=-0.020835100000000002 0.0397423 0.1052029 rpy=0.25326162380993705 -1.1977334179319483e-07 -0.26179930184968747
- joint l_shoulder_roll: origin xyz=0.004992849332498911 0.11149983845605199 0.00026865023223796025 rpy=-0.17453296136691587 -0.05374759926346641 0 -> xyz=0.004992849331690818 0.111499838456099 0.00026865022773668243 rpy=-0.17453296140985003 -0.05374759931933849 0
- joint neck_yaw: axis 0.0 0.0 -1.0 -> 1.6255499221370677e-21 1.0999983743979075e-15 -1.0

Commit message: Automatic build. GitHub Actions build: 385409274 icub-model-generator commit:e52506de571df91913e41c003fbe913687bec5f5 urdf_parser_py commit:31474b9baaf7c3845b40e5a9aa87d5900a2282c3 simmechanics-to-urdf commit:f6055ab8d627c45138ddde46532ea42a74b48caa

File: iCub/robots/iCubGazeboV3/model.urdf (robot description, URDF)
Before this commit: robot iCub, 48 links, 47 joints
Links:
- link l_upper_arm: mass 2.07167 -> 2.06334

Commit message: Automatic build. GitHub Actions build: 385441971 icub-model-generator commit:add55e8a10302f6b224ecc3d19e3053cf4ebdce3 urdf_parser_py commit:31474b9baaf7c3845b40e5a9aa87d5900a2282c3 simmechanics-to-urdf commit:f6055ab8d627c45138ddde46532ea42a74b48caa

File: iCub/robots/iCubGazeboV3/model.urdf (robot description, URDF)
Before this commit: robot iCub, 48 links, 47 joints
Joints:
- joint l_hip_roll: limit lower=-10.0 upper=115.0 effort=50000 velocity=120.0 -> lower=-0.17453292519943295 upper=2.007128639793479 effort=50000 velocity=120.0; type prismatic -> revolute

File: iCub/robots/iCubGenova09/model.urdf (robot description, URDF)
Before this commit: robot iCub, 48 links, 47 joints
Joints:
- joint l_hip_roll: limit lower=-10.0 upper=115.0 effort=50000 velocity=120.0 -> lower=-0.17453292519943295 upper=2.007128639793479 effort=50000 velocity=120.0; type prismatic -> revolute

Commit message: Automatic build. GitHub Actions build: 391722343 icub-model-generator commit:28cb1942753233009dfb679838230edd94da146a urdf_parser_py commit:31474b9baaf7c3845b40e5a9aa87d5900a2282c3 simmechanics-to-urdf commit:f6055ab8d627c45138ddde46532ea42a74b48caa

File: iCub/robots/iCubGazeboV3/model.urdf (robot description, URDF)
Before this commit: robot iCub, 48 links, 47 joints
Joints:
- joint l_shoulder_yaw: axis -2.2276474049102235e-08 4.393786247302041e-08 1.0000002566182309 -> 2.2276474049102235e-08 -4.393786247302041e-08 -1.0000002566182309
- joint l_wrist_pitch: axis 0.9999998262417685 2.0348252625938444e-07 -4.023022846062156e-08 -> -0.9999998262417685 -2.0348252625938444e-07 4.023022846062156e-08
- joint l_wrist_prosup: axis -2.2276474049102235e-08 4.393786247302041e-08 1.0000002566182309 -> 2.2276474049102235e-08 -4.393786247302041e-08 -1.0000002566182309
- joint l_wrist_yaw: axis -8.811824174789715e-08 -1.0000002733514628 4.404736120498342e-08 -> 8.811824174789715e-08 1.0000002733514628 -4.404736120498342e-08

File: iCub/robots/iCubGenova09/model.urdf (robot description, URDF)
Before this commit: robot iCub, 48 links, 47 joints
Joints:
- joint l_shoulder_yaw: axis -2.2276474049102235e-08 4.393786247302041e-08 1.0000002566182309 -> 2.2276474049102235e-08 -4.393786247302041e-08 -1.0000002566182309
- joint l_wrist_pitch: axis 0.9999998262417685 2.0348252625938444e-07 -4.023022846062156e-08 -> -0.9999998262417685 -2.0348252625938444e-07 4.023022846062156e-08
- joint l_wrist_prosup: axis -2.2276474049102235e-08 4.393786247302041e-08 1.0000002566182309 -> 2.2276474049102235e-08 -4.393786247302041e-08 -1.0000002566182309
- joint l_wrist_yaw: axis -8.811824174789715e-08 -1.0000002733514628 4.404736120498342e-08 -> 8.811824174789715e-08 1.0000002733514628 -4.404736120498342e-08

Commit message: Automatic build. GitHub Actions build: 405601897 icub-model-generator commit:1783e40d230592b2df3c19d8d40cb0ee1d327e43 urdf_parser_py commit:31474b9baaf7c3845b40e5a9aa87d5900a2282c3 simmechanics-to-urdf commit:f6055ab8d627c45138ddde46532ea42a74b48caa

File: iCub/robots/iCubGazeboV3/model.urdf (robot description, URDF)
Before this commit: robot iCub, 48 links, 47 joints
Joints:
- joint l_arm_ft_sensor: origin xyz=-0.004350133156978318 3.632573233602887e-07 -0.05430003872406172 rpy=0 0 0 -> xyz=-0.004350133156978329 3.632573233880443e-07 -0.05430003872406172 rpy=0 0 0
- joint l_elbow: axis -8.811824174789715e-08 -1.0000002733514628 4.404736120498342e-08 -> -8.811824154381087e-08 -1.0000002733514628 4.4047361189014644e-08
- joint l_shoulder_pitch: axis 3.323079797554136e-07 0.9999999783534342 1.4452224303420037e-07 -> 3.323079797673039e-07 0.9999999783534342 1.4452224303407313e-07
- joint l_shoulder_roll: axis 0.9999998262417685 2.0348252625938444e-07 -4.023022846062156e-08 -> 0.9999998262417684 2.0348252649342313e-07 -4.0230228454118944e-08; origin xyz=0.004992849331690818 0.111499838456099 0.00026865022773668243 rpy=-0.17453296140985003 -0.05374759931933849 0 -> xyz=0.004992849331690818 0.111499838456099 0.0002686502277366859 rpy=-0.17453296140985 -0.05374759931933852 0
- joint l_shoulder_yaw: axis 2.2276474049102235e-08 -4.393786247302041e-08 -1.0000002566182309 -> 2.227647404040578e-08 -4.393786245948661e-08 -1.0000002566182309; origin xyz=0 -4.2345248449371375e-07 -0.022499941373124423 rpy=0 0 0 -> xyz=0 -4.2345248449371375e-07 -0.02249994137312443 rpy=0 0 0
- joint l_wrist_pitch: axis -0.9999998262417685 -2.0348252625938444e-07 4.023022846062156e-08 -> -0.9999998262417684 -2.0348252649342313e-07 4.0230228454118944e-08; origin xyz=0.016600015934286182 0.0020068952180725685 -0.10749964114254112 rpy=0 0 0 -> xyz=0.016600015934286182 0.002006895218072541 -0.10749964114254112 rpy=0 0 0
- joint l_wrist_prosup: axis 2.2276474049102235e-08 -4.393786247302041e-08 -1.0000002566182309 -> 2.227647404040578e-08 -4.393786245948661e-08 -1.0000002566182309; origin xyz=-0.0149998706541777 0.0019996435036348514 -0.0553000635824798 rpy=0 0 0 -> xyz=-0.014999870654177704 0.0019996435036348514 -0.055300063582479825 rpy=0 0 0
- joint l_wrist_yaw: axis 8.811824174789715e-08 1.0000002733514628 -4.404736120498342e-08 -> 8.811824154381087e-08 1.0000002733514628 -4.4047361189014644e-08; origin xyz=-0.016300121744729387 -0.006999392681571209 0 rpy=0 0 0 -> xyz=-0.016300121744729387 -0.0069993926815711816 0 rpy=0 0 0
- joint r_arm_ft_sensor: origin xyz=-0.006849946385389872 2.1904996058697002e-07 -0.05429998157789099 rpy=0 0 0 -> xyz=-0.006849946385389875 2.1904996055921444e-07 -0.05429998157789099 rpy=0 0 0
- joint r_elbow: axis 2.4949582807394525e-07 -1.0000002733514362 2.7942487010105877e-08 -> 2.4949582809984105e-07 -1.0000002733514362 2.7942487004772865e-08; origin xyz=0.00999993192260382 0.0014996401320274133 -0.1237003374895465 rpy=0 0 0 -> xyz=0.009999931922603816 0.0014996401320274133 -0.1237003374895465 rpy=0 0 0
- joint r_shoulder_pitch: axis 1.499044390098182e-07 0.9999999783534812 -1.2401537036323317e-07 -> 1.499044390054707e-07 0.9999999783534812 -1.2401537036188515e-07
- joint r_shoulder_roll: axis -0.9999998262417886 4.210501434612913e-08 2.4630481182686846e-08 -> -0.9999998262417886 4.2105014356162707e-08 2.4630481189336084e-08; origin xyz=0.007489008185044645 -0.11150041046657978 0.0004027858966975245 rpy=0.17453306234069352 -0.05374779257913059 -6.132332688804098e-07 -> xyz=0.007489008185044645 -0.11150041046657978 0.0004027858966975245 rpy=0.17453306234069357 -0.053747792579130614 -6.132332688812785e-07
- joint r_shoulder_yaw: axis -3.787621790776764e-08 2.805197706023475e-08 1.0000002566182309 -> -3.787621790513063e-08 2.805197706068352e-08 1.0000002566182309; origin xyz=0 4.2183273077367467e-07 -0.02249994137315358 rpy=0 0 0 -> xyz=0 4.2183273077367467e-07 -0.022499941373153573 rpy=0 0 0
- joint r_wrist_pitch: axis 0.9999998262417886 -4.210501434612913e-08 -2.4630481182686846e-08 -> 0.9999998262417886 -4.2105014356162707e-08 -2.4630481189336084e-08
- joint r_wrist_prosup: axis -3.787621790776764e-08 2.805197706023475e-08 1.0000002566182309 -> -3.787621790513063e-08 2.805197706068352e-08 1.0000002566182309; origin xyz=-0.014999869468812953 -0.0019996499053189787 -0.05530006367251966 rpy=0 0 0 -> xyz=-0.014999869468812953 -0.001999649905318951 -0.05530006367251966 rpy=0 0 0
- joint r_wrist_yaw: axis -2.4949582807394525e-07 1.0000002733514362 -2.7942487010105877e-08 -> -2.4949582809984105e-07 1.0000002733514362 -2.7942487004772865e-08; origin xyz=-0.016300122874272734 0.006999390051091792 0 rpy=0 0 0 -> xyz=-0.016300122874272734 0.0069993900510918194 0 rpy=0 0 0

File: iCub/robots/iCubGenova09/model.urdf (robot description, URDF)
Before this commit: robot iCub, 48 links, 47 joints
Joints:
- joint l_arm_ft_sensor: origin xyz=-0.004350133156978318 3.632573233602887e-07 -0.05430003872406172 rpy=0 0 0 -> xyz=-0.004350133156978329 3.632573233880443e-07 -0.05430003872406172 rpy=0 0 0
- joint l_elbow: axis -8.811824174789715e-08 -1.0000002733514628 4.404736120498342e-08 -> -8.811824154381087e-08 -1.0000002733514628 4.4047361189014644e-08
- joint l_shoulder_pitch: axis 3.323079797554136e-07 0.9999999783534342 1.4452224303420037e-07 -> 3.323079797673039e-07 0.9999999783534342 1.4452224303407313e-07
- joint l_shoulder_roll: axis 0.9999998262417685 2.0348252625938444e-07 -4.023022846062156e-08 -> 0.9999998262417684 2.0348252649342313e-07 -4.0230228454118944e-08; origin xyz=0.004992849331690818 0.111499838456099 0.00026865022773668243 rpy=-0.17453296140985003 -0.05374759931933849 0 -> xyz=0.004992849331690818 0.111499838456099 0.0002686502277366859 rpy=-0.17453296140985 -0.05374759931933852 0
- joint l_shoulder_yaw: axis 2.2276474049102235e-08 -4.393786247302041e-08 -1.0000002566182309 -> 2.227647404040578e-08 -4.393786245948661e-08 -1.0000002566182309; origin xyz=0 -4.2345248449371375e-07 -0.022499941373124423 rpy=0 0 0 -> xyz=0 -4.2345248449371375e-07 -0.02249994137312443 rpy=0 0 0
- joint l_wrist_pitch: axis -0.9999998262417685 -2.0348252625938444e-07 4.023022846062156e-08 -> -0.9999998262417684 -2.0348252649342313e-07 4.0230228454118944e-08; origin xyz=0.016600015934286182 0.0020068952180725685 -0.10749964114254112 rpy=0 0 0 -> xyz=0.016600015934286182 0.002006895218072541 -0.10749964114254112 rpy=0 0 0
- joint l_wrist_prosup: axis 2.2276474049102235e-08 -4.393786247302041e-08 -1.0000002566182309 -> 2.227647404040578e-08 -4.393786245948661e-08 -1.0000002566182309; origin xyz=-0.0149998706541777 0.0019996435036348514 -0.0553000635824798 rpy=0 0 0 -> xyz=-0.014999870654177704 0.0019996435036348514 -0.055300063582479825 rpy=0 0 0
- joint l_wrist_yaw: axis 8.811824174789715e-08 1.0000002733514628 -4.404736120498342e-08 -> 8.811824154381087e-08 1.0000002733514628 -4.4047361189014644e-08; origin xyz=-0.016300121744729387 -0.006999392681571209 0 rpy=0 0 0 -> xyz=-0.016300121744729387 -0.0069993926815711816 0 rpy=0 0 0
- joint r_arm_ft_sensor: origin xyz=-0.006849946385389872 2.1904996058697002e-07 -0.05429998157789099 rpy=0 0 0 -> xyz=-0.006849946385389875 2.1904996055921444e-07 -0.05429998157789099 rpy=0 0 0
- joint r_elbow: axis 2.4949582807394525e-07 -1.0000002733514362 2.7942487010105877e-08 -> 2.4949582809984105e-07 -1.0000002733514362 2.7942487004772865e-08; origin xyz=0.00999993192260382 0.0014996401320274133 -0.1237003374895465 rpy=0 0 0 -> xyz=0.009999931922603816 0.0014996401320274133 -0.1237003374895465 rpy=0 0 0
- joint r_shoulder_pitch: axis 1.499044390098182e-07 0.9999999783534812 -1.2401537036323317e-07 -> 1.499044390054707e-07 0.9999999783534812 -1.2401537036188515e-07
- joint r_shoulder_roll: axis -0.9999998262417886 4.210501434612913e-08 2.4630481182686846e-08 -> -0.9999998262417886 4.2105014356162707e-08 2.4630481189336084e-08; origin xyz=0.007489008185044645 -0.11150041046657978 0.0004027858966975245 rpy=0.17453306234069352 -0.05374779257913059 -6.132332688804098e-07 -> xyz=0.007489008185044645 -0.11150041046657978 0.0004027858966975245 rpy=0.17453306234069357 -0.053747792579130614 -6.132332688812785e-07
- joint r_shoulder_yaw: axis -3.787621790776764e-08 2.805197706023475e-08 1.0000002566182309 -> -3.787621790513063e-08 2.805197706068352e-08 1.0000002566182309; origin xyz=0 4.2183273077367467e-07 -0.02249994137315358 rpy=0 0 0 -> xyz=0 4.2183273077367467e-07 -0.022499941373153573 rpy=0 0 0
- joint r_wrist_pitch: axis 0.9999998262417886 -4.210501434612913e-08 -2.4630481182686846e-08 -> 0.9999998262417886 -4.2105014356162707e-08 -2.4630481189336084e-08
- joint r_wrist_prosup: axis -3.787621790776764e-08 2.805197706023475e-08 1.0000002566182309 -> -3.787621790513063e-08 2.805197706068352e-08 1.0000002566182309; origin xyz=-0.014999869468812953 -0.0019996499053189787 -0.05530006367251966 rpy=0 0 0 -> xyz=-0.014999869468812953 -0.001999649905318951 -0.05530006367251966 rpy=0 0 0
- joint r_wrist_yaw: axis -2.4949582807394525e-07 1.0000002733514362 -2.7942487010105877e-08 -> -2.4949582809984105e-07 1.0000002733514362 -2.7942487004772865e-08; origin xyz=-0.016300122874272734 0.006999390051091792 0 rpy=0 0 0 -> xyz=-0.016300122874272734 0.0069993900510918194 0 rpy=0 0 0
