Commit message: Automatic build. GitHub Actions build: 415084145 icub-model-generator commit:24a3dd74b402c80c068076f2a55028ba9c2352a7 urdf_parser_py commit:31474b9baaf7c3845b40e5a9aa87d5900a2282c3 simmechanics-to-urdf commit:f6055ab8d627c45138ddde46532ea42a74b48caa

File: iCub/robots/iCubGazeboV3/model.urdf (robot description, URDF)
Before this commit: robot iCub, 48 links, 47 joints
Joints:
- joint l_arm_ft_sensor: origin xyz=-0.004350133156978329 3.632573233880443e-07 -0.05430003872406172 rpy=0 0 0 -> xyz=-0.004350133156978318 3.632573233602887e-07 -0.05430003872406172 rpy=0 0 0
- joint l_elbow: axis -8.811824154381087e-08 -1.0000002733514628 4.4047361189014644e-08 -> -8.811824174789715e-08 -1.0000002733514628 4.404736120498342e-08
- joint l_shoulder_pitch: axis 3.323079797673039e-07 0.9999999783534342 1.4452224303407313e-07 -> 3.323079797554136e-07 0.9999999783534342 1.4452224303420037e-07
- joint l_shoulder_roll: axis 0.9999998262417684 2.0348252649342313e-07 -4.0230228454118944e-08 -> 0.9999998262417685 2.0348252625938444e-07 -4.023022846062156e-08; origin xyz=0.004992849331690818 0.111499838456099 0.0002686502277366859 rpy=-0.17453296140985 -0.05374759931933852 0 -> xyz=0.004992849331690818 0.111499838456099 0.00026865022773668243 rpy=-0.17453296140985003 -0.05374759931933849 0
- joint l_shoulder_yaw: axis 2.227647404040578e-08 -4.393786245948661e-08 -1.0000002566182309 -> 2.2276474049102235e-08 -4.393786247302041e-08 -1.0000002566182309; origin xyz=0 -4.2345248449371375e-07 -0.02249994137312443 rpy=0 0 0 -> xyz=0 -4.2345248449371375e-07 -0.022499941373124423 rpy=0 0 0
- joint l_wrist_pitch: axis -0.9999998262417684 -2.0348252649342313e-07 4.0230228454118944e-08 -> -0.9999998262417685 -2.0348252625938444e-07 4.023022846062156e-08; origin xyz=0.016600015934286182 0.002006895218072541 -0.10749964114254112 rpy=0 0 0 -> xyz=0.016600015934286182 0.0020068952180725685 -0.10749964114254112 rpy=0 0 0
- joint l_wrist_prosup: axis 2.227647404040578e-08 -4.393786245948661e-08 -1.0000002566182309 -> 2.2276474049102235e-08 -4.393786247302041e-08 -1.0000002566182309; origin xyz=-0.014999870654177704 0.0019996435036348514 -0.055300063582479825 rpy=0 0 0 -> xyz=-0.0149998706541777 0.0019996435036348514 -0.0553000635824798 rpy=0 0 0
- joint l_wrist_yaw: axis 8.811824154381087e-08 1.0000002733514628 -4.4047361189014644e-08 -> 8.811824174789715e-08 1.0000002733514628 -4.404736120498342e-08; origin xyz=-0.016300121744729387 -0.0069993926815711816 0 rpy=0 0 0 -> xyz=-0.016300121744729387 -0.006999392681571209 0 rpy=0 0 0
- joint r_arm_ft_sensor: origin xyz=-0.006849946385389875 2.1904996055921444e-07 -0.05429998157789099 rpy=0 0 0 -> xyz=-0.006849946385389872 2.1904996058697002e-07 -0.05429998157789099 rpy=0 0 0
- joint r_elbow: axis 2.4949582809984105e-07 -1.0000002733514362 2.7942487004772865e-08 -> 2.4949582807394525e-07 -1.0000002733514362 2.7942487010105877e-08; origin xyz=0.009999931922603816 0.0014996401320274133 -0.1237003374895465 rpy=0 0 0 -> xyz=0.00999993192260382 0.0014996401320274133 -0.1237003374895465 rpy=0 0 0
- joint r_shoulder_pitch: axis 1.499044390054707e-07 0.9999999783534812 -1.2401537036188515e-07 -> 1.499044390098182e-07 0.9999999783534812 -1.2401537036323317e-07
- joint r_shoulder_roll: axis -0.9999998262417886 4.2105014356162707e-08 2.4630481189336084e-08 -> -0.9999998262417886 4.210501434612913e-08 2.4630481182686846e-08; origin xyz=0.007489008185044645 -0.11150041046657978 0.0004027858966975245 rpy=0.17453306234069357 -0.053747792579130614 -6.132332688812785e-07 -> xyz=0.007489008185044645 -0.11150041046657978 0.0004027858966975245 rpy=0.17453306234069352 -0.05374779257913059 -6.132332688804098e-07
- joint r_shoulder_yaw: axis -3.787621790513063e-08 2.805197706068352e-08 1.0000002566182309 -> -3.787621790776764e-08 2.805197706023475e-08 1.0000002566182309; origin xyz=0 4.2183273077367467e-07 -0.022499941373153573 rpy=0 0 0 -> xyz=0 4.2183273077367467e-07 -0.02249994137315358 rpy=0 0 0
- joint r_wrist_pitch: axis 0.9999998262417886 -4.2105014356162707e-08 -2.4630481189336084e-08 -> 0.9999998262417886 -4.210501434612913e-08 -2.4630481182686846e-08
- joint r_wrist_prosup: axis -3.787621790513063e-08 2.805197706068352e-08 1.0000002566182309 -> -3.787621790776764e-08 2.805197706023475e-08 1.0000002566182309; origin xyz=-0.014999869468812953 -0.001999649905318951 -0.05530006367251966 rpy=0 0 0 -> xyz=-0.014999869468812953 -0.0019996499053189787 -0.05530006367251966 rpy=0 0 0
- joint r_wrist_yaw: axis -2.4949582809984105e-07 1.0000002733514362 -2.7942487004772865e-08 -> -2.4949582807394525e-07 1.0000002733514362 -2.7942487010105877e-08; origin xyz=-0.016300122874272734 0.0069993900510918194 0 rpy=0 0 0 -> xyz=-0.016300122874272734 0.006999390051091792 0 rpy=0 0 0

File: iCub/robots/iCubGenova09/model.urdf (robot description, URDF)
Before this commit: robot iCub, 48 links, 47 joints
Joints:
- joint l_arm_ft_sensor: origin xyz=-0.004350133156978329 3.632573233880443e-07 -0.05430003872406172 rpy=0 0 0 -> xyz=-0.004350133156978318 3.632573233602887e-07 -0.05430003872406172 rpy=0 0 0
- joint l_elbow: axis -8.811824154381087e-08 -1.0000002733514628 4.4047361189014644e-08 -> -8.811824174789715e-08 -1.0000002733514628 4.404736120498342e-08
- joint l_shoulder_pitch: axis 3.323079797673039e-07 0.9999999783534342 1.4452224303407313e-07 -> 3.323079797554136e-07 0.9999999783534342 1.4452224303420037e-07
- joint l_shoulder_roll: axis 0.9999998262417684 2.0348252649342313e-07 -4.0230228454118944e-08 -> 0.9999998262417685 2.0348252625938444e-07 -4.023022846062156e-08; origin xyz=0.004992849331690818 0.111499838456099 0.0002686502277366859 rpy=-0.17453296140985 -0.05374759931933852 0 -> xyz=0.004992849331690818 0.111499838456099 0.00026865022773668243 rpy=-0.17453296140985003 -0.05374759931933849 0
- joint l_shoulder_yaw: axis 2.227647404040578e-08 -4.393786245948661e-08 -1.0000002566182309 -> 2.2276474049102235e-08 -4.393786247302041e-08 -1.0000002566182309; origin xyz=0 -4.2345248449371375e-07 -0.02249994137312443 rpy=0 0 0 -> xyz=0 -4.2345248449371375e-07 -0.022499941373124423 rpy=0 0 0
- joint l_wrist_pitch: axis -0.9999998262417684 -2.0348252649342313e-07 4.0230228454118944e-08 -> -0.9999998262417685 -2.0348252625938444e-07 4.023022846062156e-08; origin xyz=0.016600015934286182 0.002006895218072541 -0.10749964114254112 rpy=0 0 0 -> xyz=0.016600015934286182 0.0020068952180725685 -0.10749964114254112 rpy=0 0 0
- joint l_wrist_prosup: axis 2.227647404040578e-08 -4.393786245948661e-08 -1.0000002566182309 -> 2.2276474049102235e-08 -4.393786247302041e-08 -1.0000002566182309; origin xyz=-0.014999870654177704 0.0019996435036348514 -0.055300063582479825 rpy=0 0 0 -> xyz=-0.0149998706541777 0.0019996435036348514 -0.0553000635824798 rpy=0 0 0
- joint l_wrist_yaw: axis 8.811824154381087e-08 1.0000002733514628 -4.4047361189014644e-08 -> 8.811824174789715e-08 1.0000002733514628 -4.404736120498342e-08; origin xyz=-0.016300121744729387 -0.0069993926815711816 0 rpy=0 0 0 -> xyz=-0.016300121744729387 -0.006999392681571209 0 rpy=0 0 0
- joint r_arm_ft_sensor: origin xyz=-0.006849946385389875 2.1904996055921444e-07 -0.05429998157789099 rpy=0 0 0 -> xyz=-0.006849946385389872 2.1904996058697002e-07 -0.05429998157789099 rpy=0 0 0
- joint r_elbow: axis 2.4949582809984105e-07 -1.0000002733514362 2.7942487004772865e-08 -> 2.4949582807394525e-07 -1.0000002733514362 2.7942487010105877e-08; origin xyz=0.009999931922603816 0.0014996401320274133 -0.1237003374895465 rpy=0 0 0 -> xyz=0.00999993192260382 0.0014996401320274133 -0.1237003374895465 rpy=0 0 0
- joint r_shoulder_pitch: axis 1.499044390054707e-07 0.9999999783534812 -1.2401537036188515e-07 -> 1.499044390098182e-07 0.9999999783534812 -1.2401537036323317e-07
- joint r_shoulder_roll: axis -0.9999998262417886 4.2105014356162707e-08 2.4630481189336084e-08 -> -0.9999998262417886 4.210501434612913e-08 2.4630481182686846e-08; origin xyz=0.007489008185044645 -0.11150041046657978 0.0004027858966975245 rpy=0.17453306234069357 -0.053747792579130614 -6.132332688812785e-07 -> xyz=0.007489008185044645 -0.11150041046657978 0.0004027858966975245 rpy=0.17453306234069352 -0.05374779257913059 -6.132332688804098e-07
- joint r_shoulder_yaw: axis -3.787621790513063e-08 2.805197706068352e-08 1.0000002566182309 -> -3.787621790776764e-08 2.805197706023475e-08 1.0000002566182309; origin xyz=0 4.2183273077367467e-07 -0.022499941373153573 rpy=0 0 0 -> xyz=0 4.2183273077367467e-07 -0.02249994137315358 rpy=0 0 0
- joint r_wrist_pitch: axis 0.9999998262417886 -4.2105014356162707e-08 -2.4630481189336084e-08 -> 0.9999998262417886 -4.210501434612913e-08 -2.4630481182686846e-08
- joint r_wrist_prosup: axis -3.787621790513063e-08 2.805197706068352e-08 1.0000002566182309 -> -3.787621790776764e-08 2.805197706023475e-08 1.0000002566182309; origin xyz=-0.014999869468812953 -0.001999649905318951 -0.05530006367251966 rpy=0 0 0 -> xyz=-0.014999869468812953 -0.0019996499053189787 -0.05530006367251966 rpy=0 0 0
- joint r_wrist_yaw: axis -2.4949582809984105e-07 1.0000002733514362 -2.7942487004772865e-08 -> -2.4949582807394525e-07 1.0000002733514362 -2.7942487010105877e-08; origin xyz=-0.016300122874272734 0.0069993900510918194 0 rpy=0 0 0 -> xyz=-0.016300122874272734 0.006999390051091792 0 rpy=0 0 0

Commit message: Automatic build. GitHub Actions build: 415891553 icub-model-generator commit:robotology/icub-models-generator@6ffba96867cd8b3293cdb6e519a7f79b9baa7c4a urdf_parser_py commit:ros/urdf_parser_py@31474b9baaf7c3845b40e5a9aa87d5900a2282c3 simmechanics-to-urdf commit:robotology/simmechanics-to-urdf@f6055ab8d627c45138ddde46532ea42a74b48caa

File: iCub/robots/iCubGazeboV3/model.urdf (robot description, URDF)
Before this commit: robot iCub, 48 links, 47 joints
Joints:
- joint neck_yaw: axis 1.6255499221370677e-21 1.0999983743979075e-15 -1.0 -> -1.6255499221370677e-21 -1.0999983743979075e-15 1.0

File: iCub/robots/iCubGenova09/model.urdf (robot description, URDF)
Before this commit: robot iCub, 48 links, 47 joints
Joints:
- joint neck_yaw: axis 1.6255499221370677e-21 1.0999983743979075e-15 -1.0 -> -1.6255499221370677e-21 -1.0999983743979075e-15 1.0

Commit message: Automatic build. GitHub Actions build: 518010635 icub-model-generator commit: robotology/icub-models-generator@5090736272aec2e339a9eb71b21d7f00744f991e urdf_parser_py commit: ros/urdf_parser_py@31474b9baaf7c3845b40e5a9aa87d5900a2282c3 simmechanics-to-urdf commit: robotology/simmechanics-to-urdf@f6055ab8d627c45138ddde46532ea42a74b48caa

File: iCub/robots/iCubGazeboV3/model.urdf (robot description, URDF)
Before this commit: robot iCub, 48 links, 47 joints
Links:
- link head: mass 1.94302 -> 1.93676
- link l_ankle_1: mass 1.80595 -> 0.366025
- link l_foot_front: mass 0.18507432 -> 0.185074
- link l_foot_rear: mass 0.18460842 -> 0.184608
- link l_lower_leg: mass 4.59072 -> 5.66584
- link r_ankle_1: mass 1.80595 -> 0.366025
- link r_ankle_2: mass 1.06976 -> 1.06609
- link r_foot_front: mass 0.184375 -> 0.185773
- link r_foot_rear: mass 0.18484137 -> 0.184841
- link r_hip_1: mass 2.48546 -> 2.50002
- link r_hip_2: mass 1.8834 -> 1.881
- link r_hip_3: mass 2.29352 -> 2.29213
- link r_lower_leg: mass 4.59072 -> 5.89871
- link r_upper_leg: mass 2.24396 -> 2.2571
Joints:
- joint l_arm_ft_sensor: origin xyz=-0.004350133156978329 3.632573233880443e-07 -0.05430003872406172 rpy=0 0 0 -> xyz=-0.004350133156978318 3.632573233602887e-07 -0.05430003872406172 rpy=0 0 0
- joint l_elbow: axis -8.811824154381087e-08 -1.0000002733514628 4.4047361189014644e-08 -> -8.811824174789715e-08 -1.0000002733514628 4.404736120498342e-08
- joint l_shoulder_pitch: axis 3.323079797673039e-07 0.9999999783534342 1.4452224303407313e-07 -> 3.323079797554136e-07 0.9999999783534342 1.4452224303420037e-07
- joint l_shoulder_roll: axis 0.9999998262417684 2.0348252649342313e-07 -4.0230228454118944e-08 -> 0.9999998262417685 2.0348252625938444e-07 -4.023022846062156e-08; origin xyz=0.004992849331690818 0.111499838456099 0.0002686502277366859 rpy=-0.17453296140985 -0.05374759931933852 0 -> xyz=0.004992849331690818 0.111499838456099 0.00026865022773668243 rpy=-0.17453296140985003 -0.05374759931933849 0
- joint l_shoulder_yaw: axis 2.227647404040578e-08 -4.393786245948661e-08 -1.0000002566182309 -> 2.2276474049102235e-08 -4.393786247302041e-08 -1.0000002566182309; origin xyz=0 -4.2345248449371375e-07 -0.02249994137312443 rpy=0 0 0 -> xyz=0 -4.2345248449371375e-07 -0.022499941373124423 rpy=0 0 0
- joint l_wrist_pitch: axis -0.9999998262417684 -2.0348252649342313e-07 4.0230228454118944e-08 -> -0.9999998262417685 -2.0348252625938444e-07 4.023022846062156e-08; origin xyz=0.016600015934286182 0.002006895218072541 -0.10749964114254112 rpy=0 0 0 -> xyz=0.016600015934286182 0.0020068952180725685 -0.10749964114254112 rpy=0 0 0
- joint l_wrist_prosup: axis 2.227647404040578e-08 -4.393786245948661e-08 -1.0000002566182309 -> 2.2276474049102235e-08 -4.393786247302041e-08 -1.0000002566182309; origin xyz=-0.014999870654177704 0.0019996435036348514 -0.055300063582479825 rpy=0 0 0 -> xyz=-0.0149998706541777 0.0019996435036348514 -0.0553000635824798 rpy=0 0 0
- joint l_wrist_yaw: axis 8.811824154381087e-08 1.0000002733514628 -4.4047361189014644e-08 -> 8.811824174789715e-08 1.0000002733514628 -4.404736120498342e-08; origin xyz=-0.016300121744729387 -0.0069993926815711816 0 rpy=0 0 0 -> xyz=-0.016300121744729387 -0.006999392681571209 0 rpy=0 0 0
- joint r_arm_ft_sensor: origin xyz=-0.006849946385389875 2.1904996055921444e-07 -0.05429998157789099 rpy=0 0 0 -> xyz=-0.006849946385389872 2.1904996058697002e-07 -0.05429998157789099 rpy=0 0 0
- joint r_elbow: axis 2.4949582809984105e-07 -1.0000002733514362 2.7942487004772865e-08 -> 2.4949582807394525e-07 -1.0000002733514362 2.7942487010105877e-08; origin xyz=0.009999931922603816 0.0014996401320274133 -0.1237003374895465 rpy=0 0 0 -> xyz=0.00999993192260382 0.0014996401320274133 -0.1237003374895465 rpy=0 0 0
- joint r_shoulder_pitch: axis 1.499044390054707e-07 0.9999999783534812 -1.2401537036188515e-07 -> 1.499044390098182e-07 0.9999999783534812 -1.2401537036323317e-07
- joint r_shoulder_roll: axis -0.9999998262417886 4.2105014356162707e-08 2.4630481189336084e-08 -> -0.9999998262417886 4.210501434612913e-08 2.4630481182686846e-08; origin xyz=0.007489008185044645 -0.11150041046657978 0.0004027858966975245 rpy=0.17453306234069357 -0.053747792579130614 -6.132332688812785e-07 -> xyz=0.007489008185044645 -0.11150041046657978 0.0004027858966975245 rpy=0.17453306234069352 -0.05374779257913059 -6.132332688804098e-07
- joint r_shoulder_yaw: axis -3.787621790513063e-08 2.805197706068352e-08 1.0000002566182309 -> -3.787621790776764e-08 2.805197706023475e-08 1.0000002566182309; origin xyz=0 4.2183273077367467e-07 -0.022499941373153573 rpy=0 0 0 -> xyz=0 4.2183273077367467e-07 -0.02249994137315358 rpy=0 0 0
- joint r_wrist_pitch: axis 0.9999998262417886 -4.2105014356162707e-08 -2.4630481189336084e-08 -> 0.9999998262417886 -4.210501434612913e-08 -2.4630481182686846e-08
- joint r_wrist_prosup: axis -3.787621790513063e-08 2.805197706068352e-08 1.0000002566182309 -> -3.787621790776764e-08 2.805197706023475e-08 1.0000002566182309; origin xyz=-0.014999869468812953 -0.001999649905318951 -0.05530006367251966 rpy=0 0 0 -> xyz=-0.014999869468812953 -0.0019996499053189787 -0.05530006367251966 rpy=0 0 0
- joint r_wrist_yaw: axis -2.4949582809984105e-07 1.0000002733514362 -2.7942487004772865e-08 -> -2.4949582807394525e-07 1.0000002733514362 -2.7942487010105877e-08; origin xyz=-0.016300122874272734 0.0069993900510918194 0 rpy=0 0 0 -> xyz=-0.016300122874272734 0.006999390051091792 0 rpy=0 0 0

File: iCub/robots/iCubGenova09/model.urdf (robot description, URDF)
Before this commit: robot iCub, 48 links, 47 joints
Links:
- link head: mass 1.94302 -> 1.93676
- link l_ankle_1: mass 1.80595 -> 0.366025
- link l_foot_front: mass 0.18507432 -> 0.185074
- link l_foot_rear: mass 0.18460842 -> 0.184608
- link l_lower_leg: mass 4.59072 -> 5.66584
- link l_upper_arm: mass 2.07167 -> 1.9475
- link r_ankle_1: mass 1.80595 -> 0.366025
- link r_ankle_2: mass 1.06976 -> 1.06609
- link r_foot_front: mass 0.184375 -> 0.185773
- link r_foot_rear: mass 0.18484137 -> 0.184841
- link r_hip_1: mass 2.48546 -> 2.50002
- link r_hip_2: mass 1.8834 -> 1.881
- link r_hip_3: mass 2.29352 -> 2.29213
- link r_lower_leg: mass 4.59072 -> 5.89871
- link r_upper_leg: mass 2.24396 -> 2.2571
Joints:
- joint l_arm_ft_sensor: origin xyz=-0.004350133156978329 3.632573233880443e-07 -0.05430003872406172 rpy=0 0 0 -> xyz=-0.004350133156978318 3.632573233602887e-07 -0.05430003872406172 rpy=0 0 0
- joint l_elbow: axis -8.811824154381087e-08 -1.0000002733514628 4.4047361189014644e-08 -> -8.811824174789715e-08 -1.0000002733514628 4.404736120498342e-08
- joint l_shoulder_pitch: axis 3.323079797673039e-07 0.9999999783534342 1.4452224303407313e-07 -> 3.323079797554136e-07 0.9999999783534342 1.4452224303420037e-07
- joint l_shoulder_roll: axis 0.9999998262417684 2.0348252649342313e-07 -4.0230228454118944e-08 -> 0.9999998262417685 2.0348252625938444e-07 -4.023022846062156e-08; origin xyz=0.004992849331690818 0.111499838456099 0.0002686502277366859 rpy=-0.17453296140985 -0.05374759931933852 0 -> xyz=0.004992849331690818 0.111499838456099 0.00026865022773668243 rpy=-0.17453296140985003 -0.05374759931933849 0
- joint l_shoulder_yaw: axis 2.227647404040578e-08 -4.393786245948661e-08 -1.0000002566182309 -> 2.2276474049102235e-08 -4.393786247302041e-08 -1.0000002566182309; origin xyz=0 -4.2345248449371375e-07 -0.02249994137312443 rpy=0 0 0 -> xyz=0 -4.2345248449371375e-07 -0.022499941373124423 rpy=0 0 0
- joint l_wrist_pitch: axis -0.9999998262417684 -2.0348252649342313e-07 4.0230228454118944e-08 -> -0.9999998262417685 -2.0348252625938444e-07 4.023022846062156e-08; origin xyz=0.016600015934286182 0.002006895218072541 -0.10749964114254112 rpy=0 0 0 -> xyz=0.016600015934286182 0.0020068952180725685 -0.10749964114254112 rpy=0 0 0
- joint l_wrist_prosup: axis 2.227647404040578e-08 -4.393786245948661e-08 -1.0000002566182309 -> 2.2276474049102235e-08 -4.393786247302041e-08 -1.0000002566182309; origin xyz=-0.014999870654177704 0.0019996435036348514 -0.055300063582479825 rpy=0 0 0 -> xyz=-0.0149998706541777 0.0019996435036348514 -0.0553000635824798 rpy=0 0 0
- joint l_wrist_yaw: axis 8.811824154381087e-08 1.0000002733514628 -4.4047361189014644e-08 -> 8.811824174789715e-08 1.0000002733514628 -4.404736120498342e-08; origin xyz=-0.016300121744729387 -0.0069993926815711816 0 rpy=0 0 0 -> xyz=-0.016300121744729387 -0.006999392681571209 0 rpy=0 0 0
- joint r_arm_ft_sensor: origin xyz=-0.006849946385389875 2.1904996055921444e-07 -0.05429998157789099 rpy=0 0 0 -> xyz=-0.006849946385389872 2.1904996058697002e-07 -0.05429998157789099 rpy=0 0 0
- joint r_elbow: axis 2.4949582809984105e-07 -1.0000002733514362 2.7942487004772865e-08 -> 2.4949582807394525e-07 -1.0000002733514362 2.7942487010105877e-08; origin xyz=0.009999931922603816 0.0014996401320274133 -0.1237003374895465 rpy=0 0 0 -> xyz=0.00999993192260382 0.0014996401320274133 -0.1237003374895465 rpy=0 0 0
- joint r_shoulder_pitch: axis 1.499044390054707e-07 0.9999999783534812 -1.2401537036188515e-07 -> 1.499044390098182e-07 0.9999999783534812 -1.2401537036323317e-07
- joint r_shoulder_roll: axis -0.9999998262417886 4.2105014356162707e-08 2.4630481189336084e-08 -> -0.9999998262417886 4.210501434612913e-08 2.4630481182686846e-08; origin xyz=0.007489008185044645 -0.11150041046657978 0.0004027858966975245 rpy=0.17453306234069357 -0.053747792579130614 -6.132332688812785e-07 -> xyz=0.007489008185044645 -0.11150041046657978 0.0004027858966975245 rpy=0.17453306234069352 -0.05374779257913059 -6.132332688804098e-07
- joint r_shoulder_yaw: axis -3.787621790513063e-08 2.805197706068352e-08 1.0000002566182309 -> -3.787621790776764e-08 2.805197706023475e-08 1.0000002566182309; origin xyz=0 4.2183273077367467e-07 -0.022499941373153573 rpy=0 0 0 -> xyz=0 4.2183273077367467e-07 -0.02249994137315358 rpy=0 0 0
- joint r_wrist_pitch: axis 0.9999998262417886 -4.2105014356162707e-08 -2.4630481189336084e-08 -> 0.9999998262417886 -4.210501434612913e-08 -2.4630481182686846e-08
- joint r_wrist_prosup: axis -3.787621790513063e-08 2.805197706068352e-08 1.0000002566182309 -> -3.787621790776764e-08 2.805197706023475e-08 1.0000002566182309; origin xyz=-0.014999869468812953 -0.001999649905318951 -0.05530006367251966 rpy=0 0 0 -> xyz=-0.014999869468812953 -0.0019996499053189787 -0.05530006367251966 rpy=0 0 0
- joint r_wrist_yaw: axis -2.4949582809984105e-07 1.0000002733514362 -2.7942487004772865e-08 -> -2.4949582807394525e-07 1.0000002733514362 -2.7942487010105877e-08; origin xyz=-0.016300122874272734 0.0069993900510918194 0 rpy=0 0 0 -> xyz=-0.016300122874272734 0.006999390051091792 0 rpy=0 0 0
