Commit message: Automatic build. GitHub Actions build: 1104573448 icub-model-generator commit: robotology/icub-models-generator@e0f80a0a419a19f25ed98e7ff28a5fe159039c06 urdf_parser_py commit: ros/urdf_parser_py@31474b9baaf7c3845b40e5a9aa87d5900a2282c3 simmechanics-to-urdf commit: robotology/simmechanics-to-urdf@1eb31b4e2d86e091c59cbe3cfc62d1e5265d7d61

File: iCub/robots/iCubGazeboV3/model.urdf (robot description, URDF)
Before this commit: robot iCub, 48 links, 47 joints
Links:
- link chest: mass 5.75757 -> 5.771074695
- link head: mass 1.93676 -> 1.831737118
- link l_ankle_1: mass 0.366025 -> 0.346176903
- link l_ankle_2: mass 1.06953 -> 1.011533592
- link l_elbow_1: mass 0.230254 -> 0.217768231
- link l_foot_front: mass 0.185074 -> 0.175038164
- link l_foot_rear: mass 0.184608 -> 0.174597434
- link l_forearm: mass 0.90793 -> 0.858696525
- link l_hand: mass 0.263541 -> 0.249250207
- link l_hip_1: mass 2.48546 -> 2.108461113
- link l_hip_2: mass 1.8834 -> 1.781270621
- link l_hip_3: mass 2.29352 -> 2.169151426
- link l_lower_leg: mass 5.66584 -> 5.063049414
- link l_shoulder_1: mass 1.45562 -> 1.376687449
- link l_shoulder_2: mass 0.322126 -> 0.304658373
- link l_shoulder_3: mass 0.256128 -> 0.242239185
- link l_upper_leg: mass 2.24396 -> 0.968264435
- link l_wrist_1: mass 0.0344005 -> 0.032535096
- link neck_1: mass 0.380603 -> 0.359964395
- link neck_2: mass 0.125549 -> 0.118740971
- link neck_3: mass 0.190133 -> 0.179822835
- link r_ankle_1: mass 0.366025 -> 0.346176903
- link r_ankle_2: mass 1.06609 -> 1.00828013
- link r_elbow_1: mass 0.397478 -> 0.217609341
- link r_foot_front: mass 0.185773 -> 0.17569926
- link r_foot_rear: mass 0.184841 -> 0.174817799
- link r_forearm: mass 0.903262 -> 0.854281652
- link r_hand: mass 0.264229 -> 0.2499009
- link r_hip_1: mass 2.50002 -> 2.134290199
- link r_hip_2: mass 1.881 -> 1.779000764
- link r_hip_3: mass 2.29213 -> 2.1678368
- link r_lower_leg: mass 5.89871 -> 5.074105512
- link r_shoulder_1: mass 1.45988 -> 1.380716446
- link r_shoulder_2: mass 0.322126 -> 0.304658373
- link r_shoulder_3: mass 0.258699 -> 0.24467077
- link r_upper_arm: mass 2.07285 -> 1.960447492
- link r_upper_leg: mass 2.2571 -> 0.980691904
- link r_wrist_1: mass 0.0344005 -> 0.032535096
- link root_link: mass 2.67135 -> 2.52649319
- link torso_1: mass 1.81255 -> 1.714262538
- link torso_2: mass 1.45349 -> 1.374672951
Joints:
- joint l_arm_ft_sensor: origin xyz=-0.004350133156978329 3.632573233880443e-07 -0.05430003872406172 rpy=0 0 0 -> xyz=-0.004350133156978318 3.632573233602887e-07 -0.05430003872406172 rpy=0 0 0
- joint l_elbow: axis -8.811824154381087e-08 -1.0000002733514628 4.4047361189014644e-08 -> -8.811824174789715e-08 -1.0000002733514628 4.404736120498342e-08
- joint l_shoulder_pitch: axis 3.323079797673039e-07 0.9999999783534342 1.4452224303407313e-07 -> 3.323079797554136e-07 0.9999999783534342 1.4452224303420037e-07
- joint l_shoulder_roll: axis 0.9999998262417684 2.0348252649342313e-07 -4.0230228454118944e-08 -> 0.9999998262417685 2.0348252625938444e-07 -4.023022846062156e-08; origin xyz=0.004992849331690818 0.111499838456099 0.0002686502277366859 rpy=-0.17453296140985 -0.05374759931933852 0 -> xyz=0.004992849331690818 0.111499838456099 0.00026865022773668243 rpy=-0.17453296140985003 -0.05374759931933849 0
- joint l_shoulder_yaw: axis 2.227647404040578e-08 -4.393786245948661e-08 -1.0000002566182309 -> 2.2276474049102235e-08 -4.393786247302041e-08 -1.0000002566182309; origin xyz=0 -4.2345248449371375e-07 -0.02249994137312443 rpy=0 0 0 -> xyz=0 -4.2345248449371375e-07 -0.022499941373124423 rpy=0 0 0
- joint l_wrist_pitch: axis -0.9999998262417684 -2.0348252649342313e-07 4.0230228454118944e-08 -> -0.9999998262417685 -2.0348252625938444e-07 4.023022846062156e-08; origin xyz=0.016600015934286182 0.002006895218072541 -0.10749964114254112 rpy=0 0 0 -> xyz=0.016600015934286182 0.0020068952180725685 -0.10749964114254112 rpy=0 0 0
- joint l_wrist_prosup: axis 2.227647404040578e-08 -4.393786245948661e-08 -1.0000002566182309 -> 2.2276474049102235e-08 -4.393786247302041e-08 -1.0000002566182309; origin xyz=-0.014999870654177704 0.0019996435036348514 -0.055300063582479825 rpy=0 0 0 -> xyz=-0.0149998706541777 0.0019996435036348514 -0.0553000635824798 rpy=0 0 0
- joint l_wrist_yaw: axis 8.811824154381087e-08 1.0000002733514628 -4.4047361189014644e-08 -> 8.811824174789715e-08 1.0000002733514628 -4.404736120498342e-08; origin xyz=-0.016300121744729387 -0.0069993926815711816 0 rpy=0 0 0 -> xyz=-0.016300121744729387 -0.006999392681571209 0 rpy=0 0 0
- joint r_arm_ft_sensor: origin xyz=-0.006849946385389875 2.1904996055921444e-07 -0.05429998157789099 rpy=0 0 0 -> xyz=-0.006849946385389872 2.1904996058697002e-07 -0.05429998157789099 rpy=0 0 0
- joint r_elbow: axis 2.4949582809984105e-07 -1.0000002733514362 2.7942487004772865e-08 -> 2.4949582807394525e-07 -1.0000002733514362 2.7942487010105877e-08; origin xyz=0.009999931922603816 0.0014996401320274133 -0.1237003374895465 rpy=0 0 0 -> xyz=0.00999993192260382 0.0014996401320274133 -0.1237003374895465 rpy=0 0 0
- joint r_shoulder_pitch: axis 1.499044390054707e-07 0.9999999783534812 -1.2401537036188515e-07 -> 1.499044390098182e-07 0.9999999783534812 -1.2401537036323317e-07
- joint r_shoulder_roll: axis -0.9999998262417886 4.2105014356162707e-08 2.4630481189336084e-08 -> -0.9999998262417886 4.210501434612913e-08 2.4630481182686846e-08; origin xyz=0.007489008185044645 -0.11150041046657978 0.0004027858966975245 rpy=0.17453306234069357 -0.053747792579130614 -6.132332688812785e-07 -> xyz=0.007489008185044645 -0.11150041046657978 0.0004027858966975245 rpy=0.17453306234069352 -0.05374779257913059 -6.132332688804098e-07
- joint r_shoulder_yaw: axis -3.787621790513063e-08 2.805197706068352e-08 1.0000002566182309 -> -3.787621790776764e-08 2.805197706023475e-08 1.0000002566182309; origin xyz=0 4.2183273077367467e-07 -0.022499941373153573 rpy=0 0 0 -> xyz=0 4.2183273077367467e-07 -0.02249994137315358 rpy=0 0 0
- joint r_wrist_pitch: axis 0.9999998262417886 -4.2105014356162707e-08 -2.4630481189336084e-08 -> 0.9999998262417886 -4.210501434612913e-08 -2.4630481182686846e-08
- joint r_wrist_prosup: axis -3.787621790513063e-08 2.805197706068352e-08 1.0000002566182309 -> -3.787621790776764e-08 2.805197706023475e-08 1.0000002566182309; origin xyz=-0.014999869468812953 -0.001999649905318951 -0.05530006367251966 rpy=0 0 0 -> xyz=-0.014999869468812953 -0.0019996499053189787 -0.05530006367251966 rpy=0 0 0
- joint r_wrist_yaw: axis -2.4949582809984105e-07 1.0000002733514362 -2.7942487004772865e-08 -> -2.4949582807394525e-07 1.0000002733514362 -2.7942487010105877e-08; origin xyz=-0.016300122874272734 0.0069993900510918194 0 rpy=0 0 0 -> xyz=-0.016300122874272734 0.006999390051091792 0 rpy=0 0 0

File: iCub/robots/iCubGenova09/model.urdf (robot description, URDF)
Before this commit: robot iCub, 48 links, 47 joints
Links:
- link chest: mass 5.75757 -> 5.771074695
- link head: mass 1.93676 -> 1.831737118
- link l_ankle_1: mass 0.366025 -> 0.346176903
- link l_ankle_2: mass 1.06953 -> 1.011533592
- link l_elbow_1: mass 0.230254 -> 0.217768231
- link l_foot_front: mass 0.185074 -> 0.175038164
- link l_foot_rear: mass 0.184608 -> 0.174597434
- link l_forearm: mass 0.90793 -> 0.858696525
- link l_hand: mass 0.263541 -> 0.249250207
- link l_hip_1: mass 2.48546 -> 2.108461113
- link l_hip_2: mass 1.8834 -> 1.781270621
- link l_hip_3: mass 2.29352 -> 2.169151426
- link l_lower_leg: mass 5.66584 -> 5.063049414
- link l_shoulder_1: mass 1.45562 -> 1.376687449
- link l_shoulder_2: mass 0.322126 -> 0.304658373
- link l_shoulder_3: mass 0.256128 -> 0.242239185
- link l_upper_arm: mass 2.08118 -> 1.968325789
- link l_upper_leg: mass 2.24396 -> 0.968264435
- link l_wrist_1: mass 0.0344005 -> 0.032535096
- link neck_1: mass 0.380603 -> 0.359964395
- link neck_2: mass 0.125549 -> 0.118740971
- link neck_3: mass 0.190133 -> 0.179822835
- link r_ankle_1: mass 0.366025 -> 0.346176903
- link r_ankle_2: mass 1.06609 -> 1.00828013
- link r_elbow_1: mass 0.397478 -> 0.217609341
- link r_foot_front: mass 0.185773 -> 0.17569926
- link r_foot_rear: mass 0.184841 -> 0.174817799
- link r_forearm: mass 0.903262 -> 0.854281652
- link r_hand: mass 0.264229 -> 0.2499009
- link r_hip_1: mass 2.50002 -> 2.134290199
- link r_hip_2: mass 1.881 -> 1.779000764
- link r_hip_3: mass 2.29213 -> 2.1678368
- link r_lower_leg: mass 5.89871 -> 5.074105512
- link r_shoulder_1: mass 1.45988 -> 1.380716446
- link r_shoulder_2: mass 0.322126 -> 0.304658373
- link r_shoulder_3: mass 0.258699 -> 0.24467077
- link r_upper_arm: mass 2.07285 -> 1.960447492
- link r_upper_leg: mass 2.2571 -> 0.980691904
- link r_wrist_1: mass 0.0344005 -> 0.032535096
- link root_link: mass 2.67135 -> 2.52649319
- link torso_1: mass 1.81255 -> 1.714262538
- link torso_2: mass 1.45349 -> 1.374672951
Joints:
- joint l_arm_ft_sensor: origin xyz=-0.004350133156978329 3.632573233880443e-07 -0.05430003872406172 rpy=0 0 0 -> xyz=-0.004350133156978318 3.632573233602887e-07 -0.05430003872406172 rpy=0 0 0
- joint l_elbow: axis -8.811824154381087e-08 -1.0000002733514628 4.4047361189014644e-08 -> -8.811824174789715e-08 -1.0000002733514628 4.404736120498342e-08
- joint l_shoulder_pitch: axis 3.323079797673039e-07 0.9999999783534342 1.4452224303407313e-07 -> 3.323079797554136e-07 0.9999999783534342 1.4452224303420037e-07
- joint l_shoulder_roll: axis 0.9999998262417684 2.0348252649342313e-07 -4.0230228454118944e-08 -> 0.9999998262417685 2.0348252625938444e-07 -4.023022846062156e-08; origin xyz=0.004992849331690818 0.111499838456099 0.0002686502277366859 rpy=-0.17453296140985 -0.05374759931933852 0 -> xyz=0.004992849331690818 0.111499838456099 0.00026865022773668243 rpy=-0.17453296140985003 -0.05374759931933849 0
- joint l_shoulder_yaw: axis 2.227647404040578e-08 -4.393786245948661e-08 -1.0000002566182309 -> 2.2276474049102235e-08 -4.393786247302041e-08 -1.0000002566182309; origin xyz=0 -4.2345248449371375e-07 -0.02249994137312443 rpy=0 0 0 -> xyz=0 -4.2345248449371375e-07 -0.022499941373124423 rpy=0 0 0
- joint l_wrist_pitch: axis -0.9999998262417684 -2.0348252649342313e-07 4.0230228454118944e-08 -> -0.9999998262417685 -2.0348252625938444e-07 4.023022846062156e-08; origin xyz=0.016600015934286182 0.002006895218072541 -0.10749964114254112 rpy=0 0 0 -> xyz=0.016600015934286182 0.0020068952180725685 -0.10749964114254112 rpy=0 0 0
- joint l_wrist_prosup: axis 2.227647404040578e-08 -4.393786245948661e-08 -1.0000002566182309 -> 2.2276474049102235e-08 -4.393786247302041e-08 -1.0000002566182309; origin xyz=-0.014999870654177704 0.0019996435036348514 -0.055300063582479825 rpy=0 0 0 -> xyz=-0.0149998706541777 0.0019996435036348514 -0.0553000635824798 rpy=0 0 0
- joint l_wrist_yaw: axis 8.811824154381087e-08 1.0000002733514628 -4.4047361189014644e-08 -> 8.811824174789715e-08 1.0000002733514628 -4.404736120498342e-08; origin xyz=-0.016300121744729387 -0.0069993926815711816 0 rpy=0 0 0 -> xyz=-0.016300121744729387 -0.006999392681571209 0 rpy=0 0 0
- joint r_arm_ft_sensor: origin xyz=-0.006849946385389875 2.1904996055921444e-07 -0.05429998157789099 rpy=0 0 0 -> xyz=-0.006849946385389872 2.1904996058697002e-07 -0.05429998157789099 rpy=0 0 0
- joint r_elbow: axis 2.4949582809984105e-07 -1.0000002733514362 2.7942487004772865e-08 -> 2.4949582807394525e-07 -1.0000002733514362 2.7942487010105877e-08; origin xyz=0.009999931922603816 0.0014996401320274133 -0.1237003374895465 rpy=0 0 0 -> xyz=0.00999993192260382 0.0014996401320274133 -0.1237003374895465 rpy=0 0 0
- joint r_shoulder_pitch: axis 1.499044390054707e-07 0.9999999783534812 -1.2401537036188515e-07 -> 1.499044390098182e-07 0.9999999783534812 -1.2401537036323317e-07
- joint r_shoulder_roll: axis -0.9999998262417886 4.2105014356162707e-08 2.4630481189336084e-08 -> -0.9999998262417886 4.210501434612913e-08 2.4630481182686846e-08; origin xyz=0.007489008185044645 -0.11150041046657978 0.0004027858966975245 rpy=0.17453306234069357 -0.053747792579130614 -6.132332688812785e-07 -> xyz=0.007489008185044645 -0.11150041046657978 0.0004027858966975245 rpy=0.17453306234069352 -0.05374779257913059 -6.132332688804098e-07
- joint r_shoulder_yaw: axis -3.787621790513063e-08 2.805197706068352e-08 1.0000002566182309 -> -3.787621790776764e-08 2.805197706023475e-08 1.0000002566182309; origin xyz=0 4.2183273077367467e-07 -0.022499941373153573 rpy=0 0 0 -> xyz=0 4.2183273077367467e-07 -0.02249994137315358 rpy=0 0 0
- joint r_wrist_pitch: axis 0.9999998262417886 -4.2105014356162707e-08 -2.4630481189336084e-08 -> 0.9999998262417886 -4.210501434612913e-08 -2.4630481182686846e-08
- joint r_wrist_prosup: axis -3.787621790513063e-08 2.805197706068352e-08 1.0000002566182309 -> -3.787621790776764e-08 2.805197706023475e-08 1.0000002566182309; origin xyz=-0.014999869468812953 -0.001999649905318951 -0.05530006367251966 rpy=0 0 0 -> xyz=-0.014999869468812953 -0.0019996499053189787 -0.05530006367251966 rpy=0 0 0
- joint r_wrist_yaw: axis -2.4949582809984105e-07 1.0000002733514362 -2.7942487004772865e-08 -> -2.4949582807394525e-07 1.0000002733514362 -2.7942487010105877e-08; origin xyz=-0.016300122874272734 0.0069993900510918194 0 rpy=0 0 0 -> xyz=-0.016300122874272734 0.006999390051091792 0 rpy=0 0 0

File: iCub/robots/left_hand_mk3/model.urdf (robot description, URDF)
Before this commit: robot SIM_LEFT_HAND, 12 links, 11 joints
Joints:
- joint l_hand_index_distal_joint: axis -1.2968763118959004e-08 -1.0000002970337007 0.0 -> -1.2968763121522752e-08 -1.0000002970337007 0.0
- joint l_hand_index_proximal_joint: axis -1.2968763118959004e-08 -1.0000002970337007 0.0 -> -1.2968763121522752e-08 -1.0000002970337007 0.0
- joint l_hand_pinky_distal_joint: axis -1.0351589968090255e-08 -0.9999999809599038 3.313676352756367e-08 -> -1.0351589974869193e-08 -0.9999999809599038 3.3136763531130714e-08
- joint l_hand_pinky_proximal_joint: axis -1.0351589968090255e-08 -0.9999999809599038 3.313676352756367e-08 -> -1.0351589974869193e-08 -0.9999999809599038 3.3136763531130714e-08
- joint l_hand_thumb_distal_joint: axis 2.628557915773655e-08 -1.0000002854169352 -2.1835508223766453e-07 -> 2.628557918787494e-08 -1.0000002854169352 -2.183550824779987e-07; origin xyz=0.020000016253208942 0 0.001499998093791144 rpy=0 0 0 -> xyz=0.020000016253208935 0 0.0014999980937911578 rpy=0 0 0
- joint l_hand_thumb_proximal_joint: axis 2.628557915773655e-08 -1.0000002854169352 -2.1835508223766453e-07 -> 2.628557918787494e-08 -1.0000002854169352 -2.183550824779987e-07
- joint l_hand_thumb_rotation_joint: axis 1.0000003237804127 -2.554693537271113e-07 6.571824259088421e-08 -> 1.000000323780413 -2.554693535849738e-07 6.571824263261195e-08; origin xyz=0.04079150000000001 -0.048141699999999996 -4.558000000000036e-05 rpy=-1.9198619241239645 0.17453290528623008 -1.4311699319115785 -> xyz=0.04079150000000001 -0.048141699999999996 -4.558000000000036e-05 rpy=-1.919861924123965 0.17453290528622997 -1.4311699319115785
