Commit message: Automatic build. GitHub Actions build: 7652322350 icub-model-generator commit: robotology/icub-models-generator@bbb2213ad5146e638e6674435acd9f872297a526 urdf_parser_py commit: ros/urdf_parser_py@31474b9baaf7c3845b40e5a9aa87d5900a2282c3 simmechanics-to-urdf commit: robotology/simmechanics-to-urdf@a72ed738acbd16b76f89e9cffbe41cf465f6afc6

File: iCub/robots/iCubGazeboV2_6/model.urdf (robot description, URDF)
Before this commit: robot iCub, 210 links, 209 joints
Joints:
- joint head_imu_0_fixed_joint: origin xyz=0.009500000190735 0.133444 0.009299999999999996 rpy=-1.5707963267948961 1.570796326794896 0 -> xyz=0.023453700190734995 0.20544400000000002 -0.023077900000000023 rpy=1.5707963267948997 0 0

File: iCub/robots/iCubGazeboV2_7/model.urdf (robot description, URDF)
Before this commit: robot iCub, 211 links, 210 joints
Joints:
- joint head_imu_0_fixed_joint: origin xyz=0.009500000190735 0.133444 0.009299999999999996 rpy=-1.5707963267948961 1.570796326794896 0 -> xyz=0.023453700190734995 0.20544400000000002 -0.023077900000000023 rpy=1.5707963267948997 0 0

File: iCub/robots/iCubGenova11/model.urdf (robot description, URDF)
Before this commit: robot iCub, 211 links, 210 joints
Joints:
- joint head_imu_0_fixed_joint: origin xyz=0.009500000190735 0.133444 0.009299999999999996 rpy=-1.5707963267948961 1.570796326794896 0 -> xyz=0.023453700190734995 0.20544400000000002 -0.023077900000000023 rpy=1.5707963267948997 0 0

Commit message: Automatic build. GitHub Actions build: 7798427068 icub-model-generator commit: robotology/icub-models-generator@9a939e2a9fee2ea98f7fc70cb3919800fb6ab4f8 urdf_parser_py commit: ros/urdf_parser_py@31474b9baaf7c3845b40e5a9aa87d5900a2282c3 simmechanics-to-urdf commit: robotology/simmechanics-to-urdf@a72ed738acbd16b76f89e9cffbe41cf465f6afc6

File: iCub/robots/iCubGazeboV2_6/model.urdf (robot description, URDF)
Before this commit: robot iCub, 210 links, 209 joints
Joints:
- joint head_imu_0_fixed_joint: origin xyz=0.023453700190734995 0.20544400000000002 -0.023077900000000023 rpy=1.5707963267948997 0 0 -> xyz=0.023453700190734995 0.20544400000000002 -0.023077900000000023 rpy=-1.5707963267948997 0 -3.141592653589793

File: iCub/robots/iCubGazeboV2_7/model.urdf (robot description, URDF)
Before this commit: robot iCub, 211 links, 210 joints
Joints:
- joint head_imu_0_fixed_joint: origin xyz=0.023453700190734995 0.20544400000000002 -0.023077900000000023 rpy=1.5707963267948997 0 0 -> xyz=0.023453700190734995 0.20544400000000002 -0.023077900000000023 rpy=-1.5707963267948997 0 -3.141592653589793

File: iCub/robots/iCubGenova11/model.urdf (robot description, URDF)
Before this commit: robot iCub, 211 links, 210 joints
Joints:
- joint head_imu_0_fixed_joint: origin xyz=0.023453700190734995 0.20544400000000002 -0.023077900000000023 rpy=1.5707963267948997 0 0 -> xyz=0.023453700190734995 0.20544400000000002 -0.023077900000000023 rpy=-1.5707963267948997 0 -3.141592653589793
