Commit message: Commit models generated by icub-model-generator

File: iCub/robots/iCubDarmstadt01/model.urdf (robot description, URDF)
Before this commit: robot ICUB_2-5_BB_SIM_MODEL, 163 links, 162 joints
Links:
- removed link imu_frame
- added link imu
- link chest: mass 7.638 -> 5.638; geometry collision mesh filename=model://iCubGenova02/meshes/dae/sim_sea_2-5_chest_bb_prt.dae scale=0.001 0.001 0.001; visual mesh filename=model://iCubGenova02/meshes/dae/sim_sea_2-5_chest_bb_prt.dae scale=0.001 0.001 0.001
- link head: geometry collision mesh filename=model://iCubGenova02/meshes/dae/sim_sea_2-5_head_prt.dae scale=0.001 0.001 0.001; visual mesh filename=model://iCubGenova02/meshes/dae/sim_sea_2-5_head_prt.dae scale=0.001 0.001 0.001
- link l_ankle_1: geometry collision mesh filename=model://iCubGenova02/meshes/dae/sim_sea_2-5_l_ankle_prt.dae scale=0.001 0.001 0.001; visual mesh filename=model://iCubGenova02/meshes/dae/sim_sea_2-5_l_ankle_prt.dae scale=0.001 0.001 0.001
- link l_ankle_2: geometry collision mesh filename=model://iCubGenova02/meshes/dae/sim_sea_2-5_l_foot_prt.dae scale=0.001 0.001 0.001; visual mesh filename=model://iCubGenova02/meshes/dae/sim_sea_2-5_l_foot_prt.dae scale=0.001 0.001 0.001
- link l_elbow_1: geometry collision mesh filename=model://iCubGenova02/meshes/dae/sim_sea_2-5_l_elbow_prosup_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 scale=0.001 0.001 0.001; visual mesh filename=model://iCubGenova02/meshes/dae/sim_sea_2-5_l_elbow_prosup_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 scale=0.001 0.001 0.001
- link l_foot: geometry collision mesh filename=model://iCubGenova02/meshes/dae/sim_sea_2-5_l_sole_prt.dae scale=0.001 0.001 0.001; visual mesh filename=model://iCubGenova02/meshes/dae/sim_sea_2-5_l_sole_prt.dae scale=0.001 0.001 0.001
- link l_forearm: geometry collision mesh filename=model://iCubGenova02/meshes/dae/sim_sea_2-5_l_forearm_prt.d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 scale=0.001 0.001 0.001; visual mesh filename=model://iCubGenova02/meshes/dae/sim_sea_2-5_l_forearm_prt.d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 scale=0.001 0.001 0.001
- link l_hand: geometry collision mesh filename=model://iCubGenova02/meshes/dae/sim_sea_2-5_l_hand_prt.dae scale=0.001 0.001 0.001; visual mesh filename=model://iCubGenova02/meshes/dae/sim_sea_2-5_l_hand_prt.dae scale=0.001 0.001 0.001
- link l_hip_1: geometry collision mesh filename=model://iCubGenova02/meshes/dae/sim_sea_2-5_l_hip_1_prt.dae scale=0.001 0.001 0.001; visual mesh filename=model://iCubGenova02/meshes/dae/sim_sea_2-5_l_hip_1_prt.dae scale=0.001 0.001 0.001
- link l_hip_2: geometry collision mesh filename=model://iCubGenova02/meshes/dae/sim_sea_2-5_l_hip_2_prt.dae scale=0.001 0.001 0.001; visual mesh filename=model://iCubGenova02/meshes/dae/sim_sea_2-5_l_hip_2_prt.dae scale=0.001 0.001 0.001
- link l_hip_3: geometry collision mesh filename=model://iCubGenova02/meshes/dae/sim_sea_2-5_l_upper_thigh_p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 scale=0.001 0.001 0.001; visual mesh filename=model://iCubGenova02/meshes/dae/sim_sea_2-5_l_upper_thigh_p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 scale=0.001 0.001 0.001
- link l_lower_leg: geometry collision mesh filename=model://iCubGenova02/meshes/dae/sim_sea_2-5_l_shank_prt.dae scale=0.001 0.001 0.001; visual mesh filename=model://iCubGenova02/meshes/dae/sim_sea_2-5_l_shank_prt.dae scale=0.001 0.001 0.001
- link l_shoulder_1: geometry collision mesh filename=model://iCubGenova02/meshes/dae/sim_sea_2-5_l_shoulder_1_pr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 scale=0.001 0.001 0.001; visual mesh filename=model://iCubGenova02/meshes/dae/sim_sea_2-5_l_shoulder_1_pr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 scale=0.001 0.001 0.001
- link l_shoulder_2: geometry collision mesh filename=model://iCubGenova02/meshes/dae/sim_sea_2-5_l_shoulder_2_pr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 scale=0.001 0.001 0.001; visual mesh filename=model://iCubGenova02/meshes/dae/sim_sea_2-5_l_shoulder_2_pr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 scale=0.001 0.001 0.001
- link l_shoulder_3: geometry collision mesh filename=model://iCubGenova02/meshes/dae/sim_sea_2-5_l_upper_arm_prt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 scale=0.001 0.001 0.001; visual mesh filename=model://iCubGenova02/meshes/dae/sim_sea_2-5_l_upper_arm_prt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 scale=0.001 0.001 0.001
- link l_upper_arm: geometry collision mesh filename=model://iCubGenova02/meshes/dae/sim_sea_2-5_l_elbow_prt.dae scale=0.001 0.001 0.001; visual mesh filename=model://iCubGenova02/meshes/dae/sim_sea_2-5_l_elbow_prt.dae scale=0.001 0.001 0.001
- link l_upper_leg: geometry collision mesh filename=model://iCubGenova02/meshes/dae/sim_sea_2-5_l_thigh_prt.dae scale=0.001 0.001 0.001; visual mesh filename=model://iCubGenova02/meshes/dae/sim_sea_2-5_l_thigh_prt.dae scale=0.001 0.001 0.001
- link l_wrist_1: geometry collision mesh filename=model://iCubGenova02/meshes/dae/sim_sea_2-5_l_wrist_pitch_p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 scale=0.001 0.001 0.001; visual mesh filename=model://iCubGenova02/meshes/dae/sim_sea_2-5_l_wrist_pitch_p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 scale=0.001 0.001 0.001
- link neck_1: geometry collision mesh filename=model://iCubGenova02/meshes/dae/sim_sea_2-5_neck_1_prt.dae scale=0.001 0.001 0.001; visual mesh filename=model://iCubGenova02/meshes/dae/sim_sea_2-5_neck_1_prt.dae scale=0.001 0.001 0.001
- link neck_2: geometry collision mesh filename=model://iCubGenova02/meshes/dae/sim_sea_2-5_neck_2_prt.dae scale=0.001 0.001 0.001; visual mesh filename=model://iCubGenova02/meshes/dae/sim_sea_2-5_neck_2_prt.dae scale=0.001 0.001 0.001
- link r_ankle_1: geometry collision mesh filename=model://iCubGenova02/meshes/dae/sim_sea_2-5_r_ankle_prt.dae scale=0.001 0.001 0.001; visual mesh filename=model://iCubGenova02/meshes/dae/sim_sea_2-5_r_ankle_prt.dae scale=0.001 0.001 0.001
- link r_ankle_2: geometry collision mesh filename=model://iCubGenova02/meshes/dae/sim_sea_2-5_r_foot_prt.dae scale=0.001 0.001 0.001; visual mesh filename=model://iCubGenova02/meshes/dae/sim_sea_2-5_r_foot_prt.dae scale=0.001 0.001 0.001
- link r_elbow_1: geometry collision mesh filename=model://iCubGenova02/meshes/dae/sim_sea_2-5_r_elbow_prosup_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 scale=0.001 0.001 0.001; visual mesh filename=model://iCubGenova02/meshes/dae/sim_sea_2-5_r_elbow_prosup_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 scale=0.001 0.001 0.001
- link r_foot: geometry collision mesh filename=model://iCubGenova02/meshes/dae/sim_sea_2-5_r_sole_prt.dae scale=0.001 0.001 0.001; visual mesh filename=model://iCubGenova02/meshes/dae/sim_sea_2-5_r_sole_prt.dae scale=0.001 0.001 0.001
- link r_forearm: geometry collision mesh filename=model://iCubGenova02/meshes/dae/sim_sea_2-5_r_forearm_prt.d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 scale=0.001 0.001 0.001; visual mesh filename=model://iCubGenova02/meshes/dae/sim_sea_2-5_r_forearm_prt.d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 scale=0.001 0.001 0.001
- link r_hand: geometry collision mesh filename=model://iCubGenova02/meshes/dae/sim_sea_2-5_r_hand_prt.dae scale=0.001 0.001 0.001; visual mesh filename=model://iCubGenova02/meshes/dae/sim_sea_2-5_r_hand_prt.dae scale=0.001 0.001 0.001
- link r_hip_1: geometry collision mesh filename=model://iCubGenova02/meshes/dae/sim_sea_2-5_r_hip_1_prt.dae scale=0.001 0.001 0.001; visual mesh filename=model://iCubGenova02/meshes/dae/sim_sea_2-5_r_hip_1_prt.dae scale=0.001 0.001 0.001
- link r_hip_2: geometry collision mesh filename=model://iCubGenova02/meshes/dae/sim_sea_2-5_r_hip_2_prt.dae scale=0.001 0.001 0.001; visual mesh filename=model://iCubGenova02/meshes/dae/sim_sea_2-5_r_hip_2_prt.dae scale=0.001 0.001 0.001
- link r_hip_3: geometry collision mesh filename=model://iCubGenova02/meshes/dae/sim_sea_2-5_r_upper_thigh_p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 scale=0.001 0.001 0.001; visual mesh filename=model://iCubGenova02/meshes/dae/sim_sea_2-5_r_upper_thigh_p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 scale=0.001 0.001 0.001
- link r_lower_leg: geometry collision mesh filename=model://iCubGenova02/meshes/dae/sim_sea_2-5_r_shank_prt.dae scale=0.001 0.001 0.001; visual mesh filename=model://iCubGenova02/meshes/dae/sim_sea_2-5_r_shank_prt.dae scale=0.001 0.001 0.001
- link r_shoulder_1: geometry collision mesh filename=model://iCubGenova02/meshes/dae/sim_sea_2-5_r_shoulder_1_pr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 scale=0.001 0.001 0.001; visual mesh filename=model://iCubGenova02/meshes/dae/sim_sea_2-5_r_shoulder_1_pr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 scale=0.001 0.001 0.001
- link r_shoulder_2: geometry collision mesh filename=model://iCubGenova02/meshes/dae/sim_sea_2-5_r_shoulder_2_pr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 scale=0.001 0.001 0.001; visual mesh filename=model://iCubGenova02/meshes/dae/sim_sea_2-5_r_shoulder_2_pr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 scale=0.001 0.001 0.001
- link r_shoulder_3: geometry collision mesh filename=model://iCubGenova02/meshes/dae/sim_sea_2-5_r_upper_arm_prt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 scale=0.001 0.001 0.001; visual mesh filename=model://iCubGenova02/meshes/dae/sim_sea_2-5_r_upper_arm_prt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 scale=0.001 0.001 0.001
- link r_upper_arm: geometry collision mesh filename=model://iCubGenova02/meshes/dae/sim_sea_2-5_r_elbow_prt.dae scale=0.001 0.001 0.001; visual mesh filename=model://iCubGenova02/meshes/dae/sim_sea_2-5_r_elbow_prt.dae scale=0.001 0.001 0.001
- link r_upper_leg: geometry collision mesh filename=model://iCubGenova02/meshes/dae/sim_sea_2-5_r_thigh_prt.dae scale=0.001 0.001 0.001; visual mesh filename=model://iCubGenova02/meshes/dae/sim_sea_2-5_r_thigh_prt.dae scale=0.001 0.001 0.001
- link r_wrist_1: geometry collision mesh filename=model://iCubGenova02/meshes/dae/sim_sea_2-5_r_wrist_pitch_p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 scale=0.001 0.001 0.001; visual mesh filename=model://iCubGenova02/meshes/dae/sim_sea_2-5_r_wrist_pitch_p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 scale=0.001 0.001 0.001
- link root_link: geometry collision mesh filename=model://iCubGenova02/meshes/dae/sim_sea_2-5_root_link_prt.d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 scale=0.001 0.001 0.001; visual mesh filename=model://iCubGenova02/meshes/dae/sim_sea_2-5_root_link_prt.d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 scale=0.001 0.001 0.001
- link torso_1: geometry collision mesh filename=model://iCubGenova02/meshes/dae/sim_sea_2-5_lap_belt_1_prt.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 scale=0.001 0.001 0.001; visual mesh filename=model://iCubGenova02/meshes/dae/sim_sea_2-5_lap_belt_1_prt.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 scale=0.001 0.001 0.001
- link torso_2: geometry collision mesh filename=model://iCubGenova02/meshes/dae/sim_sea_2-5_lap_belt_2_prt.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 scale=0.001 0.001 0.001; visual mesh filename=model://iCubGenova02/meshes/dae/sim_sea_2-5_lap_belt_2_prt.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 scale=0.001 0.001 0.001
Joints:
- removed joint imu_frame_fixed_joint
- added joint imu_fixed_joint: type fixed, parent head, child imu, origin xyz=0.00950000019074 0.133444 0.0093 rpy=-1.57079632679 1.57079632679 0
- joint r_wrist_prosup: axis 0.965925843882 -2.22044604925e-16 -0.258818979447 -> -0.965925843882 2.22044604925e-16 0.258818979447
