Commit message: Updated joint limits of SEA legs for the Simmechanics pipeline. See https://github.com/robotology-playground/icub-model-generator/commit/340b08e1c1ede1af2597ebac2e2024a86c9ef665

File: iCub/robots/iCubDarmstadt01/model.urdf (robot description, URDF)
Before this commit: robot iCub, 97 links, 96 joints
Joints:
- joint l_ankle_pitch: limit lower=-0.349065850399 upper=0.523598775598 effort=50000 velocity=50000 -> lower=-0.610865238198 upper=0.610865238198 effort=50000 velocity=50000
- joint l_ankle_roll: limit lower=-0.349065850399 upper=0.349065850399 effort=50000 velocity=50000 -> lower=-0.436332312999 upper=0.436332312999 effort=50000 velocity=50000
- joint l_hip_pitch: limit lower=-0.523598775598 upper=1.4835298642 effort=50000 velocity=50000 -> lower=-0.785398163397 upper=2.33874119767 effort=50000 velocity=50000
- joint l_hip_roll: limit lower=0.0 upper=1.57079632679 effort=50000 velocity=50000 -> lower=-0.349065850399 upper=2.09439510239 effort=50000 velocity=50000
- joint l_hip_yaw: limit lower=-1.2217304764 upper=1.2217304764 effort=50000 velocity=50000 -> lower=-1.3962634016 upper=1.3962634016 effort=50000 velocity=50000
- joint l_knee: limit lower=-1.74532925199 upper=0.0 effort=50000 velocity=50000 -> lower=-2.16420827247 upper=0.0698131700798 effort=50000 velocity=50000
- joint r_ankle_pitch: axis 1.0 0.0 0.0 -> -1.0 -0.0 -0.0; limit lower=-0.349065850399 upper=0.523598775598 effort=50000 velocity=50000 -> lower=-0.610865238198 upper=0.610865238198 effort=50000 velocity=50000; origin xyz=-0.0188325 -0.2005 0 rpy=0 0 0 -> xyz=-0.0268325 -0.2005 0 rpy=0 0 0
- joint r_ankle_roll: axis 0.0 0.0 -1.0 -> -0.0 -0.0 -1.0; limit lower=-0.349065850399 upper=0.349065850399 effort=50000 velocity=50000 -> lower=-0.436332312999 upper=0.436332312999 effort=50000 velocity=50000; origin xyz=0.0285 0 -0.0185 rpy=0 0 0 -> xyz=0.0365 0 -0.0185 rpy=0 0 0
- joint r_hip_pitch: axis -1.0 0.0 0.0 -> -1.0 -0.0 -0.0; limit lower=-0.523598775598 upper=1.4835298642 effort=50000 velocity=50000 -> lower=-0.785398163397 upper=2.33874119767 effort=50000 velocity=50000
- joint r_hip_roll: axis 0.0 0.0 -1.0 -> -0.0 -0.0 -1.0; limit lower=0.0 upper=1.57079632679 effort=50000 velocity=50000 -> lower=-0.349065850399 upper=2.09439510239 effort=50000 velocity=50000
- joint r_hip_yaw: limit lower=-1.2217304764 upper=1.2217304764 effort=50000 velocity=50000 -> lower=-1.3962634016 upper=1.3962634016 effort=50000 velocity=50000
- joint r_knee: axis -1.0 0.0 0.0 -> -1.0 -0.0 -0.0; limit lower=-1.74532925199 upper=0.0 effort=50000 velocity=50000 -> lower=-2.16420827247 upper=0.0698131700798 effort=50000 velocity=50000

File: iCub/robots/iCubGenova02/model.urdf (robot description, URDF)
Before this commit: robot iCub, 97 links, 96 joints
Links:
- added link r_lower_leg_skin_0
- added link r_lower_leg_skin_10
- added link r_lower_leg_skin_11
- added link r_lower_leg_skin_14
- added link r_lower_leg_skin_15
- added link r_lower_leg_skin_16
- added link r_lower_leg_skin_17
- added link r_lower_leg_skin_19
- added link r_lower_leg_skin_20
- added link r_lower_leg_skin_21
- added link r_lower_leg_skin_28
- added link r_lower_leg_skin_29
- added link r_lower_leg_skin_3
- added link r_lower_leg_skin_31
- added link r_lower_leg_skin_32
- added link r_lower_leg_skin_35
- added link r_lower_leg_skin_36
- added link r_lower_leg_skin_37
- added link r_lower_leg_skin_38
- added link r_lower_leg_skin_4
- added link r_lower_leg_skin_41
- added link r_lower_leg_skin_42
- added link r_lower_leg_skin_43
- added link r_lower_leg_skin_46
- added link r_lower_leg_skin_47
- added link r_lower_leg_skin_49
- added link r_lower_leg_skin_5
- added link r_lower_leg_skin_50
- added link r_lower_leg_skin_51
- added link r_lower_leg_skin_52
- added link r_lower_leg_skin_53
- added link r_lower_leg_skin_54
- added link r_lower_leg_skin_55
- added link r_lower_leg_skin_56
- added link r_lower_leg_skin_6
- added link r_lower_leg_skin_60
- added link r_lower_leg_skin_61
- added link r_lower_leg_skin_9
Joints:
- added joint r_lower_leg_skin_0_fixed_joint: type fixed, parent r_lower_leg, child r_lower_leg_skin_0, origin xyz=-0.0215465 -0.002634 0.0544117 rpy=-0.660978905975 0.123114980697 1.4755829697
- added joint r_lower_leg_skin_10_fixed_joint: type fixed, parent r_lower_leg, child r_lower_leg_skin_10, origin xyz=0.0100099 -0.021205 0.0644607 rpy=0.000432173736511 -0.0998382821227 1.57075325095
- added joint r_lower_leg_skin_11_fixed_joint: type fixed, parent r_lower_leg, child r_lower_leg_skin_11, origin xyz=-0.0064241 -0.030885 0.0607108 rpy=-0.279936053974 -0.233577889652 1.63723971694
- added joint r_lower_leg_skin_14_fixed_joint: type fixed, parent r_lower_leg, child r_lower_leg_skin_14, origin xyz=-0.0215085 -0.0219 0.0550477 rpy=-0.65674037676 -0.0838840185901 1.6352968064
- added joint r_lower_leg_skin_15_fixed_joint: type fixed, parent r_lower_leg, child r_lower_leg_skin_15, origin xyz=-0.0065113 0.007243 0.0591708 rpy=-0.287349971655 0.306509038255 1.48186077381
- added joint r_lower_leg_skin_16_fixed_joint: type fixed, parent r_lower_leg, child r_lower_leg_skin_16, origin xyz=-0.0406195 -0.004549 0.0272875 rpy=-1.17903435098 0.0145863542197 1.53550278559
- added joint r_lower_leg_skin_17_fixed_joint: type fixed, parent r_lower_leg, child r_lower_leg_skin_17, origin xyz=-0.0406445 -0.023882 0.027875 rpy=-1.18020591847 -0.0027159844464 1.57739302393
- added joint r_lower_leg_skin_19_fixed_joint: type fixed, parent r_lower_leg, child r_lower_leg_skin_19, origin xyz=0.0507303 0.006065 0.0357534 rpy=0.987216858918 0.0751545057171 1.68402242082
- added joint r_lower_leg_skin_20_fixed_joint: type fixed, parent r_lower_leg, child r_lower_leg_skin_20, origin xyz=0.0576583 -0.004952 0.0234419 rpy=1.27473610115 0.0206410616106 1.6383594359
- added joint r_lower_leg_skin_21_fixed_joint: type fixed, parent r_lower_leg, child r_lower_leg_skin_21, origin xyz=0.0582053 -0.024277 0.0242704 rpy=1.26752944172 0.00458214989839 1.58543727798
- added joint r_lower_leg_skin_28_fixed_joint: type fixed, parent r_lower_leg, child r_lower_leg_skin_28, origin xyz=-0.0327725 -0.032756 0.04087215 rpy=-0.930251372093 -0.0288636035903 1.60949343025
- added joint r_lower_leg_skin_29_fixed_joint: type fixed, parent r_lower_leg, child r_lower_leg_skin_29, origin xyz=-0.0338485 -0.05242 0.03846637 rpy=-0.915770698544 -0.0222403533337 1.59973768678
- added joint r_lower_leg_skin_31_fixed_joint: type fixed, parent r_lower_leg, child r_lower_leg_skin_31, origin xyz=-0.0326035 0.006327 0.03914638 rpy=-0.938611596431 0.0903584824077 1.44821993266
- added joint r_lower_leg_skin_32_fixed_joint: type fixed, parent r_lower_leg, child r_lower_leg_skin_32, origin xyz=0.0422522 -0.080733 0.04598301 rpy=0.64650651578 -0.0386542965682 1.54163935643
- added joint r_lower_leg_skin_35_fixed_joint: type fixed, parent r_lower_leg, child r_lower_leg_skin_35, origin xyz=-0.0215645 -0.080113 0.04774866 rpy=-0.542152349621 -0.0455923960272 1.59824328594
- added joint r_lower_leg_skin_36_fixed_joint: type fixed, parent r_lower_leg, child r_lower_leg_skin_36, origin xyz=-0.0059343 -0.088362 0.05322409 rpy=-0.207709325297 -0.0537454077707 1.58211730453
- added joint r_lower_leg_skin_37_fixed_joint: type fixed, parent r_lower_leg, child r_lower_leg_skin_37, origin xyz=0.0106319 -0.078318 0.0552572 rpy=0.00754389164192 -0.0476116089222 1.57043779524
- added joint r_lower_leg_skin_38_fixed_joint: type fixed, parent r_lower_leg, child r_lower_leg_skin_38, origin xyz=-0.0215955 -0.060757 0.04880467 rpy=-0.542830301827 -0.0471634712563 1.59923066943
- added joint r_lower_leg_skin_3_fixed_joint: type fixed, parent r_lower_leg, child r_lower_leg_skin_3, origin xyz=0.040088 -0.002843 0.05157878 rpy=0.842654955784 0.0943728500099 1.67609780358
- added joint r_lower_leg_skin_41_fixed_joint: type fixed, parent r_lower_leg, child r_lower_leg_skin_41, origin xyz=-0.0062454 -0.049854 0.0566009 rpy=-0.251468147514 -0.158913056373 1.61142822718
- added joint r_lower_leg_skin_42_fixed_joint: type fixed, parent r_lower_leg, child r_lower_leg_skin_42, origin xyz=0.0104637 -0.05908 0.0570106 rpy=0.00694017036085 -0.135545595322 1.56985808158
- added joint r_lower_leg_skin_43_fixed_joint: type fixed, parent r_lower_leg, child r_lower_leg_skin_43, origin xyz=0.0420328 -0.061362 0.04712542 rpy=0.624467273745 -0.026260830452 1.55187529497
- added joint r_lower_leg_skin_46_fixed_joint: type fixed, parent r_lower_leg, child r_lower_leg_skin_46, origin xyz=0.0268839 -0.05018 0.0558156 rpy=0.328741310202 -0.135625619972 1.52470662181
- added joint r_lower_leg_skin_47_fixed_joint: type fixed, parent r_lower_leg, child r_lower_leg_skin_47, origin xyz=0.0273064 -0.08886 0.05264163 rpy=0.263001895535 -0.0520410015187 1.55679195888
- added joint r_lower_leg_skin_49_fixed_joint: type fixed, parent r_lower_leg, child r_lower_leg_skin_49, origin xyz=0.042106 -0.138859 0.04113137 rpy=0.731392432649 -0.0602196903016 1.51683891676
- added joint r_lower_leg_skin_4_fixed_joint: type fixed, parent r_lower_leg, child r_lower_leg_skin_4, origin xyz=0.0264511 0.007272 0.0583103 rpy=0.40039718175 0.29099345069 1.69164016714
- added joint r_lower_leg_skin_50_fixed_joint: type fixed, parent r_lower_leg, child r_lower_leg_skin_50, origin xyz=0.0421948 -0.119469 0.043016947 rpy=0.69705122002 -0.055082279609 1.52473387321
- added joint r_lower_leg_skin_51_fixed_joint: type fixed, parent r_lower_leg, child r_lower_leg_skin_51, origin xyz=0.0274265 -0.108206 0.05141583 rpy=0.272623174864 -0.0621353313747 1.55343743538
- added joint r_lower_leg_skin_52_fixed_joint: type fixed, parent r_lower_leg, child r_lower_leg_skin_52, origin xyz=0.0109339 -0.116895 0.05299832 rpy=0.0108976323462 -0.0676055809873 1.57006018656
- added joint r_lower_leg_skin_53_fixed_joint: type fixed, parent r_lower_leg, child r_lower_leg_skin_53, origin xyz=-0.0057664 -0.107654 0.05207312 rpy=-0.211841375505 -0.063397660111 1.58442104098
- added joint r_lower_leg_skin_54_fixed_joint: type fixed, parent r_lower_leg, child r_lower_leg_skin_54, origin xyz=-0.0210815 -0.118787 0.04512708 rpy=-0.576349226046 -0.0615294995172 1.61074135295
- added joint r_lower_leg_skin_55_fixed_joint: type fixed, parent r_lower_leg, child r_lower_leg_skin_55, origin xyz=-0.0208215 -0.138143 0.043502663 rpy=-0.598745472791 -0.0668224323993 1.61632329625
- added joint r_lower_leg_skin_56_fixed_joint: type fixed, parent r_lower_leg, child r_lower_leg_skin_56, origin xyz=-0.0054535 -0.146218 0.04926839 rpy=-0.224166511744 -0.0775658268571 1.58846192551
- added joint r_lower_leg_skin_5_fixed_joint: type fixed, parent r_lower_leg, child r_lower_leg_skin_5, origin xyz=0.0099769 -0.001972 0.0636503 rpy=0.000123038724669 0.184274174748 1.57081887154
- added joint r_lower_leg_skin_60_fixed_joint: type fixed, parent r_lower_leg, child r_lower_leg_skin_60, origin xyz=0.0277235 -0.146938 0.04836967 rpy=0.303887741163 -0.0772432614252 1.54660163218
- added joint r_lower_leg_skin_61_fixed_joint: type fixed, parent r_lower_leg, child r_lower_leg_skin_61, origin xyz=0.0110941 -0.136169 0.05161952 rpy=0.0132400606487 -0.0747688280205 1.56980737046
- added joint r_lower_leg_skin_6_fixed_joint: type fixed, parent r_lower_leg, child r_lower_leg_skin_6, origin xyz=0.0401109 -0.022149 0.05208552 rpy=0.840135245525 -0.0688367062203 1.49419034934
- added joint r_lower_leg_skin_9_fixed_joint: type fixed, parent r_lower_leg, child r_lower_leg_skin_9, origin xyz=0.0264648 -0.030962 0.0598214 rpy=0.388444125907 -0.212046974802 1.48487982461
- joint l_ankle_pitch: limit lower=-0.349065850399 upper=0.523598775598 effort=50000 velocity=50000 -> lower=-0.610865238198 upper=0.610865238198 effort=50000 velocity=50000
- joint l_ankle_roll: limit lower=-0.349065850399 upper=0.349065850399 effort=50000 velocity=50000 -> lower=-0.436332312999 upper=0.436332312999 effort=50000 velocity=50000
- joint l_hip_pitch: limit lower=-0.523598775598 upper=1.4835298642 effort=50000 velocity=50000 -> lower=-0.785398163397 upper=2.33874119767 effort=50000 velocity=50000
- joint l_hip_roll: limit lower=0.0 upper=1.57079632679 effort=50000 velocity=50000 -> lower=-0.349065850399 upper=2.09439510239 effort=50000 velocity=50000
- joint l_hip_yaw: limit lower=-1.2217304764 upper=1.2217304764 effort=50000 velocity=50000 -> lower=-1.3962634016 upper=1.3962634016 effort=50000 velocity=50000
- joint l_knee: limit lower=-1.74532925199 upper=0.0 effort=50000 velocity=50000 -> lower=-2.16420827247 upper=0.0698131700798 effort=50000 velocity=50000
- joint r_ankle_pitch: axis 1.0 0.0 0.0 -> -1.0 -0.0 -0.0; limit lower=-0.349065850399 upper=0.523598775598 effort=50000 velocity=50000 -> lower=-0.610865238198 upper=0.610865238198 effort=50000 velocity=50000; origin xyz=-0.0188325 -0.2005 0 rpy=0 0 0 -> xyz=-0.0268325 -0.2005 0 rpy=0 0 0
- joint r_ankle_roll: axis 0.0 0.0 -1.0 -> -0.0 -0.0 -1.0; limit lower=-0.349065850399 upper=0.349065850399 effort=50000 velocity=50000 -> lower=-0.436332312999 upper=0.436332312999 effort=50000 velocity=50000; origin xyz=0.0285 0 -0.0185 rpy=0 0 0 -> xyz=0.0365 0 -0.0185 rpy=0 0 0
- joint r_hip_pitch: axis -1.0 0.0 0.0 -> -1.0 -0.0 -0.0; limit lower=-0.523598775598 upper=1.4835298642 effort=50000 velocity=50000 -> lower=-0.785398163397 upper=2.33874119767 effort=50000 velocity=50000
- joint r_hip_roll: axis 0.0 0.0 -1.0 -> -0.0 -0.0 -1.0; limit lower=0.0 upper=1.57079632679 effort=50000 velocity=50000 -> lower=-0.349065850399 upper=2.09439510239 effort=50000 velocity=50000
- joint r_hip_yaw: limit lower=-1.2217304764 upper=1.2217304764 effort=50000 velocity=50000 -> lower=-1.3962634016 upper=1.3962634016 effort=50000 velocity=50000
- joint r_knee: axis -1.0 0.0 0.0 -> -1.0 -0.0 -0.0; limit lower=-1.74532925199 upper=0.0 effort=50000 velocity=50000 -> lower=-2.16420827247 upper=0.0698131700798 effort=50000 velocity=50000

Commit message: Updating models with correct r_ankle_pitch joint axis and added skin frames to the NO_BACKPACK

File: iCub/robots/iCubDarmstadt01/model.urdf (robot description, URDF)
Before this commit: robot iCub, 97 links, 96 joints
Links:
- added link r_lower_leg_skin_0
- added link r_lower_leg_skin_10
- added link r_lower_leg_skin_11
- added link r_lower_leg_skin_14
- added link r_lower_leg_skin_15
- added link r_lower_leg_skin_16
- added link r_lower_leg_skin_17
- added link r_lower_leg_skin_19
- added link r_lower_leg_skin_20
- added link r_lower_leg_skin_21
- added link r_lower_leg_skin_28
- added link r_lower_leg_skin_29
- added link r_lower_leg_skin_3
- added link r_lower_leg_skin_31
- added link r_lower_leg_skin_32
- added link r_lower_leg_skin_35
- added link r_lower_leg_skin_36
- added link r_lower_leg_skin_37
- added link r_lower_leg_skin_38
- added link r_lower_leg_skin_4
- added link r_lower_leg_skin_41
- added link r_lower_leg_skin_42
- added link r_lower_leg_skin_43
- added link r_lower_leg_skin_46
- added link r_lower_leg_skin_47
- added link r_lower_leg_skin_49
- added link r_lower_leg_skin_5
- added link r_lower_leg_skin_50
- added link r_lower_leg_skin_51
- added link r_lower_leg_skin_52
- added link r_lower_leg_skin_53
- added link r_lower_leg_skin_54
- added link r_lower_leg_skin_55
- added link r_lower_leg_skin_56
- added link r_lower_leg_skin_6
- added link r_lower_leg_skin_60
- added link r_lower_leg_skin_61
- added link r_lower_leg_skin_9
Joints:
- added joint r_lower_leg_skin_0_fixed_joint: type fixed, parent r_lower_leg, child r_lower_leg_skin_0, origin xyz=-0.0215465 -0.002634 0.0544117 rpy=-0.660978905975 0.123114980697 1.4755829697
- added joint r_lower_leg_skin_10_fixed_joint: type fixed, parent r_lower_leg, child r_lower_leg_skin_10, origin xyz=0.0100099 -0.021205 0.0644607 rpy=0.000432173736511 -0.0998382821227 1.57075325095
- added joint r_lower_leg_skin_11_fixed_joint: type fixed, parent r_lower_leg, child r_lower_leg_skin_11, origin xyz=-0.0064241 -0.030885 0.0607108 rpy=-0.279936053974 -0.233577889652 1.63723971694
- added joint r_lower_leg_skin_14_fixed_joint: type fixed, parent r_lower_leg, child r_lower_leg_skin_14, origin xyz=-0.0215085 -0.0219 0.0550477 rpy=-0.65674037676 -0.0838840185901 1.6352968064
- added joint r_lower_leg_skin_15_fixed_joint: type fixed, parent r_lower_leg, child r_lower_leg_skin_15, origin xyz=-0.0065113 0.007243 0.0591708 rpy=-0.287349971655 0.306509038255 1.48186077381
- added joint r_lower_leg_skin_16_fixed_joint: type fixed, parent r_lower_leg, child r_lower_leg_skin_16, origin xyz=-0.0406195 -0.004549 0.0272875 rpy=-1.17903435098 0.0145863542197 1.53550278559
- added joint r_lower_leg_skin_17_fixed_joint: type fixed, parent r_lower_leg, child r_lower_leg_skin_17, origin xyz=-0.0406445 -0.023882 0.027875 rpy=-1.18020591847 -0.0027159844464 1.57739302393
- added joint r_lower_leg_skin_19_fixed_joint: type fixed, parent r_lower_leg, child r_lower_leg_skin_19, origin xyz=0.0507303 0.006065 0.0357534 rpy=0.987216858918 0.0751545057171 1.68402242082
- added joint r_lower_leg_skin_20_fixed_joint: type fixed, parent r_lower_leg, child r_lower_leg_skin_20, origin xyz=0.0576583 -0.004952 0.0234419 rpy=1.27473610115 0.0206410616106 1.6383594359
- added joint r_lower_leg_skin_21_fixed_joint: type fixed, parent r_lower_leg, child r_lower_leg_skin_21, origin xyz=0.0582053 -0.024277 0.0242704 rpy=1.26752944172 0.00458214989839 1.58543727798
- added joint r_lower_leg_skin_28_fixed_joint: type fixed, parent r_lower_leg, child r_lower_leg_skin_28, origin xyz=-0.0327725 -0.032756 0.04087215 rpy=-0.930251372093 -0.0288636035903 1.60949343025
- added joint r_lower_leg_skin_29_fixed_joint: type fixed, parent r_lower_leg, child r_lower_leg_skin_29, origin xyz=-0.0338485 -0.05242 0.03846637 rpy=-0.915770698544 -0.0222403533337 1.59973768678
- added joint r_lower_leg_skin_31_fixed_joint: type fixed, parent r_lower_leg, child r_lower_leg_skin_31, origin xyz=-0.0326035 0.006327 0.03914638 rpy=-0.938611596431 0.0903584824077 1.44821993266
- added joint r_lower_leg_skin_32_fixed_joint: type fixed, parent r_lower_leg, child r_lower_leg_skin_32, origin xyz=0.0422522 -0.080733 0.04598301 rpy=0.64650651578 -0.0386542965682 1.54163935643
- added joint r_lower_leg_skin_35_fixed_joint: type fixed, parent r_lower_leg, child r_lower_leg_skin_35, origin xyz=-0.0215645 -0.080113 0.04774866 rpy=-0.542152349621 -0.0455923960272 1.59824328594
- added joint r_lower_leg_skin_36_fixed_joint: type fixed, parent r_lower_leg, child r_lower_leg_skin_36, origin xyz=-0.0059343 -0.088362 0.05322409 rpy=-0.207709325297 -0.0537454077707 1.58211730453
- added joint r_lower_leg_skin_37_fixed_joint: type fixed, parent r_lower_leg, child r_lower_leg_skin_37, origin xyz=0.0106319 -0.078318 0.0552572 rpy=0.00754389164192 -0.0476116089222 1.57043779524
- added joint r_lower_leg_skin_38_fixed_joint: type fixed, parent r_lower_leg, child r_lower_leg_skin_38, origin xyz=-0.0215955 -0.060757 0.04880467 rpy=-0.542830301827 -0.0471634712563 1.59923066943
- added joint r_lower_leg_skin_3_fixed_joint: type fixed, parent r_lower_leg, child r_lower_leg_skin_3, origin xyz=0.040088 -0.002843 0.05157878 rpy=0.842654955784 0.0943728500099 1.67609780358
- added joint r_lower_leg_skin_41_fixed_joint: type fixed, parent r_lower_leg, child r_lower_leg_skin_41, origin xyz=-0.0062454 -0.049854 0.0566009 rpy=-0.251468147514 -0.158913056373 1.61142822718
- added joint r_lower_leg_skin_42_fixed_joint: type fixed, parent r_lower_leg, child r_lower_leg_skin_42, origin xyz=0.0104637 -0.05908 0.0570106 rpy=0.00694017036085 -0.135545595322 1.56985808158
- added joint r_lower_leg_skin_43_fixed_joint: type fixed, parent r_lower_leg, child r_lower_leg_skin_43, origin xyz=0.0420328 -0.061362 0.04712542 rpy=0.624467273745 -0.026260830452 1.55187529497
- added joint r_lower_leg_skin_46_fixed_joint: type fixed, parent r_lower_leg, child r_lower_leg_skin_46, origin xyz=0.0268839 -0.05018 0.0558156 rpy=0.328741310202 -0.135625619972 1.52470662181
- added joint r_lower_leg_skin_47_fixed_joint: type fixed, parent r_lower_leg, child r_lower_leg_skin_47, origin xyz=0.0273064 -0.08886 0.05264163 rpy=0.263001895535 -0.0520410015187 1.55679195888
- added joint r_lower_leg_skin_49_fixed_joint: type fixed, parent r_lower_leg, child r_lower_leg_skin_49, origin xyz=0.042106 -0.138859 0.04113137 rpy=0.731392432649 -0.0602196903016 1.51683891676
- added joint r_lower_leg_skin_4_fixed_joint: type fixed, parent r_lower_leg, child r_lower_leg_skin_4, origin xyz=0.0264511 0.007272 0.0583103 rpy=0.40039718175 0.29099345069 1.69164016714
- added joint r_lower_leg_skin_50_fixed_joint: type fixed, parent r_lower_leg, child r_lower_leg_skin_50, origin xyz=0.0421948 -0.119469 0.043016947 rpy=0.69705122002 -0.055082279609 1.52473387321
- added joint r_lower_leg_skin_51_fixed_joint: type fixed, parent r_lower_leg, child r_lower_leg_skin_51, origin xyz=0.0274265 -0.108206 0.05141583 rpy=0.272623174864 -0.0621353313747 1.55343743538
- added joint r_lower_leg_skin_52_fixed_joint: type fixed, parent r_lower_leg, child r_lower_leg_skin_52, origin xyz=0.0109339 -0.116895 0.05299832 rpy=0.0108976323462 -0.0676055809873 1.57006018656
- added joint r_lower_leg_skin_53_fixed_joint: type fixed, parent r_lower_leg, child r_lower_leg_skin_53, origin xyz=-0.0057664 -0.107654 0.05207312 rpy=-0.211841375505 -0.063397660111 1.58442104098
- added joint r_lower_leg_skin_54_fixed_joint: type fixed, parent r_lower_leg, child r_lower_leg_skin_54, origin xyz=-0.0210815 -0.118787 0.04512708 rpy=-0.576349226046 -0.0615294995172 1.61074135295
- added joint r_lower_leg_skin_55_fixed_joint: type fixed, parent r_lower_leg, child r_lower_leg_skin_55, origin xyz=-0.0208215 -0.138143 0.043502663 rpy=-0.598745472791 -0.0668224323993 1.61632329625
- added joint r_lower_leg_skin_56_fixed_joint: type fixed, parent r_lower_leg, child r_lower_leg_skin_56, origin xyz=-0.0054535 -0.146218 0.04926839 rpy=-0.224166511744 -0.0775658268571 1.58846192551
- added joint r_lower_leg_skin_5_fixed_joint: type fixed, parent r_lower_leg, child r_lower_leg_skin_5, origin xyz=0.0099769 -0.001972 0.0636503 rpy=0.000123038724669 0.184274174748 1.57081887154
- added joint r_lower_leg_skin_60_fixed_joint: type fixed, parent r_lower_leg, child r_lower_leg_skin_60, origin xyz=0.0277235 -0.146938 0.04836967 rpy=0.303887741163 -0.0772432614252 1.54660163218
- added joint r_lower_leg_skin_61_fixed_joint: type fixed, parent r_lower_leg, child r_lower_leg_skin_61, origin xyz=0.0110941 -0.136169 0.05161952 rpy=0.0132400606487 -0.0747688280205 1.56980737046
- added joint r_lower_leg_skin_6_fixed_joint: type fixed, parent r_lower_leg, child r_lower_leg_skin_6, origin xyz=0.0401109 -0.022149 0.05208552 rpy=0.840135245525 -0.0688367062203 1.49419034934
- added joint r_lower_leg_skin_9_fixed_joint: type fixed, parent r_lower_leg, child r_lower_leg_skin_9, origin xyz=0.0264648 -0.030962 0.0598214 rpy=0.388444125907 -0.212046974802 1.48487982461
- joint r_ankle_pitch: axis -1.0 -0.0 -0.0 -> 1.0 0.0 0.0

File: iCub/robots/iCubGenova02/model.urdf (robot description, URDF)
Before this commit: robot iCub, 135 links, 134 joints
Joints:
- joint r_ankle_pitch: axis -1.0 -0.0 -0.0 -> 1.0 0.0 0.0
