Commit message: Travis build:134
icub-model-generator commit:97827f894a2572b10697a5a33639b530690151b0

urdf_parser_py commit:31474b9baaf7c3845b40e5a9aa87d5900a2282c3

simmechanics-to-urdf commit:eaf70e8e76b2870efa0c53ae09555c9612a689a9

codyco-superbuild commit:570a6dd3cf3218daaf3d32ba16845ebc8989f3b2

File: iCub/robots/iCubGenova02/model.urdf (robot description, URDF)
Before this commit: robot iCub, 135 links, 134 joints
Links:
- added link l_upper_leg_back_contact
- added link l_upper_leg_dh_frame
- added link r_upper_leg_back_contact
- added link r_upper_leg_dh_frame
- link l_foot: mass 0.382372 -> 0.382968
- link l_hip_1: mass 0.915608 -> 0.919725
- link l_hip_2: mass 0.421161 -> 0.421106
- link r_foot: mass 0.38227 -> 0.382866
- link r_hip_1: mass 0.920101 -> 0.919978
- link r_hip_2: mass 0.4194 -> 0.418361
Joints:
- added joint l_upper_leg_back_contact_fixed_joint: type fixed, parent l_upper_leg, child l_upper_leg_back_contact, origin xyz=-0.0512567 0 0.0146 rpy=0 1.57079632679 0
- added joint l_upper_leg_dh_frame_fixed_joint: type fixed, parent l_upper_leg, child l_upper_leg_dh_frame, origin xyz=0 0 -0.145825 rpy=1.57079632679 0 0
- added joint r_upper_leg_back_contact_fixed_joint: type fixed, parent r_upper_leg, child r_upper_leg_back_contact, origin xyz=-0.0511999 0 0.0146 rpy=0 1.57079632679 0
- added joint r_upper_leg_dh_frame_fixed_joint: type fixed, parent r_upper_leg, child r_upper_leg_dh_frame, origin xyz=0 0 -0.145825 rpy=1.57079632679 0 0
- joint l_ankle_pitch: axis 1.0 0.0 0.0 -> 2.22044604925e-16 1.0 0.0; origin xyz=0.0406034 -0.2005 0 rpy=0 0 0 -> xyz=0 0 -0.2005 rpy=0 0 0
- joint l_ankle_roll: axis 0.0 0.0 1.0 -> 1.0 0.0 2.22044604925e-16; origin xyz=-0.0270179 0 0.04808755 rpy=0 0 0 -> xyz=0 0 0 rpy=0 0 0
- joint l_foot_ft_sensor: origin xyz=0 -0.0603 -0.05158755 rpy=1.57079632679 -1.57079632679 0 -> xyz=-0.0035 0 -0.0605 rpy=3.14159265359 0 0
- joint l_hip_pitch: axis -1.0 0.0 0.0 -> -2.22044604925e-16 -1.0 0.0; origin xyz=0.0064515 -0.0223861 -0.119913 rpy=1.57079632679 0 -1.57079632679 -> xyz=0.0064515 -0.026 -0.119913 rpy=0 0 -3.14159265359
- joint l_hip_roll: axis 0.0 0.0 1.0 -> 1.0 0.0 2.22044604925e-16; origin xyz=0.0477139 0 -0.02554 rpy=0 0 0 -> xyz=0 0.0441 0 rpy=0 0 0
- joint l_hip_yaw: axis 0.0 1.0 0.0 -> 0.0 2.22044604925e-16 1.0; origin xyz=0 0 0.0146 rpy=-1.57079632679 0 -1.57079632679 -> xyz=0 0 0.0144 rpy=-3.14159265359 0 -1.57079632679
- joint l_knee: axis -1.0 0.0 0.0 -> -2.22044604925e-16 -1.0 -0.0; origin xyz=-0.0135855 -0.145625 0 rpy=0 0 0 -> xyz=0 0 -0.145825 rpy=0 0 0
- joint l_leg_ft_sensor: origin xyz=0 -0.0743 0.0246825 rpy=1.57079632679 -1.57079632679 0 -> xyz=-0.0008575 0 -0.0743 rpy=-3.14159265359 0 -1.57079632679
- joint r_ankle_pitch: axis 1.0 0.0 0.0 -> 2.22044604925e-16 1.0 0.0; origin xyz=-0.0268325 -0.2005 0 rpy=0 0 0 -> xyz=0 0 -0.2005 rpy=0 0 0
- joint r_ankle_roll: axis -0.0 -0.0 -1.0 -> -1.0 -0.0 -2.22044604925e-16; origin xyz=0.0365 0 -0.0185 rpy=0 0 0 -> xyz=0 0 0 rpy=0 0 0
- joint r_foot_ft_sensor: origin xyz=0 -0.0603 0.015 rpy=1.57079632679 -1.57079632679 0 -> xyz=-0.0035 0 -0.0605 rpy=3.14159265359 0 0
- joint r_hip_pitch: axis -1.0 -0.0 -0.0 -> -2.22044604925e-16 -1.0 -0.0; origin xyz=0.0064515 0.0233655 -0.119913 rpy=1.57079632679 0 -1.57079632679 -> xyz=0.0064515 0.026 -0.119913 rpy=0 0 -3.14159265359
- joint r_hip_roll: axis -0.0 -0.0 -1.0 -> -1.0 0.0 -2.22044604925e-16; origin xyz=-0.0467345 0 -0.0263447 rpy=0 0 0 -> xyz=0 -0.0441 0 rpy=0 0 0
- joint r_hip_yaw: axis 0.0 -1.0 0.0 -> 0.0 -2.22044604925e-16 -1.0; origin xyz=0 0 0.0146 rpy=-1.57079632679 0 -1.57079632679 -> xyz=0 0 0.0144 rpy=-3.14159265359 0 0
- joint r_knee: axis -1.0 -0.0 -0.0 -> -2.22044604925e-16 -1.0 0.0; origin xyz=-0.0096675 -0.145625 0 rpy=0 0 0 -> xyz=0 0 -0.145825 rpy=0 0 0
- joint r_leg_ft_sensor: origin xyz=0 -0.0743 0.0254872 rpy=1.57079632679 -1.57079632679 0 -> xyz=-0.0008575 0 -0.0743 rpy=3.14159265359 0 0
- joint r_lower_leg_skin_0_fixed_joint: origin xyz=-0.0215465 -0.002634 0.0544117 rpy=-0.660978905975 0.123114980697 1.4755829697 -> xyz=0.0544117 -0.031214 -0.002634 rpy=2.09173809157e-06 -1.41530676247 2.48648458622
- joint r_lower_leg_skin_10_fixed_joint: origin xyz=0.0100099 -0.021205 0.0644607 rpy=0.000432173736511 -0.0998382821227 1.57075325095 -> xyz=0.0644607 0.0003424 -0.021205 rpy=3.14159265355 -1.47095803541 0.000430021675261
- joint r_lower_leg_skin_11_fixed_joint: origin xyz=-0.0064241 -0.030885 0.0607108 rpy=-0.279936053974 -0.233577889652 1.63723971694 -> xyz=0.0607108 -0.0160916 -0.030885 rpy=-3.14159218252 -1.3281180406 -0.27213836788
- joint r_lower_leg_skin_14_fixed_joint: origin xyz=-0.0215085 -0.0219 0.0550477 rpy=-0.65674037676 -0.0838840185901 1.6352968064 -> xyz=0.0550477 -0.031176 -0.0219 rpy=-3.14159181885 -1.46502735635 -0.654033407167
- joint r_lower_leg_skin_15_fixed_joint: origin xyz=-0.0065113 0.007243 0.0591708 rpy=-0.287349971655 0.306509038255 1.48186077381 -> xyz=0.0591708 -0.0161788 0.007243 rpy=4.27484256729e-07 -1.25203633076 2.86798859471
- joint r_lower_leg_skin_16_fixed_joint: origin xyz=-0.0406195 -0.004549 0.0272875 rpy=-1.17903435098 0.0145863542197 1.53550278559 -> xyz=0.0272875 -0.050287 -0.004549 rpy=1.33075915123e-05 -1.53260853515 1.96280242835
- joint r_lower_leg_skin_17_fixed_joint: origin xyz=-0.0406445 -0.023882 0.027875 rpy=-1.18020591847 -0.0027159844464 1.57739302393 -> xyz=0.027875 -0.050312 -0.023882 rpy=-3.1415645262 -1.56366240237 -1.18022508756
- joint r_lower_leg_skin_19_fixed_joint: origin xyz=0.0507303 0.006065 0.0357534 rpy=0.987216858918 0.0751545057171 1.68402242082 -> xyz=0.0357534 0.0410628 0.006065 rpy=-8.90877717426e-07 -1.43498696978 -2.15863618017
- joint r_lower_leg_skin_20_fixed_joint: origin xyz=0.0576583 -0.004952 0.0234419 rpy=1.27473610115 0.0206410616106 1.6383594359 -> xyz=0.0234419 0.0479908 -0.004952 rpy=-3.20556549428e-06 -1.50015513031 -1.86755092413
- joint r_lower_leg_skin_21_fixed_joint: origin xyz=0.0582053 -0.024277 0.0242704 rpy=1.26752944172 0.00458214989839 1.58543727798 -> xyz=0.0242704 0.0485378 -0.024277 rpy=2.29671149558e-05 -1.55545513881 -1.87411972316
- joint r_lower_leg_skin_28_fixed_joint: origin xyz=-0.0327725 -0.032756 0.04087215 rpy=-0.930251372093 -0.0288636035903 1.60949343025 -> xyz=0.04087215 -0.04244 -0.032756 rpy=3.14158088865 -1.52252462169 -0.929681029763
- joint r_lower_leg_skin_29_fixed_joint: origin xyz=-0.0338485 -0.05242 0.03846637 rpy=-0.915770698544 -0.0222403533337 1.59973768678 -> xyz=0.03846637 -0.043516 -0.05242 rpy=3.14158017044 -1.53429841563 -0.915436346631
- joint r_lower_leg_skin_31_fixed_joint: origin xyz=-0.0326035 0.006327 0.03914638 rpy=-0.938611596431 0.0903584824077 1.44821993266 -> xyz=0.03914638 -0.042271 0.006327 rpy=-6.58381747139e-07 -1.4186494462 2.20853032986
- joint r_lower_leg_skin_32_fixed_joint: origin xyz=0.0422522 -0.080733 0.04598301 rpy=0.64650651578 -0.0386542965682 1.54163935643 -> xyz=0.04598301 0.0325847 -0.080733 rpy=-3.14159014988 -1.52238289798 0.645940380887
- joint r_lower_leg_skin_35_fixed_joint: origin xyz=-0.0215645 -0.080113 0.04774866 rpy=-0.542152349621 -0.0455923960272 1.59824328594 -> xyz=0.04774866 -0.031232 -0.080113 rpy=-3.14158668275 -1.51758467332 -0.541532486468
- joint r_lower_leg_skin_36_fixed_joint: origin xyz=-0.0059343 -0.088362 0.05322409 rpy=-0.207709325297 -0.0537454077707 1.58211730453 -> xyz=0.05322409 -0.0156018 -0.088362 rpy=-3.14159034144 -1.51587265281 -0.20740733566
- joint r_lower_leg_skin_37_fixed_joint: origin xyz=0.0106319 -0.078318 0.0552572 rpy=0.00754389164192 -0.0476116089222 1.57043779524 -> xyz=0.0552572 0.0009644 -0.078318 rpy=-3.14158180452 -1.52318336898 0.00752450583063
- joint r_lower_leg_skin_38_fixed_joint: origin xyz=-0.0215955 -0.060757 0.04880467 rpy=-0.542830301827 -0.0471634712563 1.59923066943 -> xyz=0.04880467 -0.031263 -0.060757 rpy=3.14158665199 -1.5157299554 -0.54215359959
- joint r_lower_leg_skin_3_fixed_joint: origin xyz=0.040088 -0.002843 0.05157878 rpy=0.842654955784 0.0943728500099 1.67609780358 -> xyz=0.05157878 0.0304205 -0.002843 rpy=0 -1.42951054083 -2.30391484186
- joint r_lower_leg_skin_41_fixed_joint: origin xyz=-0.0062454 -0.049854 0.0566009 rpy=-0.251468147514 -0.158913056373 1.61142822718 -> xyz=0.0566009 -0.0159129 -0.049854 rpy=-3.14159198825 -1.40681343597 -0.248233089413
- joint r_lower_leg_skin_42_fixed_joint: origin xyz=0.0104637 -0.05908 0.0570106 rpy=0.00694017036085 -0.135545595322 1.56985808158 -> xyz=0.0570106 0.0007962 -0.05908 rpy=3.14158970239 -1.43524750416 0.00687943651504
- joint r_lower_leg_skin_43_fixed_joint: origin xyz=0.0420328 -0.061362 0.04712542 rpy=0.624467273745 -0.026260830452 1.55187529497 -> xyz=0.04712542 0.0323653 -0.061362 rpy=-3.14159136621 -1.53843038237 0.624217523667
- joint r_lower_leg_skin_46_fixed_joint: origin xyz=0.0268839 -0.05018 0.0558156 rpy=0.328741310202 -0.135625619972 1.52470662181 -> xyz=0.0558156 0.0172164 -0.05018 rpy=-3.14158987809 -1.42759881603 0.325607710876
- joint r_lower_leg_skin_47_fixed_joint: origin xyz=0.0273064 -0.08886 0.05264163 rpy=0.263001895535 -0.0520410015187 1.55679195888 -> xyz=0.05264163 0.0176389 -0.08886 rpy=3.14158963519 -1.51690559406 0.262640425058
- joint r_lower_leg_skin_49_fixed_joint: origin xyz=0.042106 -0.138859 0.04113137 rpy=0.731392432649 -0.0602196903016 1.51683891676 -> xyz=0.04113137 0.0324385 -0.138859 rpy=-3.14158934751 -1.48996135695 0.729763592113
- joint r_lower_leg_skin_4_fixed_joint: origin xyz=0.0264511 0.007272 0.0583103 rpy=0.40039718175 0.29099345069 1.69164016714 -> xyz=0.0583103 0.0167836 0.007272 rpy=-2.98636361519e-07 -1.25636748876 -2.75892380087
- joint r_lower_leg_skin_50_fixed_joint: origin xyz=0.0421948 -0.119469 0.043016947 rpy=0.69705122002 -0.055082279609 1.52473387321 -> xyz=0.043016947 0.0325273 -0.119469 rpy=3.14159069596 -1.49900732636 0.695784020081
- joint r_lower_leg_skin_51_fixed_joint: origin xyz=0.0274265 -0.108206 0.05141583 rpy=0.272623174864 -0.0621353313747 1.55343743538 -> xyz=0.05141583 0.017759 -0.108206 rpy=-3.14158890179 -1.50628475717 0.272079935713
- joint r_lower_leg_skin_52_fixed_joint: origin xyz=0.0109339 -0.116895 0.05299832 rpy=0.0108976323462 -0.0676055809873 1.57006018656 -> xyz=0.05299832 0.0012664 -0.116895 rpy=-3.14159164042 -1.50318674421 0.0108717260994
- joint r_lower_leg_skin_53_fixed_joint: origin xyz=-0.0057664 -0.107654 0.05207312 rpy=-0.211841375505 -0.063397660111 1.58442104098 -> xyz=0.05207312 -0.0154339 -0.107654 rpy=3.14159063987 -1.50595307447 -0.211407322892
- joint r_lower_leg_skin_54_fixed_joint: origin xyz=-0.0210815 -0.118787 0.04512708 rpy=-0.576349226046 -0.0615294995172 1.61074135295 -> xyz=0.04512708 -0.030749 -0.118787 rpy=3.14158825193 -1.49745145571 -0.575115374473
- joint r_lower_leg_skin_55_fixed_joint: origin xyz=-0.0208215 -0.138143 0.043502663 rpy=-0.598745472791 -0.0668224323993 1.61632329625 -> xyz=0.043502663 -0.030489 -0.138143 rpy=3.14158906486 -1.48995787038 -0.597219943789
- joint r_lower_leg_skin_56_fixed_joint: origin xyz=-0.0054535 -0.146218 0.04926839 rpy=-0.224166511744 -0.0775658268571 1.58846192551 -> xyz=0.04926839 -0.015121 -0.146218 rpy=-3.14158920404 -1.49124819828 -0.2234844764
- joint r_lower_leg_skin_5_fixed_joint: origin xyz=0.0099769 -0.001972 0.0636503 rpy=0.000123038724669 0.184274174748 1.57081887154 -> xyz=0.0636503 0.0003094 -0.001972 rpy=0 -1.38652215068 -3.14147169807
- joint r_lower_leg_skin_60_fixed_joint: origin xyz=0.0277235 -0.146938 0.04836967 rpy=0.303887741163 -0.0772432614252 1.54660163218 -> xyz=0.04836967 0.018056 -0.146938 rpy=-3.14159173337 -1.48985968527 0.302951871954
- joint r_lower_leg_skin_61_fixed_joint: origin xyz=0.0110941 -0.136169 0.05161952 rpy=0.0132400606487 -0.0747688280205 1.56980737046 -> xyz=0.05161952 0.0014266 -0.136169 rpy=-3.14159100925 -1.49602097086 0.0132014275205
- joint r_lower_leg_skin_6_fixed_joint: origin xyz=0.0401109 -0.022149 0.05208552 rpy=0.840135245525 -0.0688367062203 1.49419034934 -> xyz=0.05208552 0.0304434 -0.022149 rpy=-3.14158927953 -1.46785123411 0.837492889077
- joint r_lower_leg_skin_9_fixed_joint: origin xyz=0.0264648 -0.030962 0.0598214 rpy=0.388444125907 -0.212046974802 1.48487982461 -> xyz=0.0598214 0.0167973 -0.030962 rpy=-3.14159202356 -1.34224755325 0.379294477718

Commit message: Automatic build. Travis build:137
icub-model-generator commit:f05e54586e450725b7ac6364dc26e90fa0fd9324

urdf_parser_py commit:31474b9baaf7c3845b40e5a9aa87d5900a2282c3

simmechanics-to-urdf commit:2a7a34ebeaed81ac059825447879d715d175489d

codyco-superbuild commit:39293fe2863e1e8afc522eac683c96250078eea1

File: iCub/robots/iCubDarmstadt01/model.urdf (robot description, URDF)
Before this commit: robot iCub, 139 links, 138 joints
Joints:
- joint l_ankle_pitch: limit lower=-0.610865238198 upper=0.610865238198 effort=50000 velocity=50000 -> lower=-0.610865238198 upper=0.610865238198 effort=37.0 velocity=7.64
- joint l_ankle_roll: limit lower=-0.436332312999 upper=0.436332312999 effort=50000 velocity=50000 -> lower=-0.436332312999 upper=0.436332312999 effort=37.0 velocity=7.64
- joint l_hip_pitch: limit lower=-0.785398163397 upper=2.33874119767 effort=50000 velocity=50000 -> lower=-0.785398163397 upper=2.33874119767 effort=55.5 velocity=5.1
- joint l_hip_roll: limit lower=-0.349065850399 upper=2.09439510239 effort=50000 velocity=50000 -> lower=-0.349065850399 upper=2.09439510239 effort=37.0 velocity=7.64
- joint l_hip_yaw: limit lower=-1.3962634016 upper=1.3962634016 effort=50000 velocity=50000 -> lower=-1.3962634016 upper=1.3962634016 effort=37.0 velocity=7.64
- joint l_knee: limit lower=-2.16420827247 upper=0.0698131700798 effort=50000 velocity=50000 -> lower=-2.16420827247 upper=0.0698131700798 effort=37.0 velocity=7.64
- joint r_ankle_pitch: limit lower=-0.610865238198 upper=0.610865238198 effort=50000 velocity=50000 -> lower=-0.610865238198 upper=0.610865238198 effort=37.0 velocity=7.64
- joint r_ankle_roll: limit lower=-0.436332312999 upper=0.436332312999 effort=50000 velocity=50000 -> lower=-0.436332312999 upper=0.436332312999 effort=37.0 velocity=7.64
- joint r_hip_pitch: limit lower=-0.785398163397 upper=2.33874119767 effort=50000 velocity=50000 -> lower=-0.785398163397 upper=2.33874119767 effort=55.5 velocity=5.1
- joint r_hip_roll: limit lower=-0.349065850399 upper=2.09439510239 effort=50000 velocity=50000 -> lower=-0.349065850399 upper=2.09439510239 effort=37.0 velocity=7.64
- joint r_hip_yaw: limit lower=-1.3962634016 upper=1.3962634016 effort=50000 velocity=50000 -> lower=-1.3962634016 upper=1.3962634016 effort=37.0 velocity=7.64
- joint r_knee: limit lower=-2.16420827247 upper=0.0698131700798 effort=50000 velocity=50000 -> lower=-2.16420827247 upper=0.0698131700798 effort=37.0 velocity=7.64

File: iCub/robots/iCubGenova02/model.urdf (robot description, URDF)
Before this commit: robot iCub, 139 links, 138 joints
Joints:
- joint l_ankle_pitch: limit lower=-0.610865238198 upper=0.610865238198 effort=50000 velocity=50000 -> lower=-0.610865238198 upper=0.610865238198 effort=37.0 velocity=7.64
- joint l_ankle_roll: limit lower=-0.436332312999 upper=0.436332312999 effort=50000 velocity=50000 -> lower=-0.436332312999 upper=0.436332312999 effort=37.0 velocity=7.64
- joint l_hip_pitch: limit lower=-0.785398163397 upper=2.33874119767 effort=50000 velocity=50000 -> lower=-0.785398163397 upper=2.33874119767 effort=55.5 velocity=5.1
- joint l_hip_roll: limit lower=-0.349065850399 upper=2.09439510239 effort=50000 velocity=50000 -> lower=-0.349065850399 upper=2.09439510239 effort=37.0 velocity=7.64
- joint l_hip_yaw: limit lower=-1.3962634016 upper=1.3962634016 effort=50000 velocity=50000 -> lower=-1.3962634016 upper=1.3962634016 effort=37.0 velocity=7.64
- joint l_knee: limit lower=-2.16420827247 upper=0.0698131700798 effort=50000 velocity=50000 -> lower=-2.16420827247 upper=0.0698131700798 effort=37.0 velocity=7.64
- joint r_ankle_pitch: limit lower=-0.610865238198 upper=0.610865238198 effort=50000 velocity=50000 -> lower=-0.610865238198 upper=0.610865238198 effort=37.0 velocity=7.64
- joint r_ankle_roll: limit lower=-0.436332312999 upper=0.436332312999 effort=50000 velocity=50000 -> lower=-0.436332312999 upper=0.436332312999 effort=37.0 velocity=7.64
- joint r_hip_pitch: limit lower=-0.785398163397 upper=2.33874119767 effort=50000 velocity=50000 -> lower=-0.785398163397 upper=2.33874119767 effort=55.5 velocity=5.1
- joint r_hip_roll: limit lower=-0.349065850399 upper=2.09439510239 effort=50000 velocity=50000 -> lower=-0.349065850399 upper=2.09439510239 effort=37.0 velocity=7.64
- joint r_hip_yaw: limit lower=-1.3962634016 upper=1.3962634016 effort=50000 velocity=50000 -> lower=-1.3962634016 upper=1.3962634016 effort=37.0 velocity=7.64
- joint r_knee: limit lower=-2.16420827247 upper=0.0698131700798 effort=50000 velocity=50000 -> lower=-2.16420827247 upper=0.0698131700798 effort=37.0 velocity=7.64

Commit message: Automatic build. Travis build:180
icub-model-generator commit:bc1ed7765d51be14a323b02cbe1936644e029d22

urdf_parser_py commit:31474b9baaf7c3845b40e5a9aa87d5900a2282c3

simmechanics-to-urdf commit:6af33bb59e2ebd2b850041b8f324d136727ff413

codyco-superbuild commit:52bcb48758c8c92074fa8971e615cf6897de1984

File: iCub/robots/iCubDarmstadt01/model.urdf (robot description, URDF)
Before this commit: robot iCub, 139 links, 138 joints
Links:
- link l_foot: geometry collision box size=0.16 0.072 0.001; visual mesh filename=package://iCub/meshes/simmechanics/sim_sea_2-5_l_sole_prt-b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 scale=0.001 0.001 0.001
- link r_foot: geometry collision box size=0.16 0.072 0.001; visual mesh filename=package://iCub/meshes/simmechanics/sim_sea_2-5_r_sole_prt-b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 scale=0.001 0.001 0.001

File: iCub/robots/iCubGazeboV2_5/model.urdf (robot description, URDF)
Before this commit: robot iCub, 139 links, 138 joints
Links:
- link l_foot: geometry collision box size=0.16 0.072 0.001; visual mesh filename=package://iCub/meshes/simmechanics/sim_sea_2-5_l_sole_prt-b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 scale=0.001 0.001 0.001
- link r_foot: geometry collision box size=0.16 0.072 0.001; visual mesh filename=package://iCub/meshes/simmechanics/sim_sea_2-5_r_sole_prt-b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 scale=0.001 0.001 0.001

File: iCub/robots/iCubGazeboV2_5_plus/model.urdf (robot description, URDF)
Before this commit: robot iCub, 140 links, 139 joints
Links:
- link l_foot: geometry collision box size=0.16 0.072 0.001; visual mesh filename=package://iCub/meshes/simmechanics/2-5_plus/sim_sea_2-5_l_s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 scale=0.001 0.001 0.001
- link r_foot: geometry collision box size=0.16 0.072 0.001; visual mesh filename=package://iCub/meshes/simmechanics/2-5_plus/sim_sea_2-5_r_s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 scale=0.001 0.001 0.001

File: iCub/robots/iCubGenova02/model.urdf (robot description, URDF)
Before this commit: robot iCub, 139 links, 138 joints
Links:
- link l_foot: geometry collision box size=0.16 0.072 0.001; visual mesh filename=package://iCub/meshes/simmechanics/sim_sea_2-5_l_sole_prt-b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 scale=0.001 0.001 0.001
- link r_foot: geometry collision box size=0.16 0.072 0.001; visual mesh filename=package://iCub/meshes/simmechanics/sim_sea_2-5_r_sole_prt-b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 scale=0.001 0.001 0.001

File: iCub/robots/iCubGenova04_plus/model.urdf (robot description, URDF)
Before this commit: robot iCub, 140 links, 139 joints
Links:
- link l_foot: geometry collision box size=0.16 0.072 0.001; visual mesh filename=package://iCub/meshes/simmechanics/2-5_plus/sim_sea_2-5_l_s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 scale=0.001 0.001 0.001
- link r_foot: geometry collision box size=0.16 0.072 0.001; visual mesh filename=package://iCub/meshes/simmechanics/2-5_plus/sim_sea_2-5_r_s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 scale=0.001 0.001 0.001

Commit message: Automatic build. Travis build:185
icub-model-generator commit:ff76e33642df09c3de746a1104e0aa112a588386

urdf_parser_py commit:31474b9baaf7c3845b40e5a9aa87d5900a2282c3

simmechanics-to-urdf commit:6af33bb59e2ebd2b850041b8f324d136727ff413

codyco-superbuild commit:52bcb48758c8c92074fa8971e615cf6897de1984

File: iCub/robots/iCubDarmstadt01/model.urdf (robot description, URDF)
Before this commit: robot iCub, 139 links, 138 joints
Links:
- link l_foot: geometry collision mesh filename=package://iCub/meshes/simmechanics/sim_sea_2-5_l_sole_prt-b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 scale=0.001 0.001 0.001; visual mesh filename=package://iCub/meshes/simmechanics/sim_sea_2-5_l_sole_prt-b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 scale=0.001 0.001 0.001
- link r_foot: geometry collision mesh filename=package://iCub/meshes/simmechanics/sim_sea_2-5_r_sole_prt-b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 scale=0.001 0.001 0.001; visual mesh filename=package://iCub/meshes/simmechanics/sim_sea_2-5_r_sole_prt-b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 scale=0.001 0.001 0.001

File: iCub/robots/iCubGenova02/model.urdf (robot description, URDF)
Before this commit: robot iCub, 139 links, 138 joints
Links:
- link l_foot: geometry collision mesh filename=package://iCub/meshes/simmechanics/sim_sea_2-5_l_sole_prt-b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 scale=0.001 0.001 0.001; visual mesh filename=package://iCub/meshes/simmechanics/sim_sea_2-5_l_sole_prt-b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 scale=0.001 0.001 0.001
- link r_foot: geometry collision mesh filename=package://iCub/meshes/simmechanics/sim_sea_2-5_r_sole_prt-b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 scale=0.001 0.001 0.001; visual mesh filename=package://iCub/meshes/simmechanics/sim_sea_2-5_r_sole_prt-b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 scale=0.001 0.001 0.001

File: iCub/robots/iCubGenova04_plus/model.urdf (robot description, URDF)
Before this commit: robot iCub, 140 links, 139 joints
Links:
- link l_foot: geometry collision mesh filename=package://iCub/meshes/simmechanics/2-5_plus/sim_sea_2-5_l_s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 scale=0.001 0.001 0.001; visual mesh filename=package://iCub/meshes/simmechanics/2-5_plus/sim_sea_2-5_l_s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 scale=0.001 0.001 0.001
- link r_foot: geometry collision mesh filename=package://iCub/meshes/simmechanics/2-5_plus/sim_sea_2-5_r_s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 scale=0.001 0.001 0.001; visual mesh filename=package://iCub/meshes/simmechanics/2-5_plus/sim_sea_2-5_r_s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 scale=0.001 0.001 0.001
