Commit message: Automatic build. Travis build:208
icub-model-generator commit:ee5dfd1797836faabea7f492a6b283495089c76d

urdf_parser_py commit:31474b9baaf7c3845b40e5a9aa87d5900a2282c3

simmechanics-to-urdf commit:6af33bb59e2ebd2b850041b8f324d136727ff413

yarp commit:643a973b388588cd39f498b94e630f3371d05b14

icub-main commit:4f5881acafab693f763dd277f87a8996fdea01a3

idyntree commit:94cee9db71266d65445a7a752342fa473159faaf

File: iCub/robots/iCubDarmstadt01/model.urdf (robot description, URDF)
Before this commit: robot iCub, 139 links, 138 joints
Joints:
- joint l_knee: axis -2.22044604925e-16 -1.0 -0.0 -> -2.22044604925e-16 -1.0 0.0
- joint r_ankle_roll: axis -1.0 -0.0 -2.22044604925e-16 -> -1.0 0.0 -2.22044604925e-16
- joint r_hip_pitch: axis -2.22044604925e-16 -1.0 -0.0 -> -2.22044604925e-16 -1.0 0.0

File: iCub/robots/iCubGazeboV2_5/model.urdf (robot description, URDF)
Before this commit: robot iCub, 139 links, 138 joints
Joints:
- joint l_knee: axis -2.22044604925e-16 -1.0 -0.0 -> -2.22044604925e-16 -1.0 0.0
- joint r_ankle_roll: axis -1.0 -0.0 -2.22044604925e-16 -> -1.0 0.0 -2.22044604925e-16
- joint r_hip_pitch: axis -2.22044604925e-16 -1.0 -0.0 -> -2.22044604925e-16 -1.0 0.0

File: iCub/robots/iCubGazeboV2_5_plus/model.urdf (robot description, URDF)
Before this commit: robot iCub, 140 links, 139 joints
Joints:
- joint l_hip_pitch: axis -2.22044604925e-16 -1.0 -0.0 -> -2.22044604925e-16 -1.0 0.0
- joint l_knee: axis -2.22044604925e-16 -1.0 -0.0 -> -2.22044604925e-16 -1.0 0.0

File: iCub/robots/iCubGenova02/model.urdf (robot description, URDF)
Before this commit: robot iCub, 139 links, 138 joints
Joints:
- joint l_knee: axis -2.22044604925e-16 -1.0 -0.0 -> -2.22044604925e-16 -1.0 0.0
- joint r_ankle_roll: axis -1.0 -0.0 -2.22044604925e-16 -> -1.0 0.0 -2.22044604925e-16
- joint r_hip_pitch: axis -2.22044604925e-16 -1.0 -0.0 -> -2.22044604925e-16 -1.0 0.0

File: iCub/robots/iCubGenova03/model.urdf (robot description, URDF)
Before this commit: robot iCub, 56 links, 55 joints
Joints:
- joint l_shoulder_roll: origin xyz=0 0 0 rpy=1.5708 -0 -1.5708 -> xyz=0 0 0 rpy=1.5708 -1.11022e-16 -1.5708
- joint l_wrist_pitch: origin xyz=0 0.1373 8.4072e-18 rpy=1.5708 -0 1.5708 -> xyz=0 0.1373 8.4072e-18 rpy=1.5708 1.11022e-16 1.5708
- joint l_wrist_prosup: origin xyz=-0.015 0 0 rpy=1.5708 -0 -1.5708 -> xyz=-0.015 0 0 rpy=1.5708 -1.11022e-16 -1.5708
- joint neck_pitch: origin xyz=0.00231 0.1933 -1.18362e-17 rpy=1.5708 -0 1.5708 -> xyz=0.00231 0.1933 -1.18362e-17 rpy=1.5708 1.11022e-16 1.5708
- joint neck_roll: origin xyz=0.0095 0 0 rpy=-1.5708 -0 -1.5708 -> xyz=0.0095 0 0 rpy=-1.5708 1.11022e-16 -1.5708
- joint neck_yaw: origin xyz=-5.77779e-34 0 0 rpy=-1.5708 -0 1.5708 -> xyz=-5.77779e-34 0 0 rpy=-1.5708 -1.11022e-16 1.5708
- joint r_shoulder_roll: origin xyz=0 0 0 rpy=-1.5708 -0 -1.5708 -> xyz=0 0 0 rpy=-1.5708 1.11022e-16 -1.5708
- joint r_wrist_pitch: origin xyz=0 -0.1373 -8.4072e-18 rpy=1.5708 -0 1.5708 -> xyz=0 -0.1373 -8.4072e-18 rpy=1.5708 1.11022e-16 1.5708
- joint r_wrist_prosup: origin xyz=0.015 0 0 rpy=1.5708 -0 -1.5708 -> xyz=0.015 0 0 rpy=1.5708 -1.11022e-16 -1.5708
- joint torso_roll: origin xyz=0.032 -2.67276e-51 0 rpy=1.5708 -0 -1.5708 -> xyz=0.032 -2.67276e-51 0 rpy=1.5708 -1.11022e-16 -1.5708
- joint torso_yaw: origin xyz=-7.46298e-34 -0.0055 0 rpy=-1.5708 -0 -1.5708 -> xyz=-7.46298e-34 -0.0055 0 rpy=-1.5708 1.11022e-16 -1.5708

File: iCub/robots/iCubGenova04_plus/model.urdf (robot description, URDF)
Before this commit: robot iCub, 140 links, 139 joints
Joints:
- joint l_hip_pitch: axis -2.22044604925e-16 -1.0 -0.0 -> -2.22044604925e-16 -1.0 0.0
- joint l_knee: axis -2.22044604925e-16 -1.0 -0.0 -> -2.22044604925e-16 -1.0 0.0

File: iCub/robots/iCubLisboa01/model.urdf (robot description, URDF)
Before this commit: robot iCub, 54 links, 53 joints
Joints:
- joint l_shoulder_roll: origin xyz=0 0 0 rpy=1.5708 -0 -1.5708 -> xyz=0 0 0 rpy=1.5708 -1.11022e-16 -1.5708
- joint l_wrist_pitch: origin xyz=0 0.1373 8.4072e-18 rpy=1.5708 -0 1.5708 -> xyz=0 0.1373 8.4072e-18 rpy=1.5708 1.11022e-16 1.5708
- joint l_wrist_prosup: origin xyz=-0.015 0 0 rpy=1.5708 -0 -1.5708 -> xyz=-0.015 0 0 rpy=1.5708 -1.11022e-16 -1.5708
- joint neck_pitch: origin xyz=0.00231 0.1933 -1.18362e-17 rpy=1.5708 -0 1.5708 -> xyz=0.00231 0.1933 -1.18362e-17 rpy=1.5708 1.11022e-16 1.5708
- joint neck_roll: origin xyz=0.0095 0 0 rpy=-1.5708 -0 -1.5708 -> xyz=0.0095 0 0 rpy=-1.5708 1.11022e-16 -1.5708
- joint neck_yaw: origin xyz=-5.77779e-34 0 0 rpy=-1.5708 -0 1.5708 -> xyz=-5.77779e-34 0 0 rpy=-1.5708 -1.11022e-16 1.5708
- joint r_shoulder_roll: origin xyz=0 0 0 rpy=-1.5708 -0 -1.5708 -> xyz=0 0 0 rpy=-1.5708 1.11022e-16 -1.5708
- joint r_wrist_pitch: origin xyz=0 -0.1373 -8.4072e-18 rpy=1.5708 -0 1.5708 -> xyz=0 -0.1373 -8.4072e-18 rpy=1.5708 1.11022e-16 1.5708
- joint r_wrist_prosup: origin xyz=0.015 0 0 rpy=1.5708 -0 -1.5708 -> xyz=0.015 0 0 rpy=1.5708 -1.11022e-16 -1.5708
- joint torso_roll: origin xyz=0.032 -2.67276e-51 0 rpy=1.5708 -0 -1.5708 -> xyz=0.032 -2.67276e-51 0 rpy=1.5708 -1.11022e-16 -1.5708
- joint torso_yaw: origin xyz=-7.46298e-34 -0.0055 0 rpy=-1.5708 -0 -1.5708 -> xyz=-7.46298e-34 -0.0055 0 rpy=-1.5708 1.11022e-16 -1.5708

File: iCub/robots/iCubNancy01/model.urdf (robot description, URDF)
Before this commit: robot iCub, 56 links, 55 joints
Joints:
- joint l_shoulder_roll: origin xyz=0 0 0 rpy=1.5708 -0 -1.5708 -> xyz=0 0 0 rpy=1.5708 -1.11022e-16 -1.5708
- joint l_wrist_pitch: origin xyz=0 0.1373 8.4072e-18 rpy=1.5708 -0 1.5708 -> xyz=0 0.1373 8.4072e-18 rpy=1.5708 1.11022e-16 1.5708
- joint l_wrist_prosup: origin xyz=-0.015 0 0 rpy=1.5708 -0 -1.5708 -> xyz=-0.015 0 0 rpy=1.5708 -1.11022e-16 -1.5708
- joint neck_pitch: origin xyz=0.00231 0.1933 -1.18362e-17 rpy=1.5708 -0 1.5708 -> xyz=0.00231 0.1933 -1.18362e-17 rpy=1.5708 1.11022e-16 1.5708
- joint neck_roll: origin xyz=0.0095 0 0 rpy=-1.5708 -0 -1.5708 -> xyz=0.0095 0 0 rpy=-1.5708 1.11022e-16 -1.5708
- joint neck_yaw: origin xyz=-5.77779e-34 0 0 rpy=-1.5708 -0 1.5708 -> xyz=-5.77779e-34 0 0 rpy=-1.5708 -1.11022e-16 1.5708
- joint r_shoulder_roll: origin xyz=0 0 0 rpy=-1.5708 -0 -1.5708 -> xyz=0 0 0 rpy=-1.5708 1.11022e-16 -1.5708
- joint r_wrist_pitch: origin xyz=0 -0.1373 -8.4072e-18 rpy=1.5708 -0 1.5708 -> xyz=0 -0.1373 -8.4072e-18 rpy=1.5708 1.11022e-16 1.5708
- joint r_wrist_prosup: origin xyz=0.015 0 0 rpy=1.5708 -0 -1.5708 -> xyz=0.015 0 0 rpy=1.5708 -1.11022e-16 -1.5708
- joint torso_roll: origin xyz=0.032 -2.67276e-51 0 rpy=1.5708 -0 -1.5708 -> xyz=0.032 -2.67276e-51 0 rpy=1.5708 -1.11022e-16 -1.5708
- joint torso_yaw: origin xyz=-7.46298e-34 -0.0055 0 rpy=-1.5708 -0 -1.5708 -> xyz=-7.46298e-34 -0.0055 0 rpy=-1.5708 1.11022e-16 -1.5708

File: iCub/robots/iCubParis01/model.urdf (robot description, URDF)
Before this commit: robot iCub, 56 links, 55 joints
Joints:
- joint l_shoulder_roll: origin xyz=0 0 0 rpy=1.5708 -0 -1.5708 -> xyz=0 0 0 rpy=1.5708 -1.11022e-16 -1.5708
- joint l_wrist_pitch: origin xyz=0 0.1373 8.4072e-18 rpy=1.5708 -0 1.5708 -> xyz=0 0.1373 8.4072e-18 rpy=1.5708 1.11022e-16 1.5708
- joint l_wrist_prosup: origin xyz=-0.015 0 0 rpy=1.5708 -0 -1.5708 -> xyz=-0.015 0 0 rpy=1.5708 -1.11022e-16 -1.5708
- joint neck_pitch: origin xyz=0.00231 0.1933 -1.18362e-17 rpy=1.5708 -0 1.5708 -> xyz=0.00231 0.1933 -1.18362e-17 rpy=1.5708 1.11022e-16 1.5708
- joint neck_roll: origin xyz=0.033 -2.13821e-50 0 rpy=-1.5708 -0 -1.5708 -> xyz=0.033 -2.13821e-50 0 rpy=-1.5708 1.11022e-16 -1.5708
- joint neck_yaw: origin xyz=0 -0.001 0 rpy=-1.5708 -0 1.5708 -> xyz=0 -0.001 0 rpy=-1.5708 -1.11022e-16 1.5708
- joint r_shoulder_roll: origin xyz=0 0 0 rpy=-1.5708 -0 -1.5708 -> xyz=0 0 0 rpy=-1.5708 1.11022e-16 -1.5708
- joint r_wrist_pitch: origin xyz=0 -0.1373 -8.4072e-18 rpy=1.5708 -0 1.5708 -> xyz=0 -0.1373 -8.4072e-18 rpy=1.5708 1.11022e-16 1.5708
- joint r_wrist_prosup: origin xyz=0.015 0 0 rpy=1.5708 -0 -1.5708 -> xyz=0.015 0 0 rpy=1.5708 -1.11022e-16 -1.5708
- joint torso_roll: origin xyz=0.032 -2.67276e-51 0 rpy=1.5708 -0 -1.5708 -> xyz=0.032 -2.67276e-51 0 rpy=1.5708 -1.11022e-16 -1.5708
- joint torso_yaw: origin xyz=-7.46298e-34 -0.0055 0 rpy=-1.5708 -0 -1.5708 -> xyz=-7.46298e-34 -0.0055 0 rpy=-1.5708 1.11022e-16 -1.5708

File: iCub/robots/iCubParis02/model.urdf (robot description, URDF)
Before this commit: robot iCub, 56 links, 55 joints
Joints:
- joint l_shoulder_roll: origin xyz=0 0 0 rpy=1.5708 -0 -1.5708 -> xyz=0 0 0 rpy=1.5708 -1.11022e-16 -1.5708
- joint l_wrist_pitch: origin xyz=0 0.1373 8.4072e-18 rpy=1.5708 -0 1.5708 -> xyz=0 0.1373 8.4072e-18 rpy=1.5708 1.11022e-16 1.5708
- joint l_wrist_prosup: origin xyz=-0.015 0 0 rpy=1.5708 -0 -1.5708 -> xyz=-0.015 0 0 rpy=1.5708 -1.11022e-16 -1.5708
- joint neck_pitch: origin xyz=0.00231 0.1933 -1.18362e-17 rpy=1.5708 -0 1.5708 -> xyz=0.00231 0.1933 -1.18362e-17 rpy=1.5708 1.11022e-16 1.5708
- joint neck_roll: origin xyz=0.0095 0 0 rpy=-1.5708 -0 -1.5708 -> xyz=0.0095 0 0 rpy=-1.5708 1.11022e-16 -1.5708
- joint neck_yaw: origin xyz=-5.77779e-34 0 0 rpy=-1.5708 -0 1.5708 -> xyz=-5.77779e-34 0 0 rpy=-1.5708 -1.11022e-16 1.5708
- joint r_shoulder_roll: origin xyz=0 0 0 rpy=-1.5708 -0 -1.5708 -> xyz=0 0 0 rpy=-1.5708 1.11022e-16 -1.5708
- joint r_wrist_pitch: origin xyz=0 -0.1373 -8.4072e-18 rpy=1.5708 -0 1.5708 -> xyz=0 -0.1373 -8.4072e-18 rpy=1.5708 1.11022e-16 1.5708
- joint r_wrist_prosup: origin xyz=0.015 0 0 rpy=1.5708 -0 -1.5708 -> xyz=0.015 0 0 rpy=1.5708 -1.11022e-16 -1.5708
- joint torso_roll: origin xyz=0.032 -2.67276e-51 0 rpy=1.5708 -0 -1.5708 -> xyz=0.032 -2.67276e-51 0 rpy=1.5708 -1.11022e-16 -1.5708
- joint torso_yaw: origin xyz=-7.46298e-34 -0.0055 0 rpy=-1.5708 -0 -1.5708 -> xyz=-7.46298e-34 -0.0055 0 rpy=-1.5708 1.11022e-16 -1.5708

Commit message: Automatic build. Travis build:209
icub-model-generator commit:e18d734aa65b91ec24fc2aa2148b1513db4a26d2

urdf_parser_py commit:31474b9baaf7c3845b40e5a9aa87d5900a2282c3

simmechanics-to-urdf commit:1bd48b2d02b1d155a782f35d96865753c2e49706

yarp commit:643a973b388588cd39f498b94e630f3371d05b14

icub-main commit:4f5881acafab693f763dd277f87a8996fdea01a3

idyntree commit:c8bf721b771fa4b1e7c3a940632e121060719a19

File: iCub/robots/iCubDarmstadt01/model.urdf (robot description, URDF)
Before this commit: robot iCub, 139 links, 138 joints
Joints:
- joint l_hip_yaw: origin xyz=0 0 0.0144 rpy=-3.14159265359 0 -1.57079632679 -> xyz=0 0 0.0144 rpy=-3.14159265359 0 0
- joint l_leg_ft_sensor: origin xyz=-0.0008575 0 -0.0743 rpy=-3.14159265359 0 -1.57079632679 -> xyz=-0.0008575 0 -0.0743 rpy=3.14159265359 0 0

File: iCub/robots/iCubGazeboV2_5/model.urdf (robot description, URDF)
Before this commit: robot iCub, 139 links, 138 joints
Joints:
- joint l_hip_yaw: origin xyz=0 0 0.0144 rpy=-3.14159265359 0 -1.57079632679 -> xyz=0 0 0.0144 rpy=-3.14159265359 0 0
- joint l_leg_ft_sensor: origin xyz=-0.0008575 0 -0.0743 rpy=-3.14159265359 0 -1.57079632679 -> xyz=-0.0008575 0 -0.0743 rpy=3.14159265359 0 0

File: iCub/robots/iCubGenova02/model.urdf (robot description, URDF)
Before this commit: robot iCub, 139 links, 138 joints
Joints:
- joint l_hip_yaw: origin xyz=0 0 0.0144 rpy=-3.14159265359 0 -1.57079632679 -> xyz=0 0 0.0144 rpy=-3.14159265359 0 0
- joint l_leg_ft_sensor: origin xyz=-0.0008575 0 -0.0743 rpy=-3.14159265359 0 -1.57079632679 -> xyz=-0.0008575 0 -0.0743 rpy=3.14159265359 0 0
