Commit message: Automatic build. Travis build:217
icub-model-generator commit:52ee80fdbfc588e09010dd418fd5904c6ac7383c

urdf_parser_py commit:31474b9baaf7c3845b40e5a9aa87d5900a2282c3

simmechanics-to-urdf commit:1bd48b2d02b1d155a782f35d96865753c2e49706

yarp commit:643a973b388588cd39f498b94e630f3371d05b14

icub-main commit:4f5881acafab693f763dd277f87a8996fdea01a3

idyntree commit:2f00c6c5011b02d36b076fca2feae7058b784f5f

File: iCub/robots/iCubDarmstadt01/model.urdf (robot description, URDF)
Before this commit: robot iCub, 139 links, 138 joints
Links:
- added link l_sole_skin_0
- added link l_sole_skin_1
- added link l_sole_skin_10
- added link l_sole_skin_11
- added link l_sole_skin_12
- added link l_sole_skin_13
- added link l_sole_skin_14
- added link l_sole_skin_15
- added link l_sole_skin_17
- added link l_sole_skin_18
- added link l_sole_skin_19
- added link l_sole_skin_2
- added link l_sole_skin_20
- added link l_sole_skin_21
- added link l_sole_skin_22
- added link l_sole_skin_24
- added link l_sole_skin_25
- added link l_sole_skin_26
- added link l_sole_skin_27
- added link l_sole_skin_28
- added link l_sole_skin_29
- added link l_sole_skin_3
- added link l_sole_skin_4
- added link l_sole_skin_8
- added link l_sole_skin_9
- added link r_sole_skin_0
- added link r_sole_skin_1
- added link r_sole_skin_10
- added link r_sole_skin_11
- added link r_sole_skin_12
- added link r_sole_skin_13
- added link r_sole_skin_14
- added link r_sole_skin_15
- added link r_sole_skin_17
- added link r_sole_skin_18
- added link r_sole_skin_19
- added link r_sole_skin_2
- added link r_sole_skin_20
- added link r_sole_skin_21
- added link r_sole_skin_22
- added link r_sole_skin_24
- added link r_sole_skin_25
- added link r_sole_skin_26
- added link r_sole_skin_27
- added link r_sole_skin_28
- added link r_sole_skin_29
- added link r_sole_skin_3
- added link r_sole_skin_4
- added link r_sole_skin_8
- added link r_sole_skin_9
Joints:
- added joint l_sole_skin_0_fixed_joint: type fixed, parent l_foot, child l_sole_skin_0, origin xyz=0.0932087 0.032368 0.0075 rpy=0 0 0
- added joint l_sole_skin_10_fixed_joint: type fixed, parent l_foot, child l_sole_skin_10, origin xyz=0.1052593 -0.0243254 0.0075 rpy=0 0 0
- added joint l_sole_skin_11_fixed_joint: type fixed, parent l_foot, child l_sole_skin_11, origin xyz=0.1012424 -0.0054281 0.0075 rpy=0 0 0
- added joint l_sole_skin_12_fixed_joint: type fixed, parent l_foot, child l_sole_skin_12, origin xyz=0.082868 0.0005426 0.0075 rpy=0 0 0
- added joint l_sole_skin_13_fixed_joint: type fixed, parent l_foot, child l_sole_skin_13, origin xyz=0.0685104 -0.0123855 0.0075 rpy=0 0 0
- added joint l_sole_skin_14_fixed_joint: type fixed, parent l_foot, child l_sole_skin_14, origin xyz=0.1156 0.0074995 0.0075 rpy=0 0 0
- added joint l_sole_skin_15_fixed_joint: type fixed, parent l_foot, child l_sole_skin_15, origin xyz=0.1115831 0.0263973 0.0075 rpy=0 0 0
- added joint l_sole_skin_17_fixed_joint: type fixed, parent l_foot, child l_sole_skin_17, origin xyz=-0.0377192 0.0045384 0.0075 rpy=0 0 0
- added joint l_sole_skin_18_fixed_joint: type fixed, parent l_foot, child l_sole_skin_18, origin xyz=-0.0520767 -0.0083897 0.0075 rpy=0 0 0
- added joint l_sole_skin_19_fixed_joint: type fixed, parent l_foot, child l_sole_skin_19, origin xyz=-0.0480599 -0.027287 0.0075 rpy=0 0 0
- added joint l_sole_skin_1_fixed_joint: type fixed, parent l_foot, child l_sole_skin_1, origin xyz=0.0788511 0.0194399 0.0075 rpy=0 0 0
- added joint l_sole_skin_20_fixed_joint: type fixed, parent l_foot, child l_sole_skin_20, origin xyz=-0.0296855 -0.033258 0.0075 rpy=0 0 0
- added joint l_sole_skin_21_fixed_joint: type fixed, parent l_foot, child l_sole_skin_21, origin xyz=0.0277448 0.0184532 0.0075 rpy=0 0 0
- added joint l_sole_skin_22_fixed_joint: type fixed, parent l_foot, child l_sole_skin_22, origin xyz=0.0357785 -0.0193429 0.0075 rpy=0 0 0
- added joint l_sole_skin_24_fixed_joint: type fixed, parent l_foot, child l_sole_skin_24, origin xyz=0.0030465 -0.0263003 0.0075 rpy=0 0 0
- added joint l_sole_skin_25_fixed_joint: type fixed, parent l_foot, child l_sole_skin_25, origin xyz=0.0174041 -0.0133722 0.0075 rpy=0 0 0
- added joint l_sole_skin_26_fixed_joint: type fixed, parent l_foot, child l_sole_skin_26, origin xyz=0.0133872 0.0055251 0.0075 rpy=0 0 0
- added joint l_sole_skin_27_fixed_joint: type fixed, parent l_foot, child l_sole_skin_27, origin xyz=-0.0049872 0.0114958 0.0075 rpy=0 0 0
- added joint l_sole_skin_28_fixed_joint: type fixed, parent l_foot, child l_sole_skin_28, origin xyz=-0.0193448 -0.0014323 0.0075 rpy=0 0 0
- added joint l_sole_skin_29_fixed_joint: type fixed, parent l_foot, child l_sole_skin_29, origin xyz=-0.0153279 -0.0203296 0.0075 rpy=0 0 0
- added joint l_sole_skin_2_fixed_joint: type fixed, parent l_foot, child l_sole_skin_2, origin xyz=0.0604767 0.0254106 0.0075 rpy=0 0 0
- added joint l_sole_skin_3_fixed_joint: type fixed, parent l_foot, child l_sole_skin_3, origin xyz=0.04611917 0.0124825 0.0075 rpy=0 0 0
- added joint l_sole_skin_4_fixed_joint: type fixed, parent l_foot, child l_sole_skin_4, origin xyz=0.05013603 -0.0064148 0.0075 rpy=0 0 0
- added joint l_sole_skin_8_fixed_joint: type fixed, parent l_foot, child l_sole_skin_8, origin xyz=0.0725273 -0.031283 0.0075 rpy=0 0 0
- added joint l_sole_skin_9_fixed_joint: type fixed, parent l_foot, child l_sole_skin_9, origin xyz=0.0909017 -0.037254 0.0075 rpy=0 0 0
- added joint r_sole_skin_0_fixed_joint: type fixed, parent r_foot, child r_sole_skin_0, origin xyz=0.0604767 -0.0254106 0.0075 rpy=0 0 0
- added joint r_sole_skin_10_fixed_joint: type fixed, parent r_foot, child r_sole_skin_10, origin xyz=0.0725273 0.031283 0.0075 rpy=0 0 0
- added joint r_sole_skin_11_fixed_joint: type fixed, parent r_foot, child r_sole_skin_11, origin xyz=0.0685104 0.012385 0.0075 rpy=0 0 0
- added joint r_sole_skin_12_fixed_joint: type fixed, parent r_foot, child r_sole_skin_12, origin xyz=0.082868 -0.0005426 0.0075 rpy=0 0 0
- added joint r_sole_skin_13_fixed_joint: type fixed, parent r_foot, child r_sole_skin_13, origin xyz=0.1012424 0.0054276 0.0075 rpy=0 0 0
- added joint r_sole_skin_14_fixed_joint: type fixed, parent r_foot, child r_sole_skin_14, origin xyz=0.05013603 0.0064148 0.0075 rpy=0 0 0
- added joint r_sole_skin_15_fixed_joint: type fixed, parent r_foot, child r_sole_skin_15, origin xyz=0.04611917 -0.012483 0.0075 rpy=0 0 0
- added joint r_sole_skin_17_fixed_joint: type fixed, parent r_foot, child r_sole_skin_17, origin xyz=-0.0296855 0.033257 0.0075 rpy=0 0 0
- added joint r_sole_skin_18_fixed_joint: type fixed, parent r_foot, child r_sole_skin_18, origin xyz=-0.0480599 0.027287 0.0075 rpy=0 0 0
- added joint r_sole_skin_19_fixed_joint: type fixed, parent r_foot, child r_sole_skin_19, origin xyz=-0.0520767 0.0083892 0.0075 rpy=0 0 0
- added joint r_sole_skin_1_fixed_joint: type fixed, parent r_foot, child r_sole_skin_1, origin xyz=0.0788511 -0.0194404 0.0075 rpy=0 0 0
- added joint r_sole_skin_20_fixed_joint: type fixed, parent r_foot, child r_sole_skin_20, origin xyz=-0.0377192 -0.0045384 0.0075 rpy=0 0 0
- added joint r_sole_skin_21_fixed_joint: type fixed, parent r_foot, child r_sole_skin_21, origin xyz=0.0357785 0.0193424 0.0075 rpy=0 0 0
- added joint r_sole_skin_22_fixed_joint: type fixed, parent r_foot, child r_sole_skin_22, origin xyz=0.0277448 -0.0184532 0.0075 rpy=0 0 0
- added joint r_sole_skin_24_fixed_joint: type fixed, parent r_foot, child r_sole_skin_24, origin xyz=-0.0049872 -0.0114958 0.0075 rpy=0 0 0
- added joint r_sole_skin_25_fixed_joint: type fixed, parent r_foot, child r_sole_skin_25, origin xyz=0.0133872 -0.0055256 0.0075 rpy=0 0 0
- added joint r_sole_skin_26_fixed_joint: type fixed, parent r_foot, child r_sole_skin_26, origin xyz=0.0174041 0.0133722 0.0075 rpy=0 0 0
- added joint r_sole_skin_27_fixed_joint: type fixed, parent r_foot, child r_sole_skin_27, origin xyz=0.0030465 0.0262998 0.0075 rpy=0 0 0
- added joint r_sole_skin_28_fixed_joint: type fixed, parent r_foot, child r_sole_skin_28, origin xyz=-0.0153279 0.0203296 0.0075 rpy=0 0 0
- added joint r_sole_skin_29_fixed_joint: type fixed, parent r_foot, child r_sole_skin_29, origin xyz=-0.0193448 0.0014318 0.0075 rpy=0 0 0
- added joint r_sole_skin_2_fixed_joint: type fixed, parent r_foot, child r_sole_skin_2, origin xyz=0.0932087 -0.032368 0.0075 rpy=0 0 0
- added joint r_sole_skin_3_fixed_joint: type fixed, parent r_foot, child r_sole_skin_3, origin xyz=0.1115831 -0.0263978 0.0075 rpy=0 0 0
- added joint r_sole_skin_4_fixed_joint: type fixed, parent r_foot, child r_sole_skin_4, origin xyz=0.1156 -0.0075 0.0075 rpy=0 0 0
- added joint r_sole_skin_8_fixed_joint: type fixed, parent r_foot, child r_sole_skin_8, origin xyz=0.1052593 0.0243254 0.0075 rpy=0 0 0
- added joint r_sole_skin_9_fixed_joint: type fixed, parent r_foot, child r_sole_skin_9, origin xyz=0.0909017 0.037253 0.0075 rpy=0 0 0

File: iCub/robots/iCubGazeboV2_5/model.urdf (robot description, URDF)
Before this commit: robot iCub, 139 links, 138 joints
Links:
- added link l_sole_skin_0
- added link l_sole_skin_1
- added link l_sole_skin_10
- added link l_sole_skin_11
- added link l_sole_skin_12
- added link l_sole_skin_13
- added link l_sole_skin_14
- added link l_sole_skin_15
- added link l_sole_skin_17
- added link l_sole_skin_18
- added link l_sole_skin_19
- added link l_sole_skin_2
- added link l_sole_skin_20
- added link l_sole_skin_21
- added link l_sole_skin_22
- added link l_sole_skin_24
- added link l_sole_skin_25
- added link l_sole_skin_26
- added link l_sole_skin_27
- added link l_sole_skin_28
- added link l_sole_skin_29
- added link l_sole_skin_3
- added link l_sole_skin_4
- added link l_sole_skin_8
- added link l_sole_skin_9
- added link r_sole_skin_0
- added link r_sole_skin_1
- added link r_sole_skin_10
- added link r_sole_skin_11
- added link r_sole_skin_12
- added link r_sole_skin_13
- added link r_sole_skin_14
- added link r_sole_skin_15
- added link r_sole_skin_17
- added link r_sole_skin_18
- added link r_sole_skin_19
- added link r_sole_skin_2
- added link r_sole_skin_20
- added link r_sole_skin_21
- added link r_sole_skin_22
- added link r_sole_skin_24
- added link r_sole_skin_25
- added link r_sole_skin_26
- added link r_sole_skin_27
- added link r_sole_skin_28
- added link r_sole_skin_29
- added link r_sole_skin_3
- added link r_sole_skin_4
- added link r_sole_skin_8
- added link r_sole_skin_9
Joints:
- added joint l_sole_skin_0_fixed_joint: type fixed, parent l_foot, child l_sole_skin_0, origin xyz=0.0932087 0.032368 0.0075 rpy=0 0 0
- added joint l_sole_skin_10_fixed_joint: type fixed, parent l_foot, child l_sole_skin_10, origin xyz=0.1052593 -0.0243254 0.0075 rpy=0 0 0
- added joint l_sole_skin_11_fixed_joint: type fixed, parent l_foot, child l_sole_skin_11, origin xyz=0.1012424 -0.0054281 0.0075 rpy=0 0 0
- added joint l_sole_skin_12_fixed_joint: type fixed, parent l_foot, child l_sole_skin_12, origin xyz=0.082868 0.0005426 0.0075 rpy=0 0 0
- added joint l_sole_skin_13_fixed_joint: type fixed, parent l_foot, child l_sole_skin_13, origin xyz=0.0685104 -0.0123855 0.0075 rpy=0 0 0
- added joint l_sole_skin_14_fixed_joint: type fixed, parent l_foot, child l_sole_skin_14, origin xyz=0.1156 0.0074995 0.0075 rpy=0 0 0
- added joint l_sole_skin_15_fixed_joint: type fixed, parent l_foot, child l_sole_skin_15, origin xyz=0.1115831 0.0263973 0.0075 rpy=0 0 0
- added joint l_sole_skin_17_fixed_joint: type fixed, parent l_foot, child l_sole_skin_17, origin xyz=-0.0377192 0.0045384 0.0075 rpy=0 0 0
- added joint l_sole_skin_18_fixed_joint: type fixed, parent l_foot, child l_sole_skin_18, origin xyz=-0.0520767 -0.0083897 0.0075 rpy=0 0 0
- added joint l_sole_skin_19_fixed_joint: type fixed, parent l_foot, child l_sole_skin_19, origin xyz=-0.0480599 -0.027287 0.0075 rpy=0 0 0
- added joint l_sole_skin_1_fixed_joint: type fixed, parent l_foot, child l_sole_skin_1, origin xyz=0.0788511 0.0194399 0.0075 rpy=0 0 0
- added joint l_sole_skin_20_fixed_joint: type fixed, parent l_foot, child l_sole_skin_20, origin xyz=-0.0296855 -0.033258 0.0075 rpy=0 0 0
- added joint l_sole_skin_21_fixed_joint: type fixed, parent l_foot, child l_sole_skin_21, origin xyz=0.0277448 0.0184532 0.0075 rpy=0 0 0
- added joint l_sole_skin_22_fixed_joint: type fixed, parent l_foot, child l_sole_skin_22, origin xyz=0.0357785 -0.0193429 0.0075 rpy=0 0 0
- added joint l_sole_skin_24_fixed_joint: type fixed, parent l_foot, child l_sole_skin_24, origin xyz=0.0030465 -0.0263003 0.0075 rpy=0 0 0
- added joint l_sole_skin_25_fixed_joint: type fixed, parent l_foot, child l_sole_skin_25, origin xyz=0.0174041 -0.0133722 0.0075 rpy=0 0 0
- added joint l_sole_skin_26_fixed_joint: type fixed, parent l_foot, child l_sole_skin_26, origin xyz=0.0133872 0.0055251 0.0075 rpy=0 0 0
- added joint l_sole_skin_27_fixed_joint: type fixed, parent l_foot, child l_sole_skin_27, origin xyz=-0.0049872 0.0114958 0.0075 rpy=0 0 0
- added joint l_sole_skin_28_fixed_joint: type fixed, parent l_foot, child l_sole_skin_28, origin xyz=-0.0193448 -0.0014323 0.0075 rpy=0 0 0
- added joint l_sole_skin_29_fixed_joint: type fixed, parent l_foot, child l_sole_skin_29, origin xyz=-0.0153279 -0.0203296 0.0075 rpy=0 0 0
- added joint l_sole_skin_2_fixed_joint: type fixed, parent l_foot, child l_sole_skin_2, origin xyz=0.0604767 0.0254106 0.0075 rpy=0 0 0
- added joint l_sole_skin_3_fixed_joint: type fixed, parent l_foot, child l_sole_skin_3, origin xyz=0.04611917 0.0124825 0.0075 rpy=0 0 0
- added joint l_sole_skin_4_fixed_joint: type fixed, parent l_foot, child l_sole_skin_4, origin xyz=0.05013603 -0.0064148 0.0075 rpy=0 0 0
- added joint l_sole_skin_8_fixed_joint: type fixed, parent l_foot, child l_sole_skin_8, origin xyz=0.0725273 -0.031283 0.0075 rpy=0 0 0
- added joint l_sole_skin_9_fixed_joint: type fixed, parent l_foot, child l_sole_skin_9, origin xyz=0.0909017 -0.037254 0.0075 rpy=0 0 0
- added joint r_sole_skin_0_fixed_joint: type fixed, parent r_foot, child r_sole_skin_0, origin xyz=0.0604767 -0.0254106 0.0075 rpy=0 0 0
- added joint r_sole_skin_10_fixed_joint: type fixed, parent r_foot, child r_sole_skin_10, origin xyz=0.0725273 0.031283 0.0075 rpy=0 0 0
- added joint r_sole_skin_11_fixed_joint: type fixed, parent r_foot, child r_sole_skin_11, origin xyz=0.0685104 0.012385 0.0075 rpy=0 0 0
- added joint r_sole_skin_12_fixed_joint: type fixed, parent r_foot, child r_sole_skin_12, origin xyz=0.082868 -0.0005426 0.0075 rpy=0 0 0
- added joint r_sole_skin_13_fixed_joint: type fixed, parent r_foot, child r_sole_skin_13, origin xyz=0.1012424 0.0054276 0.0075 rpy=0 0 0
- added joint r_sole_skin_14_fixed_joint: type fixed, parent r_foot, child r_sole_skin_14, origin xyz=0.05013603 0.0064148 0.0075 rpy=0 0 0
- added joint r_sole_skin_15_fixed_joint: type fixed, parent r_foot, child r_sole_skin_15, origin xyz=0.04611917 -0.012483 0.0075 rpy=0 0 0
- added joint r_sole_skin_17_fixed_joint: type fixed, parent r_foot, child r_sole_skin_17, origin xyz=-0.0296855 0.033257 0.0075 rpy=0 0 0
- added joint r_sole_skin_18_fixed_joint: type fixed, parent r_foot, child r_sole_skin_18, origin xyz=-0.0480599 0.027287 0.0075 rpy=0 0 0
- added joint r_sole_skin_19_fixed_joint: type fixed, parent r_foot, child r_sole_skin_19, origin xyz=-0.0520767 0.0083892 0.0075 rpy=0 0 0
- added joint r_sole_skin_1_fixed_joint: type fixed, parent r_foot, child r_sole_skin_1, origin xyz=0.0788511 -0.0194404 0.0075 rpy=0 0 0
- added joint r_sole_skin_20_fixed_joint: type fixed, parent r_foot, child r_sole_skin_20, origin xyz=-0.0377192 -0.0045384 0.0075 rpy=0 0 0
- added joint r_sole_skin_21_fixed_joint: type fixed, parent r_foot, child r_sole_skin_21, origin xyz=0.0357785 0.0193424 0.0075 rpy=0 0 0
- added joint r_sole_skin_22_fixed_joint: type fixed, parent r_foot, child r_sole_skin_22, origin xyz=0.0277448 -0.0184532 0.0075 rpy=0 0 0
- added joint r_sole_skin_24_fixed_joint: type fixed, parent r_foot, child r_sole_skin_24, origin xyz=-0.0049872 -0.0114958 0.0075 rpy=0 0 0
- added joint r_sole_skin_25_fixed_joint: type fixed, parent r_foot, child r_sole_skin_25, origin xyz=0.0133872 -0.0055256 0.0075 rpy=0 0 0
- added joint r_sole_skin_26_fixed_joint: type fixed, parent r_foot, child r_sole_skin_26, origin xyz=0.0174041 0.0133722 0.0075 rpy=0 0 0
- added joint r_sole_skin_27_fixed_joint: type fixed, parent r_foot, child r_sole_skin_27, origin xyz=0.0030465 0.0262998 0.0075 rpy=0 0 0
- added joint r_sole_skin_28_fixed_joint: type fixed, parent r_foot, child r_sole_skin_28, origin xyz=-0.0153279 0.0203296 0.0075 rpy=0 0 0
- added joint r_sole_skin_29_fixed_joint: type fixed, parent r_foot, child r_sole_skin_29, origin xyz=-0.0193448 0.0014318 0.0075 rpy=0 0 0
- added joint r_sole_skin_2_fixed_joint: type fixed, parent r_foot, child r_sole_skin_2, origin xyz=0.0932087 -0.032368 0.0075 rpy=0 0 0
- added joint r_sole_skin_3_fixed_joint: type fixed, parent r_foot, child r_sole_skin_3, origin xyz=0.1115831 -0.0263978 0.0075 rpy=0 0 0
- added joint r_sole_skin_4_fixed_joint: type fixed, parent r_foot, child r_sole_skin_4, origin xyz=0.1156 -0.0075 0.0075 rpy=0 0 0
- added joint r_sole_skin_8_fixed_joint: type fixed, parent r_foot, child r_sole_skin_8, origin xyz=0.1052593 0.0243254 0.0075 rpy=0 0 0
- added joint r_sole_skin_9_fixed_joint: type fixed, parent r_foot, child r_sole_skin_9, origin xyz=0.0909017 0.037253 0.0075 rpy=0 0 0
