Commit message: Automatic build. Travis build:294
icub-model-generator commit:3d61348ded9390e7d0e31057ebd09f8f439f7357

urdf_parser_py commit:31474b9baaf7c3845b40e5a9aa87d5900a2282c3

simmechanics-to-urdf commit:1bd48b2d02b1d155a782f35d96865753c2e49706

yarp commit:48613af088ab5b3c41ddd6def6afaea0dd179b20

icub-main commit:439b12855b73275459540f263ec28cae09c9ee19

idyntree commit:40ba1b919b5f730faf597cc4237b492d03f45708

File: iCub/robots/iCubDarmstadt01/model.urdf (robot description, URDF)
Before this commit: robot iCub, 189 links, 188 joints
Links:
- link l_ankle_2: mass 0.267485 -> 0.265122
- link l_hip_2: mass 0.421106 -> 0.415987
- link r_ankle_2: mass 0.267485 -> 0.265122
- link r_hip_2: mass 0.418361 -> 0.413242
Joints:
- joint l_leg_ft_sensor: origin xyz=-0.0008575 0 -0.0743 rpy=3.14159265359 0 0 -> xyz=-0.0008302 7.52e-05 -0.0743 rpy=3.14159265359 0 0
- joint l_sole_skin_0_fixed_joint: origin xyz=0.0932087 0.032368 0.0075 rpy=0 0 0 -> xyz=0.0932088 0.032368 0.0075 rpy=0 0 0
- joint l_sole_skin_11_fixed_joint: origin xyz=0.1012424 -0.0054281 0.0075 rpy=0 0 0 -> xyz=0.1012425 -0.0054281 0.0075 rpy=0 0 0
- joint l_sole_skin_12_fixed_joint: origin xyz=0.082868 0.0005426 0.0075 rpy=0 0 0 -> xyz=0.0828681 0.0005426 0.0075 rpy=0 0 0
- joint l_sole_skin_13_fixed_joint: origin xyz=0.0685104 -0.0123855 0.0075 rpy=0 0 0 -> xyz=0.0685105 -0.0123855 0.0075 rpy=0 0 0
- joint l_sole_skin_15_fixed_joint: origin xyz=0.1115831 0.0263973 0.0075 rpy=0 0 0 -> xyz=0.1115832 0.0263973 0.0075 rpy=0 0 0
- joint l_sole_skin_17_fixed_joint: origin xyz=-0.0377192 0.0045384 0.0075 rpy=0 0 0 -> xyz=-0.0377191 0.0045385 0.0075 rpy=0 0 0
- joint l_sole_skin_19_fixed_joint: origin xyz=-0.0480599 -0.027287 0.0075 rpy=0 0 0 -> xyz=-0.0480598 -0.027287 0.0075 rpy=0 0 0
- joint l_sole_skin_1_fixed_joint: origin xyz=0.0788511 0.0194399 0.0075 rpy=0 0 0 -> xyz=0.0788512 0.0194399 0.0075 rpy=0 0 0
- joint l_sole_skin_20_fixed_joint: origin xyz=-0.0296855 -0.033258 0.0075 rpy=0 0 0 -> xyz=-0.0296854 -0.0332578 0.0075 rpy=0 0 0
- joint l_sole_skin_21_fixed_joint: origin xyz=0.0277448 0.0184532 0.0075 rpy=0 0 0 -> xyz=0.0277448 0.0184533 0.0075 rpy=0 0 0
- joint l_sole_skin_24_fixed_joint: origin xyz=0.0030465 -0.0263003 0.0075 rpy=0 0 0 -> xyz=0.0030466 -0.0263003 0.0075 rpy=0 0 0
- joint l_sole_skin_26_fixed_joint: origin xyz=0.0133872 0.0055251 0.0075 rpy=0 0 0 -> xyz=0.0133873 0.0055251 0.0075 rpy=0 0 0
- joint l_sole_skin_27_fixed_joint: origin xyz=-0.0049872 0.0114958 0.0075 rpy=0 0 0 -> xyz=-0.0049871 0.0114959 0.0075 rpy=0 0 0
- joint l_sole_skin_28_fixed_joint: origin xyz=-0.0193448 -0.0014323 0.0075 rpy=0 0 0 -> xyz=-0.0193447 -0.0014323 0.0075 rpy=0 0 0
- joint l_sole_skin_2_fixed_joint: origin xyz=0.0604767 0.0254106 0.0075 rpy=0 0 0 -> xyz=0.0604768 0.0254106 0.0075 rpy=0 0 0
- joint l_sole_skin_3_fixed_joint: origin xyz=0.04611917 0.0124825 0.0075 rpy=0 0 0 -> xyz=0.04611923 0.0124825 0.0075 rpy=0 0 0
- joint l_sole_skin_4_fixed_joint: origin xyz=0.05013603 -0.0064148 0.0075 rpy=0 0 0 -> xyz=0.05013609 -0.0064148 0.0075 rpy=0 0 0
- joint l_sole_skin_8_fixed_joint: origin xyz=0.0725273 -0.031283 0.0075 rpy=0 0 0 -> xyz=0.0725274 -0.0312828 0.0075 rpy=0 0 0
- joint l_sole_skin_9_fixed_joint: origin xyz=0.0909017 -0.037254 0.0075 rpy=0 0 0 -> xyz=0.0909018 -0.0372538 0.0075 rpy=0 0 0
- joint r_leg_ft_sensor: origin xyz=-0.0008575 0 -0.0743 rpy=3.14159265359 0 0 -> xyz=-0.0009363 1.39e-05 -0.0743 rpy=3.14159265359 0 0
- joint r_lower_leg_skin_0_fixed_joint: origin xyz=0.0544117 -0.031214 -0.002634 rpy=2.09173809157e-06 -1.41530676247 2.48648458622 -> xyz=0.0544117 -0.0312149 -0.002634 rpy=2.09173809157e-06 -1.41530676247 2.48648458622
- joint r_lower_leg_skin_14_fixed_joint: origin xyz=0.0550477 -0.031176 -0.0219 rpy=-3.14159181885 -1.46502735635 -0.654033407167 -> xyz=0.0550477 -0.0311759 -0.0219 rpy=-3.14159181885 -1.46502735635 -0.654033407167
- joint r_lower_leg_skin_16_fixed_joint: origin xyz=0.0272875 -0.050287 -0.004549 rpy=1.33075915123e-05 -1.53260853515 1.96280242835 -> xyz=0.0272876 -0.0502869 -0.004549 rpy=1.33075915123e-05 -1.53260853515 1.96280242835
- joint r_lower_leg_skin_17_fixed_joint: origin xyz=0.027875 -0.050312 -0.023882 rpy=-3.1415645262 -1.56366240237 -1.18022508756 -> xyz=0.027875 -0.0503119 -0.023882 rpy=-3.1415645262 -1.56366240237 -1.18022508756
- joint r_lower_leg_skin_19_fixed_joint: origin xyz=0.0357534 0.0410628 0.006065 rpy=-8.90877717426e-07 -1.43498696978 -2.15863618017 -> xyz=0.03575341 0.0410628 0.006065 rpy=-8.90877717426e-07 -1.43498696978 -2.15863618017
- joint r_lower_leg_skin_28_fixed_joint: origin xyz=0.04087215 -0.04244 -0.032756 rpy=3.14158088865 -1.52252462169 -0.929681029763 -> xyz=0.04087216 -0.0424399 -0.032756 rpy=3.14158088865 -1.52252462169 -0.929681029763
- joint r_lower_leg_skin_29_fixed_joint: origin xyz=0.03846637 -0.043516 -0.05242 rpy=3.14158017044 -1.53429841563 -0.915436346631 -> xyz=0.03846638 -0.0435159 -0.05242 rpy=3.14158017044 -1.53429841563 -0.915436346631
- joint r_lower_leg_skin_31_fixed_joint: origin xyz=0.03914638 -0.042271 0.006327 rpy=-6.58381747139e-07 -1.4186494462 2.20853032986 -> xyz=0.0391464 -0.0422709 0.006327 rpy=-6.58381747139e-07 -1.4186494462 2.20853032986
- joint r_lower_leg_skin_32_fixed_joint: origin xyz=0.04598301 0.0325847 -0.080733 rpy=-3.14159014988 -1.52238289798 0.645940380887 -> xyz=0.04598303 0.0325847 -0.080733 rpy=-3.14159014988 -1.52238289798 0.645940380887
- joint r_lower_leg_skin_35_fixed_joint: origin xyz=0.04774866 -0.031232 -0.080113 rpy=-3.14158668275 -1.51758467332 -0.541532486468 -> xyz=0.04774868 -0.0312319 -0.080113 rpy=-3.14158668275 -1.51758467332 -0.541532486468
- joint r_lower_leg_skin_36_fixed_joint: origin xyz=0.05322409 -0.0156018 -0.088362 rpy=-3.14159034144 -1.51587265281 -0.20740733566 -> xyz=0.0532241 -0.0156018 -0.088362 rpy=-3.14159034144 -1.51587265281 -0.20740733566
- joint r_lower_leg_skin_38_fixed_joint: origin xyz=0.04880467 -0.031263 -0.060757 rpy=3.14158665199 -1.5157299554 -0.54215359959 -> xyz=0.04880469 -0.0312629 -0.060757 rpy=3.14158665199 -1.5157299554 -0.54215359959
- joint r_lower_leg_skin_3_fixed_joint: origin xyz=0.05157878 0.0304205 -0.002843 rpy=0 -1.42951054083 -2.30391484186 -> xyz=0.05157879 0.0304205 -0.002843 rpy=0 -1.42951054083 -2.30391484186
- joint r_lower_leg_skin_43_fixed_joint: origin xyz=0.04712542 0.0323653 -0.061362 rpy=-3.14159136621 -1.53843038237 0.624217523667 -> xyz=0.04712544 0.0323653 -0.061362 rpy=-3.14159136621 -1.53843038237 0.624217523667
- joint r_lower_leg_skin_46_fixed_joint: origin xyz=0.0558156 0.0172164 -0.05018 rpy=-3.14158987809 -1.42759881603 0.325607710876 -> xyz=0.0558157 0.0172164 -0.05018 rpy=-3.14158987809 -1.42759881603 0.325607710876
- joint r_lower_leg_skin_47_fixed_joint: origin xyz=0.05264163 0.0176389 -0.08886 rpy=3.14158963519 -1.51690559406 0.262640425058 -> xyz=0.05264165 0.0176388 -0.08886 rpy=3.14158963519 -1.51690559406 0.262640425058
- joint r_lower_leg_skin_49_fixed_joint: origin xyz=0.04113137 0.0324385 -0.138859 rpy=-3.14158934751 -1.48996135695 0.729763592113 -> xyz=0.04113139 0.0324385 -0.138859 rpy=-3.14158934751 -1.48996135695 0.729763592113
- joint r_lower_leg_skin_50_fixed_joint: origin xyz=0.043016947 0.0325273 -0.119469 rpy=3.14159069596 -1.49900732636 0.695784020081 -> xyz=0.043016963 0.0325273 -0.119469 rpy=3.14159069596 -1.49900732636 0.695784020081
- joint r_lower_leg_skin_51_fixed_joint: origin xyz=0.05141583 0.017759 -0.108206 rpy=-3.14158890179 -1.50628475717 0.272079935713 -> xyz=0.05141584 0.017759 -0.108206 rpy=-3.14158890179 -1.50628475717 0.272079935713
- joint r_lower_leg_skin_52_fixed_joint: origin xyz=0.05299832 0.0012664 -0.116895 rpy=-3.14159164042 -1.50318674421 0.0108717260994 -> xyz=0.05299834 0.0012664 -0.116895 rpy=-3.14159164042 -1.50318674421 0.0108717260994
- joint r_lower_leg_skin_53_fixed_joint: origin xyz=0.05207312 -0.0154339 -0.107654 rpy=3.14159063987 -1.50595307447 -0.211407322892 -> xyz=0.05207314 -0.0154339 -0.107654 rpy=3.14159063987 -1.50595307447 -0.211407322892
- joint r_lower_leg_skin_54_fixed_joint: origin xyz=0.04512708 -0.030749 -0.118787 rpy=3.14158825193 -1.49745145571 -0.575115374473 -> xyz=0.0451271 -0.0307489 -0.118787 rpy=3.14158825193 -1.49745145571 -0.575115374473
- joint r_lower_leg_skin_55_fixed_joint: origin xyz=0.043502663 -0.030489 -0.138143 rpy=3.14158906486 -1.48995787038 -0.597219943789 -> xyz=0.043502679 -0.0304889 -0.138143 rpy=3.14158906486 -1.48995787038 -0.597219943789
- joint r_lower_leg_skin_56_fixed_joint: origin xyz=0.04926839 -0.015121 -0.146218 rpy=-3.14158920404 -1.49124819828 -0.2234844764 -> xyz=0.04926841 -0.015121 -0.146218 rpy=-3.14158920404 -1.49124819828 -0.2234844764
- joint r_lower_leg_skin_5_fixed_joint: origin xyz=0.0636503 0.0003094 -0.001972 rpy=0 -1.38652215068 -3.14147169807 -> xyz=0.0636504 0.0003094 -0.001972 rpy=0 -1.38652215068 -3.14147169807
- joint r_lower_leg_skin_60_fixed_joint: origin xyz=0.04836967 0.018056 -0.146938 rpy=-3.14159173337 -1.48985968527 0.302951871954 -> xyz=0.04836968 0.018056 -0.146938 rpy=-3.14159173337 -1.48985968527 0.302951871954
- joint r_lower_leg_skin_61_fixed_joint: origin xyz=0.05161952 0.0014266 -0.136169 rpy=-3.14159100925 -1.49602097086 0.0132014275205 -> xyz=0.05161954 0.0014266 -0.136169 rpy=-3.14159100925 -1.49602097086 0.0132014275205
- joint r_lower_leg_skin_6_fixed_joint: origin xyz=0.05208552 0.0304434 -0.022149 rpy=-3.14158927953 -1.46785123411 0.837492889077 -> xyz=0.05208554 0.0304434 -0.022149 rpy=-3.14158927953 -1.46785123411 0.837492889077
- joint r_lower_leg_skin_9_fixed_joint: origin xyz=0.0598214 0.0167973 -0.030962 rpy=-3.14159202356 -1.34224755325 0.379294477718 -> xyz=0.0598214 0.0167972 -0.030962 rpy=-3.14159202356 -1.34224755325 0.379294477718
- joint r_sole_skin_10_fixed_joint: origin xyz=0.0725273 0.031283 0.0075 rpy=0 0 0 -> xyz=0.0725273 0.0312829 0.0075 rpy=0 0 0
- joint r_sole_skin_11_fixed_joint: origin xyz=0.0685104 0.012385 0.0075 rpy=0 0 0 -> xyz=0.0685105 0.012385 0.0075 rpy=0 0 0
- joint r_sole_skin_14_fixed_joint: origin xyz=0.05013603 0.0064148 0.0075 rpy=0 0 0 -> xyz=0.05013604 0.0064148 0.0075 rpy=0 0 0
- joint r_sole_skin_15_fixed_joint: origin xyz=0.04611917 -0.012483 0.0075 rpy=0 0 0 -> xyz=0.04611919 -0.012483 0.0075 rpy=0 0 0
- joint r_sole_skin_17_fixed_joint: origin xyz=-0.0296855 0.033257 0.0075 rpy=0 0 0 -> xyz=-0.0296855 0.0332569 0.0075 rpy=0 0 0
- joint r_sole_skin_1_fixed_joint: origin xyz=0.0788511 -0.0194404 0.0075 rpy=0 0 0 -> xyz=0.0788512 -0.0194404 0.0075 rpy=0 0 0
- joint r_sole_skin_9_fixed_joint: origin xyz=0.0909017 0.037253 0.0075 rpy=0 0 0 -> xyz=0.0909017 0.0372529 0.0075 rpy=0 0 0
- joint r_upper_leg_back_contact_fixed_joint: origin xyz=-0.0511999 0 0.0146 rpy=0 1.57079632679 0 -> xyz=-0.0511998 0 0.0146 rpy=0 1.57079632679 0

File: iCub/robots/iCubGazeboV2_5/model.urdf (robot description, URDF)
Before this commit: robot iCub, 189 links, 188 joints
Links:
- link l_ankle_2: mass 0.267485 -> 0.265122
- link l_hip_2: mass 0.421106 -> 0.415987
- link r_ankle_2: mass 0.267485 -> 0.265122
- link r_hip_2: mass 0.418361 -> 0.413242
Joints:
- joint l_leg_ft_sensor: origin xyz=-0.0008575 0 -0.0743 rpy=3.14159265359 0 0 -> xyz=-0.0008302 7.52e-05 -0.0743 rpy=3.14159265359 0 0
- joint l_sole_skin_0_fixed_joint: origin xyz=0.0932087 0.032368 0.0075 rpy=0 0 0 -> xyz=0.0932088 0.032368 0.0075 rpy=0 0 0
- joint l_sole_skin_11_fixed_joint: origin xyz=0.1012424 -0.0054281 0.0075 rpy=0 0 0 -> xyz=0.1012425 -0.0054281 0.0075 rpy=0 0 0
- joint l_sole_skin_12_fixed_joint: origin xyz=0.082868 0.0005426 0.0075 rpy=0 0 0 -> xyz=0.0828681 0.0005426 0.0075 rpy=0 0 0
- joint l_sole_skin_13_fixed_joint: origin xyz=0.0685104 -0.0123855 0.0075 rpy=0 0 0 -> xyz=0.0685105 -0.0123855 0.0075 rpy=0 0 0
- joint l_sole_skin_15_fixed_joint: origin xyz=0.1115831 0.0263973 0.0075 rpy=0 0 0 -> xyz=0.1115832 0.0263973 0.0075 rpy=0 0 0
- joint l_sole_skin_17_fixed_joint: origin xyz=-0.0377192 0.0045384 0.0075 rpy=0 0 0 -> xyz=-0.0377191 0.0045385 0.0075 rpy=0 0 0
- joint l_sole_skin_19_fixed_joint: origin xyz=-0.0480599 -0.027287 0.0075 rpy=0 0 0 -> xyz=-0.0480598 -0.027287 0.0075 rpy=0 0 0
- joint l_sole_skin_1_fixed_joint: origin xyz=0.0788511 0.0194399 0.0075 rpy=0 0 0 -> xyz=0.0788512 0.0194399 0.0075 rpy=0 0 0
- joint l_sole_skin_20_fixed_joint: origin xyz=-0.0296855 -0.033258 0.0075 rpy=0 0 0 -> xyz=-0.0296854 -0.0332578 0.0075 rpy=0 0 0
- joint l_sole_skin_21_fixed_joint: origin xyz=0.0277448 0.0184532 0.0075 rpy=0 0 0 -> xyz=0.0277448 0.0184533 0.0075 rpy=0 0 0
- joint l_sole_skin_24_fixed_joint: origin xyz=0.0030465 -0.0263003 0.0075 rpy=0 0 0 -> xyz=0.0030466 -0.0263003 0.0075 rpy=0 0 0
- joint l_sole_skin_26_fixed_joint: origin xyz=0.0133872 0.0055251 0.0075 rpy=0 0 0 -> xyz=0.0133873 0.0055251 0.0075 rpy=0 0 0
- joint l_sole_skin_27_fixed_joint: origin xyz=-0.0049872 0.0114958 0.0075 rpy=0 0 0 -> xyz=-0.0049871 0.0114959 0.0075 rpy=0 0 0
- joint l_sole_skin_28_fixed_joint: origin xyz=-0.0193448 -0.0014323 0.0075 rpy=0 0 0 -> xyz=-0.0193447 -0.0014323 0.0075 rpy=0 0 0
- joint l_sole_skin_2_fixed_joint: origin xyz=0.0604767 0.0254106 0.0075 rpy=0 0 0 -> xyz=0.0604768 0.0254106 0.0075 rpy=0 0 0
- joint l_sole_skin_3_fixed_joint: origin xyz=0.04611917 0.0124825 0.0075 rpy=0 0 0 -> xyz=0.04611923 0.0124825 0.0075 rpy=0 0 0
- joint l_sole_skin_4_fixed_joint: origin xyz=0.05013603 -0.0064148 0.0075 rpy=0 0 0 -> xyz=0.05013609 -0.0064148 0.0075 rpy=0 0 0
- joint l_sole_skin_8_fixed_joint: origin xyz=0.0725273 -0.031283 0.0075 rpy=0 0 0 -> xyz=0.0725274 -0.0312828 0.0075 rpy=0 0 0
- joint l_sole_skin_9_fixed_joint: origin xyz=0.0909017 -0.037254 0.0075 rpy=0 0 0 -> xyz=0.0909018 -0.0372538 0.0075 rpy=0 0 0
- joint r_leg_ft_sensor: origin xyz=-0.0008575 0 -0.0743 rpy=3.14159265359 0 0 -> xyz=-0.0009363 1.39e-05 -0.0743 rpy=3.14159265359 0 0
- joint r_lower_leg_skin_0_fixed_joint: origin xyz=0.0544117 -0.031214 -0.002634 rpy=2.09173809157e-06 -1.41530676247 2.48648458622 -> xyz=0.0544117 -0.0312149 -0.002634 rpy=2.09173809157e-06 -1.41530676247 2.48648458622
- joint r_lower_leg_skin_14_fixed_joint: origin xyz=0.0550477 -0.031176 -0.0219 rpy=-3.14159181885 -1.46502735635 -0.654033407167 -> xyz=0.0550477 -0.0311759 -0.0219 rpy=-3.14159181885 -1.46502735635 -0.654033407167
- joint r_lower_leg_skin_16_fixed_joint: origin xyz=0.0272875 -0.050287 -0.004549 rpy=1.33075915123e-05 -1.53260853515 1.96280242835 -> xyz=0.0272876 -0.0502869 -0.004549 rpy=1.33075915123e-05 -1.53260853515 1.96280242835
- joint r_lower_leg_skin_17_fixed_joint: origin xyz=0.027875 -0.050312 -0.023882 rpy=-3.1415645262 -1.56366240237 -1.18022508756 -> xyz=0.027875 -0.0503119 -0.023882 rpy=-3.1415645262 -1.56366240237 -1.18022508756
- joint r_lower_leg_skin_19_fixed_joint: origin xyz=0.0357534 0.0410628 0.006065 rpy=-8.90877717426e-07 -1.43498696978 -2.15863618017 -> xyz=0.03575341 0.0410628 0.006065 rpy=-8.90877717426e-07 -1.43498696978 -2.15863618017
- joint r_lower_leg_skin_28_fixed_joint: origin xyz=0.04087215 -0.04244 -0.032756 rpy=3.14158088865 -1.52252462169 -0.929681029763 -> xyz=0.04087216 -0.0424399 -0.032756 rpy=3.14158088865 -1.52252462169 -0.929681029763
- joint r_lower_leg_skin_29_fixed_joint: origin xyz=0.03846637 -0.043516 -0.05242 rpy=3.14158017044 -1.53429841563 -0.915436346631 -> xyz=0.03846638 -0.0435159 -0.05242 rpy=3.14158017044 -1.53429841563 -0.915436346631
- joint r_lower_leg_skin_31_fixed_joint: origin xyz=0.03914638 -0.042271 0.006327 rpy=-6.58381747139e-07 -1.4186494462 2.20853032986 -> xyz=0.0391464 -0.0422709 0.006327 rpy=-6.58381747139e-07 -1.4186494462 2.20853032986
- joint r_lower_leg_skin_32_fixed_joint: origin xyz=0.04598301 0.0325847 -0.080733 rpy=-3.14159014988 -1.52238289798 0.645940380887 -> xyz=0.04598303 0.0325847 -0.080733 rpy=-3.14159014988 -1.52238289798 0.645940380887
- joint r_lower_leg_skin_35_fixed_joint: origin xyz=0.04774866 -0.031232 -0.080113 rpy=-3.14158668275 -1.51758467332 -0.541532486468 -> xyz=0.04774868 -0.0312319 -0.080113 rpy=-3.14158668275 -1.51758467332 -0.541532486468
- joint r_lower_leg_skin_36_fixed_joint: origin xyz=0.05322409 -0.0156018 -0.088362 rpy=-3.14159034144 -1.51587265281 -0.20740733566 -> xyz=0.0532241 -0.0156018 -0.088362 rpy=-3.14159034144 -1.51587265281 -0.20740733566
- joint r_lower_leg_skin_38_fixed_joint: origin xyz=0.04880467 -0.031263 -0.060757 rpy=3.14158665199 -1.5157299554 -0.54215359959 -> xyz=0.04880469 -0.0312629 -0.060757 rpy=3.14158665199 -1.5157299554 -0.54215359959
- joint r_lower_leg_skin_3_fixed_joint: origin xyz=0.05157878 0.0304205 -0.002843 rpy=0 -1.42951054083 -2.30391484186 -> xyz=0.05157879 0.0304205 -0.002843 rpy=0 -1.42951054083 -2.30391484186
- joint r_lower_leg_skin_43_fixed_joint: origin xyz=0.04712542 0.0323653 -0.061362 rpy=-3.14159136621 -1.53843038237 0.624217523667 -> xyz=0.04712544 0.0323653 -0.061362 rpy=-3.14159136621 -1.53843038237 0.624217523667
- joint r_lower_leg_skin_46_fixed_joint: origin xyz=0.0558156 0.0172164 -0.05018 rpy=-3.14158987809 -1.42759881603 0.325607710876 -> xyz=0.0558157 0.0172164 -0.05018 rpy=-3.14158987809 -1.42759881603 0.325607710876
- joint r_lower_leg_skin_47_fixed_joint: origin xyz=0.05264163 0.0176389 -0.08886 rpy=3.14158963519 -1.51690559406 0.262640425058 -> xyz=0.05264165 0.0176388 -0.08886 rpy=3.14158963519 -1.51690559406 0.262640425058
- joint r_lower_leg_skin_49_fixed_joint: origin xyz=0.04113137 0.0324385 -0.138859 rpy=-3.14158934751 -1.48996135695 0.729763592113 -> xyz=0.04113139 0.0324385 -0.138859 rpy=-3.14158934751 -1.48996135695 0.729763592113
- joint r_lower_leg_skin_50_fixed_joint: origin xyz=0.043016947 0.0325273 -0.119469 rpy=3.14159069596 -1.49900732636 0.695784020081 -> xyz=0.043016963 0.0325273 -0.119469 rpy=3.14159069596 -1.49900732636 0.695784020081
- joint r_lower_leg_skin_51_fixed_joint: origin xyz=0.05141583 0.017759 -0.108206 rpy=-3.14158890179 -1.50628475717 0.272079935713 -> xyz=0.05141584 0.017759 -0.108206 rpy=-3.14158890179 -1.50628475717 0.272079935713
- joint r_lower_leg_skin_52_fixed_joint: origin xyz=0.05299832 0.0012664 -0.116895 rpy=-3.14159164042 -1.50318674421 0.0108717260994 -> xyz=0.05299834 0.0012664 -0.116895 rpy=-3.14159164042 -1.50318674421 0.0108717260994
- joint r_lower_leg_skin_53_fixed_joint: origin xyz=0.05207312 -0.0154339 -0.107654 rpy=3.14159063987 -1.50595307447 -0.211407322892 -> xyz=0.05207314 -0.0154339 -0.107654 rpy=3.14159063987 -1.50595307447 -0.211407322892
- joint r_lower_leg_skin_54_fixed_joint: origin xyz=0.04512708 -0.030749 -0.118787 rpy=3.14158825193 -1.49745145571 -0.575115374473 -> xyz=0.0451271 -0.0307489 -0.118787 rpy=3.14158825193 -1.49745145571 -0.575115374473
- joint r_lower_leg_skin_55_fixed_joint: origin xyz=0.043502663 -0.030489 -0.138143 rpy=3.14158906486 -1.48995787038 -0.597219943789 -> xyz=0.043502679 -0.0304889 -0.138143 rpy=3.14158906486 -1.48995787038 -0.597219943789
- joint r_lower_leg_skin_56_fixed_joint: origin xyz=0.04926839 -0.015121 -0.146218 rpy=-3.14158920404 -1.49124819828 -0.2234844764 -> xyz=0.04926841 -0.015121 -0.146218 rpy=-3.14158920404 -1.49124819828 -0.2234844764
- joint r_lower_leg_skin_5_fixed_joint: origin xyz=0.0636503 0.0003094 -0.001972 rpy=0 -1.38652215068 -3.14147169807 -> xyz=0.0636504 0.0003094 -0.001972 rpy=0 -1.38652215068 -3.14147169807
- joint r_lower_leg_skin_60_fixed_joint: origin xyz=0.04836967 0.018056 -0.146938 rpy=-3.14159173337 -1.48985968527 0.302951871954 -> xyz=0.04836968 0.018056 -0.146938 rpy=-3.14159173337 -1.48985968527 0.302951871954
- joint r_lower_leg_skin_61_fixed_joint: origin xyz=0.05161952 0.0014266 -0.136169 rpy=-3.14159100925 -1.49602097086 0.0132014275205 -> xyz=0.05161954 0.0014266 -0.136169 rpy=-3.14159100925 -1.49602097086 0.0132014275205
- joint r_lower_leg_skin_6_fixed_joint: origin xyz=0.05208552 0.0304434 -0.022149 rpy=-3.14158927953 -1.46785123411 0.837492889077 -> xyz=0.05208554 0.0304434 -0.022149 rpy=-3.14158927953 -1.46785123411 0.837492889077
- joint r_lower_leg_skin_9_fixed_joint: origin xyz=0.0598214 0.0167973 -0.030962 rpy=-3.14159202356 -1.34224755325 0.379294477718 -> xyz=0.0598214 0.0167972 -0.030962 rpy=-3.14159202356 -1.34224755325 0.379294477718
- joint r_sole_skin_10_fixed_joint: origin xyz=0.0725273 0.031283 0.0075 rpy=0 0 0 -> xyz=0.0725273 0.0312829 0.0075 rpy=0 0 0
- joint r_sole_skin_11_fixed_joint: origin xyz=0.0685104 0.012385 0.0075 rpy=0 0 0 -> xyz=0.0685105 0.012385 0.0075 rpy=0 0 0
- joint r_sole_skin_14_fixed_joint: origin xyz=0.05013603 0.0064148 0.0075 rpy=0 0 0 -> xyz=0.05013604 0.0064148 0.0075 rpy=0 0 0
- joint r_sole_skin_15_fixed_joint: origin xyz=0.04611917 -0.012483 0.0075 rpy=0 0 0 -> xyz=0.04611919 -0.012483 0.0075 rpy=0 0 0
- joint r_sole_skin_17_fixed_joint: origin xyz=-0.0296855 0.033257 0.0075 rpy=0 0 0 -> xyz=-0.0296855 0.0332569 0.0075 rpy=0 0 0
- joint r_sole_skin_1_fixed_joint: origin xyz=0.0788511 -0.0194404 0.0075 rpy=0 0 0 -> xyz=0.0788512 -0.0194404 0.0075 rpy=0 0 0
- joint r_sole_skin_9_fixed_joint: origin xyz=0.0909017 0.037253 0.0075 rpy=0 0 0 -> xyz=0.0909017 0.0372529 0.0075 rpy=0 0 0
- joint r_upper_leg_back_contact_fixed_joint: origin xyz=-0.0511999 0 0.0146 rpy=0 1.57079632679 0 -> xyz=-0.0511998 0 0.0146 rpy=0 1.57079632679 0
