Commit message: Automatic build. GitHub Actions build: 3470957903 icub-model-generator commit: robotology/icub-models-generator@f08e8964cf8b2333c4eead8430d30df4dee4f838 urdf_parser_py commit: ros/urdf_parser_py@31474b9baaf7c3845b40e5a9aa87d5900a2282c3 simmechanics-to-urdf commit: robotology/simmechanics-to-urdf@4de30ebf6e6eb33b1f3009c9e5b68f529ff8f2b8

File: iCub/robots/iCubGazeboV2_7/model.urdf (robot description, URDF)
Before this commit: robot iCub, 190 links, 189 joints
Links:
- added link chest_ems_gyro_eb1
- added link chest_ems_gyro_eb2
- added link chest_ems_gyro_eb3
- added link chest_ems_gyro_eb4
- added link l_foot_ft_gyro_3b13
- added link l_lower_leg_ems_gyro_eb7
- added link l_upper_leg_ems_gyro_eb10
- added link l_upper_leg_ems_gyro_eb6
- added link l_upper_leg_ft_gyro_3b12
- added link r_foot_ft_gyro_3b14
- added link r_lower_leg_ems_gyro_eb9
- added link r_upper_leg_ems_gyro_eb11
- added link r_upper_leg_ems_gyro_eb8
- added link r_upper_leg_ft_gyro_3b11
- added link root_link_ems_gyro_eb5
Joints:
- added joint chest_ems_gyro_eb1_fixed_joint: type fixed, parent chest, child chest_ems_gyro_eb1, origin xyz=0.069201600190735 0.06454800000000001 -0.0635258 rpy=3.1415169122972952 -0.2617993091222473 0.0002926418802545251
- added joint chest_ems_gyro_eb2_fixed_joint: type fixed, parent chest, child chest_ems_gyro_eb2, origin xyz=0.016037100190735 0.08755899999999998 -0.0653479 rpy=3.141590501042822 0.2617993198185103 3.1415843367812997
- added joint chest_ems_gyro_eb3_fixed_joint: type fixed, parent chest, child chest_ems_gyro_eb3, origin xyz=-0.018641699809265 0.064521 -0.0770785 rpy=3.141109162025268 0.26110051647116095 -0.00030907146255546275
- added joint chest_ems_gyro_eb4_fixed_joint: type fixed, parent chest, child chest_ems_gyro_eb4, origin xyz=-0.06657839980926501 0.08755899999999998 -0.0518054 rpy=-3.1415905047625503 -0.26179931981852844 3.141584339870295
- added joint l_foot_ft_gyro_3b13_fixed_joint: type fixed, parent l_ankle_2, child l_foot_ft_gyro_3b13, origin xyz=0.0040001999999999885 -0.008600000000000003 -0.045282000000000044 rpy=0 0 1.5707963267948966
- added joint l_lower_leg_ems_gyro_eb7_fixed_joint: type fixed, parent l_lower_leg, child l_lower_leg_ems_gyro_eb7, origin xyz=0.04450335399999999 0.011818499999999968 -0.08830099999999996 rpy=3.1415926535897922 -1.3526297834539558 0
- added joint l_upper_leg_ems_gyro_eb10_fixed_joint: type fixed, parent l_upper_leg, child l_upper_leg_ems_gyro_eb10, origin xyz=-0.013079 0.04040679999999998 -0.035654999999999964 rpy=-1.570796326794897 -1.570796326794896 0
- added joint l_upper_leg_ems_gyro_eb6_fixed_joint: type fixed, parent l_upper_leg, child l_upper_leg_ems_gyro_eb6, origin xyz=-0.013081000000000016 -0.04040720000000002 -0.087979 rpy=1.5707963267948966 1.5707963267948961 0
- added joint l_upper_leg_ft_gyro_3b12_fixed_joint: type fixed, parent l_hip_2, child l_upper_leg_ft_gyro_3b12, origin xyz=0.006669999999999995 -0.008524799999999999 -0.059281999999999946 rpy=0 0 1.5707963267948966
- added joint r_foot_ft_gyro_3b14_fixed_joint: type fixed, parent r_ankle_2, child r_foot_ft_gyro_3b14, origin xyz=0.0040000999999999926 -0.00860000000000001 -0.045282000000000044 rpy=0 0 1.5707963267948966
- added joint r_lower_leg_ems_gyro_eb9_fixed_joint: type fixed, parent r_lower_leg, child r_lower_leg_ems_gyro_eb9, origin xyz=0.04450330799999999 0.014343499999999974 -0.08830099999999996 rpy=3.1415926535897922 -1.3526297834539558 0
- added joint r_upper_leg_ems_gyro_eb11_fixed_joint: type fixed, parent r_upper_leg, child r_upper_leg_ems_gyro_eb11, origin xyz=-0.013081000000000016 -0.040406899999999996 -0.087979 rpy=1.5707963267948966 1.5707963267948961 0
- added joint r_upper_leg_ems_gyro_eb8_fixed_joint: type fixed, parent r_upper_leg, child r_upper_leg_ems_gyro_eb8, origin xyz=-0.013078999999999993 0.04040709999999999 -0.035654999999999964 rpy=1.5707963267948966 1.5707963267948961 0
- added joint r_upper_leg_ft_gyro_3b11_fixed_joint: type fixed, parent r_hip_2, child r_upper_leg_ft_gyro_3b11, origin xyz=0.006563800000000002 -0.008586100000000013 -0.059281999999999946 rpy=0 0 1.5707963267948966
- added joint root_link_ems_gyro_eb5_fixed_joint: type fixed, parent root_link, child root_link_ems_gyro_eb5, origin xyz=0.0493308 -0.012577100000000023 -0.11569100000000002 rpy=3.141592653589793 1.2915440450258349 3.141592653589793

File: iCub/robots/iCubGazeboV3/model.urdf (robot description, URDF)
Before this commit: robot iCub, 48 links, 47 joints
Links:
- removed link chest_depth_frame
- removed link imu_frame
- added link chest_imu_acc_1x1
- added link head_imu_acc_1x1
Joints:
- removed joint chest_depth_frame_fixed_joint
- removed joint imu_frame_fixed_joint
- added joint chest_imu_acc_1x1_fixed_joint: type fixed, parent chest, child chest_imu_acc_1x1, origin xyz=0.0894115 0.0175 0.09929950000000001 rpy=-1.5707963267948968 0 -1.5707963267948968
- added joint head_imu_acc_1x1_fixed_joint: type fixed, parent head, child head_imu_acc_1x1, origin xyz=0.0035000000000000005 0.0055 0.10133400000000001 rpy=3.141592653589793 0 -1.5707963267948966

File: iCub/robots/iCubGenova02/model.urdf (robot description, URDF)
Before this commit: robot iCub, 140 links, 139 joints
Links:
- removed link root_link_imu_frame
- added link chest_ems_gyro_eb1
- added link chest_ems_gyro_eb2
- added link chest_ems_gyro_eb3
- added link chest_ems_gyro_eb4
- added link l_lower_leg_ems_gyro_eb7
- added link l_upper_leg_ems_gyro_eb10
- added link l_upper_leg_ems_gyro_eb6
- added link r_lower_leg_ems_gyro_eb9
- added link r_upper_leg_ems_gyro_eb11
- added link r_upper_leg_ems_gyro_eb8
- added link root_link_ems_gyro_eb5
- added link root_link_imu_acc
Joints:
- removed joint root_link_imu_frame_fixed_joint
- added joint chest_ems_gyro_eb1_fixed_joint: type fixed, parent chest, child chest_ems_gyro_eb1, origin xyz=0.069201600190735 0.06454800000000001 -0.0635258 rpy=3.1415169122972952 -0.2617993091222473 0.0002926418802545251
- added joint chest_ems_gyro_eb2_fixed_joint: type fixed, parent chest, child chest_ems_gyro_eb2, origin xyz=0.016037100190735 0.08755899999999998 -0.0653479 rpy=3.141590501042822 0.2617993198185103 3.1415843367812997
- added joint chest_ems_gyro_eb3_fixed_joint: type fixed, parent chest, child chest_ems_gyro_eb3, origin xyz=-0.018641699809265 0.064521 -0.0770785 rpy=3.141109162025268 0.26110051647116095 -0.00030907146255546275
- added joint chest_ems_gyro_eb4_fixed_joint: type fixed, parent chest, child chest_ems_gyro_eb4, origin xyz=-0.06657839980926501 0.08755899999999998 -0.0518054 rpy=-3.1415905047625503 -0.26179931981852844 3.141584339870295
- added joint l_lower_leg_ems_gyro_eb7_fixed_joint: type fixed, parent l_lower_leg, child l_lower_leg_ems_gyro_eb7, origin xyz=0.04450329199999999 0.011818499999999968 -0.08830099999999996 rpy=3.1415926535897922 -1.3526297834539558 0
- added joint l_upper_leg_ems_gyro_eb10_fixed_joint: type fixed, parent l_upper_leg, child l_upper_leg_ems_gyro_eb10, origin xyz=-0.013078999999999986 0.040407 -0.035654999999999964 rpy=-1.570796326794897 -1.570796326794896 0
- added joint l_upper_leg_ems_gyro_eb6_fixed_joint: type fixed, parent l_upper_leg, child l_upper_leg_ems_gyro_eb6, origin xyz=-0.013081000000000002 -0.040407200000000004 -0.087979 rpy=1.5707963267948966 1.5707963267948961 0
- added joint r_lower_leg_ems_gyro_eb9_fixed_joint: type fixed, parent r_lower_leg, child r_lower_leg_ems_gyro_eb9, origin xyz=0.044503292 0.014343499999999974 -0.08830099999999996 rpy=3.1415926535897922 -1.3526297834539558 0
- added joint r_upper_leg_ems_gyro_eb11_fixed_joint: type fixed, parent r_upper_leg, child r_upper_leg_ems_gyro_eb11, origin xyz=-0.013081000000000002 -0.04040700000000001 -0.087979 rpy=1.5707963267948966 1.5707963267948961 0
- added joint r_upper_leg_ems_gyro_eb8_fixed_joint: type fixed, parent r_upper_leg, child r_upper_leg_ems_gyro_eb8, origin xyz=-0.01307899999999998 0.04040719999999998 -0.035654999999999964 rpy=1.5707963267948966 1.5707963267948961 0
- added joint root_link_ems_gyro_eb5_fixed_joint: type fixed, parent root_link, child root_link_ems_gyro_eb5, origin xyz=0.0493308 -0.012577100000000023 -0.11569100000000002 rpy=3.141592653589793 1.2915440450258349 3.141592653589793
- added joint root_link_imu_acc_fixed_joint: type fixed, parent root_link, child root_link_imu_acc, origin xyz=0.08515499999999998 -0.011000000000000022 -0.11230899999999999 rpy=-2.0943952105869323 0 -1.5707963267948963

File: iCub/robots/iCubGenova09/model.urdf (robot description, URDF)
Before this commit: robot iCub, 48 links, 47 joints
Links:
- removed link chest_depth_frame
- removed link imu_frame
- added link chest_imu_acc_1x1
- added link head_imu_acc_1x1
Joints:
- removed joint chest_depth_frame_fixed_joint
- removed joint imu_frame_fixed_joint
- added joint chest_imu_acc_1x1_fixed_joint: type fixed, parent chest, child chest_imu_acc_1x1, origin xyz=0.0894115 0.0175 0.09929950000000001 rpy=-1.5707963267948968 0 -1.5707963267948968
- added joint head_imu_acc_1x1_fixed_joint: type fixed, parent head, child head_imu_acc_1x1, origin xyz=0.0035000000000000005 0.0055 0.10133400000000001 rpy=3.141592653589793 0 -1.5707963267948966

Commit message: Automatic build. GitHub Actions build: 3957889275 icub-model-generator commit: robotology/icub-models-generator@1a5d6b4e1a680a2d7fffea939e6dbf186acabb7d urdf_parser_py commit: ros/urdf_parser_py@31474b9baaf7c3845b40e5a9aa87d5900a2282c3 simmechanics-to-urdf commit: robotology/simmechanics-to-urdf@30ceec80f8c37fb9638f6117a04e64267c0d9a08

File: iCub/robots/iCubDarmstadt01/model.urdf (robot description, URDF)
Before this commit: robot iCub, 204 links, 203 joints
Links:
- added link l_arm_ft
- added link l_foot_ft
- added link l_leg_ft
- added link r_arm_ft
- added link r_foot_ft
- added link r_leg_ft
Joints:
- added joint l_arm_ft_fixed_joint: type fixed, parent l_shoulder_3, child l_arm_ft, origin xyz=0.05093014324520106 0 0.029175829465900395 rpy=0 -1.3089970069677395 3.1415926535897927
- added joint l_foot_ft_fixed_joint: type fixed, parent l_foot, child l_foot_ft, origin xyz=0 0 0 rpy=0 0 0
- added joint l_leg_ft_fixed_joint: type fixed, parent l_hip_3, child l_leg_ft, origin xyz=0 0 0 rpy=0 0 0
- added joint r_arm_ft_fixed_joint: type fixed, parent r_shoulder_3, child r_arm_ft, origin xyz=-0.05089730176650909 0 0.029167029620599215 rpy=0 -1.3089970069677397 0
- added joint r_foot_ft_fixed_joint: type fixed, parent r_foot, child r_foot_ft, origin xyz=0 0 0 rpy=0 0 0
- added joint r_leg_ft_fixed_joint: type fixed, parent r_hip_3, child r_leg_ft, origin xyz=0 0 0 rpy=0 0 0

File: iCub/robots/iCubErzelli02/model.urdf (robot description, URDF)
Before this commit: robot iCub, 204 links, 203 joints
Links:
- added link l_arm_ft
- added link l_foot_ft
- added link l_leg_ft
- added link r_arm_ft
- added link r_foot_ft
- added link r_leg_ft
Joints:
- added joint l_arm_ft_fixed_joint: type fixed, parent l_shoulder_3, child l_arm_ft, origin xyz=0.05093014324520106 0 0.029175829465900395 rpy=0 -1.3089970069677395 3.1415926535897927
- added joint l_foot_ft_fixed_joint: type fixed, parent l_foot, child l_foot_ft, origin xyz=0 0 0 rpy=0 0 0
- added joint l_leg_ft_fixed_joint: type fixed, parent l_hip_3, child l_leg_ft, origin xyz=0 0 0 rpy=0 0 0
- added joint r_arm_ft_fixed_joint: type fixed, parent r_shoulder_3, child r_arm_ft, origin xyz=-0.05089730176650909 0 0.029167029620599215 rpy=0 -1.3089970069677397 0
- added joint r_foot_ft_fixed_joint: type fixed, parent r_foot, child r_foot_ft, origin xyz=0 0 0 rpy=0 0 0
- added joint r_leg_ft_fixed_joint: type fixed, parent r_hip_3, child r_leg_ft, origin xyz=0 0 0 rpy=0 0 0

File: iCub/robots/iCubGazeboV2_5/model.urdf (robot description, URDF)
Before this commit: robot iCub, 204 links, 203 joints
Links:
- added link l_arm_ft
- added link l_foot_ft
- added link l_leg_ft
- added link r_arm_ft
- added link r_foot_ft
- added link r_leg_ft
Joints:
- added joint l_arm_ft_fixed_joint: type fixed, parent l_shoulder_3, child l_arm_ft, origin xyz=0.05093014324520106 0 0.029175829465900395 rpy=0 -1.3089970069677395 3.1415926535897927
- added joint l_foot_ft_fixed_joint: type fixed, parent l_foot, child l_foot_ft, origin xyz=0 0 0 rpy=0 0 0
- added joint l_leg_ft_fixed_joint: type fixed, parent l_hip_3, child l_leg_ft, origin xyz=0 0 0 rpy=0 0 0
- added joint r_arm_ft_fixed_joint: type fixed, parent r_shoulder_3, child r_arm_ft, origin xyz=-0.05089730176650909 0 0.029167029620599215 rpy=0 -1.3089970069677397 0
- added joint r_foot_ft_fixed_joint: type fixed, parent r_foot, child r_foot_ft, origin xyz=0 0 0 rpy=0 0 0
- added joint r_leg_ft_fixed_joint: type fixed, parent r_hip_3, child r_leg_ft, origin xyz=0 0 0 rpy=0 0 0

File: iCub/robots/iCubGazeboV2_5_plus/model.urdf (robot description, URDF)
Before this commit: robot iCub, 151 links, 150 joints
Links:
- added link l_arm_ft
- added link l_foot_ft
- added link l_leg_ft
- added link r_arm_ft
- added link r_foot_ft
- added link r_leg_ft
Joints:
- added joint l_arm_ft_fixed_joint: type fixed, parent l_shoulder_3, child l_arm_ft, origin xyz=0.05093014324520106 0 0.029175829465900395 rpy=0 -1.3089970069677395 3.1415926535897927
- added joint l_foot_ft_fixed_joint: type fixed, parent l_foot, child l_foot_ft, origin xyz=0 0 0 rpy=0 0 0
- added joint l_leg_ft_fixed_joint: type fixed, parent l_hip_3, child l_leg_ft, origin xyz=0 0 0 rpy=0 0 0
- added joint r_arm_ft_fixed_joint: type fixed, parent r_shoulder_3, child r_arm_ft, origin xyz=-0.05089730176650909 0 0.029167029620599215 rpy=0 -1.3089970069677397 0
- added joint r_foot_ft_fixed_joint: type fixed, parent r_foot, child r_foot_ft, origin xyz=0 0 0 rpy=0 0 0
- added joint r_leg_ft_fixed_joint: type fixed, parent r_hip_3, child r_leg_ft, origin xyz=0 0 0 rpy=0 0 0

File: iCub/robots/iCubGazeboV2_6/model.urdf (robot description, URDF)
Before this commit: robot iCub, 204 links, 203 joints
Links:
- added link l_arm_ft
- added link l_foot_ft
- added link l_leg_ft
- added link r_arm_ft
- added link r_foot_ft
- added link r_leg_ft
Joints:
- added joint l_arm_ft_fixed_joint: type fixed, parent l_shoulder_3, child l_arm_ft, origin xyz=0.05093014324520106 0 0.029175829465900395 rpy=0 -1.3089970069677395 3.1415926535897927
- added joint l_foot_ft_fixed_joint: type fixed, parent l_foot, child l_foot_ft, origin xyz=0 0 0 rpy=0 0 0
- added joint l_leg_ft_fixed_joint: type fixed, parent l_hip_3, child l_leg_ft, origin xyz=0 0 0 rpy=0 0 0
- added joint r_arm_ft_fixed_joint: type fixed, parent r_shoulder_3, child r_arm_ft, origin xyz=-0.05089730176650909 0 0.029167029620599215 rpy=0 -1.3089970069677397 0
- added joint r_foot_ft_fixed_joint: type fixed, parent r_foot, child r_foot_ft, origin xyz=0 0 0 rpy=0 0 0
- added joint r_leg_ft_fixed_joint: type fixed, parent r_hip_3, child r_leg_ft, origin xyz=0 0 0 rpy=0 0 0

File: iCub/robots/iCubGazeboV2_7/model.urdf (robot description, URDF)
Before this commit: robot iCub, 205 links, 204 joints
Links:
- added link l_arm_ft
- added link l_foot_ft
- added link l_leg_ft
- added link r_arm_ft
- added link r_foot_ft
- added link r_leg_ft
Joints:
- added joint l_arm_ft_fixed_joint: type fixed, parent l_shoulder_3, child l_arm_ft, origin xyz=0.05093014324520106 0 0.029175829465900395 rpy=0 -1.3089970069677395 3.1415926535897927
- added joint l_foot_ft_fixed_joint: type fixed, parent l_foot, child l_foot_ft, origin xyz=0 0 0 rpy=0 0 0
- added joint l_leg_ft_fixed_joint: type fixed, parent l_hip_3, child l_leg_ft, origin xyz=0 0 0 rpy=0 0 0
- added joint r_arm_ft_fixed_joint: type fixed, parent r_shoulder_3, child r_arm_ft, origin xyz=-0.05089730176650909 0 0.029167029620599215 rpy=0 -1.3089970069677397 0
- added joint r_foot_ft_fixed_joint: type fixed, parent r_foot, child r_foot_ft, origin xyz=0 0 0 rpy=0 0 0
- added joint r_leg_ft_fixed_joint: type fixed, parent r_hip_3, child r_leg_ft, origin xyz=0 0 0 rpy=0 0 0

File: iCub/robots/iCubGenova02/model.urdf (robot description, URDF)
Before this commit: robot iCub, 151 links, 150 joints
Links:
- added link l_arm_ft
- added link l_foot_ft
- added link l_leg_ft
- added link r_arm_ft
- added link r_foot_ft
- added link r_leg_ft
Joints:
- added joint l_arm_ft_fixed_joint: type fixed, parent l_shoulder_3, child l_arm_ft, origin xyz=0.05093014324520106 0 0.029175829465900395 rpy=0 -1.3089970069677395 3.1415926535897927
- added joint l_foot_ft_fixed_joint: type fixed, parent l_foot, child l_foot_ft, origin xyz=0 0 0 rpy=0 0 0
- added joint l_leg_ft_fixed_joint: type fixed, parent l_hip_3, child l_leg_ft, origin xyz=0 0 0 rpy=0 0 0
- added joint r_arm_ft_fixed_joint: type fixed, parent r_shoulder_3, child r_arm_ft, origin xyz=-0.05089730176650909 0 0.029167029620599215 rpy=0 -1.3089970069677397 0
- added joint r_foot_ft_fixed_joint: type fixed, parent r_foot, child r_foot_ft, origin xyz=0 0 0 rpy=0 0 0
- added joint r_leg_ft_fixed_joint: type fixed, parent r_hip_3, child r_leg_ft, origin xyz=0 0 0 rpy=0 0 0

Commit message: Automatic build. GitHub Actions build: 4055274942 icub-model-generator commit: robotology/icub-models-generator@2597ab6a2e8116776aafc75eb43f6801e8c9cf96 urdf_parser_py commit: ros/urdf_parser_py@31474b9baaf7c3845b40e5a9aa87d5900a2282c3 simmechanics-to-urdf commit: robotology/simmechanics-to-urdf@30ceec80f8c37fb9638f6117a04e64267c0d9a08

File: iCub/robots/iCubDarmstadt01/model.urdf (robot description, URDF)
Before this commit: robot iCub, 210 links, 209 joints
Links:
- removed link imu_frame
- added link head_imu_0
Joints:
- removed joint imu_frame_fixed_joint
- added joint head_imu_0_fixed_joint: type fixed, parent head, child head_imu_0, origin xyz=0.009500000190735 0.133444 0.009299999999999996 rpy=-1.5707963267948961 1.570796326794896 0

File: iCub/robots/iCubErzelli02/model.urdf (robot description, URDF)
Before this commit: robot iCub, 210 links, 209 joints
Links:
- removed link imu_frame
- added link head_imu_0
Joints:
- removed joint imu_frame_fixed_joint
- added joint head_imu_0_fixed_joint: type fixed, parent head, child head_imu_0, origin xyz=0.009500000190735 0.133444 0.009299999999999996 rpy=-1.5707963267948961 1.570796326794896 0

File: iCub/robots/iCubGazeboV2_5/model.urdf (robot description, URDF)
Before this commit: robot iCub, 210 links, 209 joints
Links:
- removed link imu_frame
- added link head_imu_0
Joints:
- removed joint imu_frame_fixed_joint
- added joint head_imu_0_fixed_joint: type fixed, parent head, child head_imu_0, origin xyz=0.009500000190735 0.133444 0.009299999999999996 rpy=-1.5707963267948961 1.570796326794896 0

File: iCub/robots/iCubGazeboV2_5_plus/model.urdf (robot description, URDF)
Before this commit: robot iCub, 157 links, 156 joints
Links:
- removed link imu_frame
- added link head_imu_0
Joints:
- removed joint imu_frame_fixed_joint
- added joint head_imu_0_fixed_joint: type fixed, parent head, child head_imu_0, origin xyz=0.009500000190735 0.133444 0.009299999999999996 rpy=-1.5707963267948961 1.570796326794896 0

File: iCub/robots/iCubGazeboV2_6/model.urdf (robot description, URDF)
Before this commit: robot iCub, 210 links, 209 joints
Links:
- removed link imu_frame
- added link head_imu_0
Joints:
- removed joint imu_frame_fixed_joint
- added joint head_imu_0_fixed_joint: type fixed, parent head, child head_imu_0, origin xyz=0.009500000190735 0.133444 0.009299999999999996 rpy=-1.5707963267948961 1.570796326794896 0

File: iCub/robots/iCubGazeboV2_7/model.urdf (robot description, URDF)
Before this commit: robot iCub, 211 links, 210 joints
Links:
- removed link imu_frame
- added link head_imu_0
Joints:
- removed joint imu_frame_fixed_joint
- added joint head_imu_0_fixed_joint: type fixed, parent head, child head_imu_0, origin xyz=0.009500000190735 0.133444 0.009299999999999996 rpy=-1.5707963267948961 1.570796326794896 0

File: iCub/robots/iCubGazeboV3/model.urdf (robot description, URDF)
Before this commit: robot iCub, 56 links, 55 joints
Links:
- removed link chest_imu_acc_1x1
- removed link head_imu_acc_1x1
- added link chest_imu_0
- added link head_imu_0
Joints:
- removed joint chest_imu_acc_1x1_fixed_joint
- removed joint head_imu_acc_1x1_fixed_joint
- added joint chest_imu_0_fixed_joint: type fixed, parent chest, child chest_imu_0, origin xyz=0.0894115 0.0175 0.09929950000000001 rpy=-1.5707963267948968 0 -1.5707963267948968
- added joint head_imu_0_fixed_joint: type fixed, parent head, child head_imu_0, origin xyz=0.0035000000000000005 0.0055 0.10133400000000001 rpy=3.141592653589793 0 -1.5707963267948966

File: iCub/robots/iCubGenova02/model.urdf (robot description, URDF)
Before this commit: robot iCub, 157 links, 156 joints
Links:
- removed link imu_frame
- added link head_imu_0
Joints:
- removed joint imu_frame_fixed_joint
- added joint head_imu_0_fixed_joint: type fixed, parent head, child head_imu_0, origin xyz=0.009500000190735 0.133444 0.009299999999999996 rpy=-1.5707963267948961 1.570796326794896 0

File: iCub/robots/iCubGenova09/model.urdf (robot description, URDF)
Before this commit: robot iCub, 56 links, 55 joints
Links:
- removed link chest_imu_acc_1x1
- removed link head_imu_acc_1x1
- added link chest_imu_0
- added link head_imu_0
Joints:
- removed joint chest_imu_acc_1x1_fixed_joint
- removed joint head_imu_acc_1x1_fixed_joint
- added joint chest_imu_0_fixed_joint: type fixed, parent chest, child chest_imu_0, origin xyz=0.0894115 0.0175 0.09929950000000001 rpy=-1.5707963267948968 0 -1.5707963267948968
- added joint head_imu_0_fixed_joint: type fixed, parent head, child head_imu_0, origin xyz=0.0035000000000000005 0.0055 0.10133400000000001 rpy=3.141592653589793 0 -1.5707963267948966
