Commit message: Automatic build. GitHub Actions build: 6695395395 icub-model-generator commit: robotology/icub-models-generator@cf90d5e2a6e96cc65c8652ee5e0900760145a957 urdf_parser_py commit: ros/urdf_parser_py@31474b9baaf7c3845b40e5a9aa87d5900a2282c3 simmechanics-to-urdf commit: robotology/simmechanics-to-urdf@9431d99570921d20002461a02d4974020e97f22a

File: iCub/robots/iCubDarmstadt01/model.urdf (robot description, URDF)
Before this commit: robot iCub, 210 links, 209 joints
Joints:
- joint l_sole_skin_0_fixed_joint: origin xyz=0.09320879999999998 0.032367999999999994 0.007500000000000062 rpy=0 0 0 -> xyz=0.05013608999999999 -0.006414799999999998 0.007500000000000062 rpy=0 0 0
- joint l_sole_skin_10_fixed_joint: origin xyz=0.10525929999999997 -0.024325399999999983 0.007500000000000062 rpy=0 0 0 -> xyz=0.09320879999999998 0.032367999999999994 0.007500000000000062 rpy=0 0 0
- joint l_sole_skin_11_fixed_joint: origin xyz=0.10124249999999999 -0.005428100000000005 0.007500000000000062 rpy=0 0 0 -> xyz=0.07885119999999998 0.019439899999999996 0.007500000000000062 rpy=0 0 0
- joint l_sole_skin_13_fixed_joint: origin xyz=0.06851049999999999 -0.012385499999999994 0.007500000000000062 rpy=0 0 0 -> xyz=0.10124249999999999 -0.005428100000000005 0.007500000000000062 rpy=0 0 0
- joint l_sole_skin_14_fixed_joint: origin xyz=0.11559999999999998 0.007499500000000006 0.007500000000000062 rpy=0 0 0 -> xyz=0.06047679999999998 0.02541059999999999 0.007500000000000062 rpy=0 0 0
- joint l_sole_skin_15_fixed_joint: origin xyz=0.11158319999999997 0.02639729999999999 0.007500000000000062 rpy=0 0 0 -> xyz=0.04611922999999998 0.012482499999999994 0.007500000000000062 rpy=0 0 0
- joint l_sole_skin_1_fixed_joint: origin xyz=0.07885119999999998 0.019439899999999996 0.007500000000000062 rpy=0 0 0 -> xyz=0.06851049999999999 -0.012385499999999994 0.007500000000000062 rpy=0 0 0
- joint l_sole_skin_2_fixed_joint: origin xyz=0.06047679999999998 0.02541059999999999 0.007500000000000062 rpy=0 0 0 -> xyz=0.07252739999999999 -0.031282799999999986 0.007500000000000062 rpy=0 0 0
- joint l_sole_skin_3_fixed_joint: origin xyz=0.04611922999999998 0.012482499999999994 0.007500000000000062 rpy=0 0 0 -> xyz=0.09090179999999999 -0.03725379999999999 0.007500000000000062 rpy=0 0 0
- joint l_sole_skin_4_fixed_joint: origin xyz=0.05013608999999999 -0.006414799999999998 0.007500000000000062 rpy=0 0 0 -> xyz=0.10525929999999997 -0.024325399999999983 0.007500000000000062 rpy=0 0 0
- joint l_sole_skin_8_fixed_joint: origin xyz=0.07252739999999999 -0.031282799999999986 0.007500000000000062 rpy=0 0 0 -> xyz=0.11559999999999998 0.007499500000000006 0.007500000000000062 rpy=0 0 0
- joint l_sole_skin_9_fixed_joint: origin xyz=0.09090179999999999 -0.03725379999999999 0.007500000000000062 rpy=0 0 0 -> xyz=0.11158319999999997 0.02639729999999999 0.007500000000000062 rpy=0 0 0
- joint r_sole_skin_0_fixed_joint: origin xyz=0.060476699999999994 -0.0254106 0.007500000000000062 rpy=0 0 0 -> xyz=0.11559999999999998 -0.007499999999999993 0.007500000000000062 rpy=0 0 0
- joint r_sole_skin_10_fixed_joint: origin xyz=0.07252729999999998 0.03128289999999999 0.007500000000000062 rpy=0 0 0 -> xyz=0.060476699999999994 -0.0254106 0.007500000000000062 rpy=0 0 0
- joint r_sole_skin_11_fixed_joint: origin xyz=0.06851049999999997 0.012385000000000007 0.007500000000000062 rpy=0 0 0 -> xyz=0.07885119999999998 -0.019440400000000004 0.007500000000000062 rpy=0 0 0
- joint r_sole_skin_13_fixed_joint: origin xyz=0.10124239999999998 0.005427600000000005 0.007500000000000062 rpy=0 0 0 -> xyz=0.06851049999999997 0.012385000000000007 0.007500000000000062 rpy=0 0 0
- joint r_sole_skin_14_fixed_joint: origin xyz=0.050136039999999986 0.006414799999999998 0.007500000000000062 rpy=0 0 0 -> xyz=0.09320869999999999 -0.032368 0.007500000000000062 rpy=0 0 0
- joint r_sole_skin_15_fixed_joint: origin xyz=0.04611918999999999 -0.012483000000000008 0.007500000000000062 rpy=0 0 0 -> xyz=0.11158309999999998 -0.0263978 0.007500000000000062 rpy=0 0 0
- joint r_sole_skin_1_fixed_joint: origin xyz=0.07885119999999998 -0.019440400000000004 0.007500000000000062 rpy=0 0 0 -> xyz=0.10124239999999998 0.005427600000000005 0.007500000000000062 rpy=0 0 0
- joint r_sole_skin_2_fixed_joint: origin xyz=0.09320869999999999 -0.032368 0.007500000000000062 rpy=0 0 0 -> xyz=0.10525929999999997 0.024325399999999997 0.007500000000000062 rpy=0 0 0
- joint r_sole_skin_3_fixed_joint: origin xyz=0.11158309999999998 -0.0263978 0.007500000000000062 rpy=0 0 0 -> xyz=0.09090169999999997 0.03725289999999999 0.007500000000000062 rpy=0 0 0
- joint r_sole_skin_4_fixed_joint: origin xyz=0.11559999999999998 -0.007499999999999993 0.007500000000000062 rpy=0 0 0 -> xyz=0.07252729999999998 0.03128289999999999 0.007500000000000062 rpy=0 0 0
- joint r_sole_skin_8_fixed_joint: origin xyz=0.10525929999999997 0.024325399999999997 0.007500000000000062 rpy=0 0 0 -> xyz=0.050136039999999986 0.006414799999999998 0.007500000000000062 rpy=0 0 0
- joint r_sole_skin_9_fixed_joint: origin xyz=0.09090169999999997 0.03725289999999999 0.007500000000000062 rpy=0 0 0 -> xyz=0.04611918999999999 -0.012483000000000008 0.007500000000000062 rpy=0 0 0

File: iCub/robots/iCubErzelli02/model.urdf (robot description, URDF)
Before this commit: robot iCub, 210 links, 209 joints
Joints:
- joint l_sole_skin_0_fixed_joint: origin xyz=0.09320879999999998 0.032367999999999994 0.007500000000000062 rpy=0 0 0 -> xyz=0.05013608999999999 -0.006414799999999998 0.007500000000000062 rpy=0 0 0
- joint l_sole_skin_10_fixed_joint: origin xyz=0.10525929999999997 -0.024325399999999983 0.007500000000000062 rpy=0 0 0 -> xyz=0.09320879999999998 0.032367999999999994 0.007500000000000062 rpy=0 0 0
- joint l_sole_skin_11_fixed_joint: origin xyz=0.10124249999999999 -0.005428100000000005 0.007500000000000062 rpy=0 0 0 -> xyz=0.07885119999999998 0.019439899999999996 0.007500000000000062 rpy=0 0 0
- joint l_sole_skin_13_fixed_joint: origin xyz=0.06851049999999999 -0.012385499999999994 0.007500000000000062 rpy=0 0 0 -> xyz=0.10124249999999999 -0.005428100000000005 0.007500000000000062 rpy=0 0 0
- joint l_sole_skin_14_fixed_joint: origin xyz=0.11559999999999998 0.007499500000000006 0.007500000000000062 rpy=0 0 0 -> xyz=0.06047679999999998 0.02541059999999999 0.007500000000000062 rpy=0 0 0
- joint l_sole_skin_15_fixed_joint: origin xyz=0.11158319999999997 0.02639729999999999 0.007500000000000062 rpy=0 0 0 -> xyz=0.04611922999999998 0.012482499999999994 0.007500000000000062 rpy=0 0 0
- joint l_sole_skin_1_fixed_joint: origin xyz=0.07885119999999998 0.019439899999999996 0.007500000000000062 rpy=0 0 0 -> xyz=0.06851049999999999 -0.012385499999999994 0.007500000000000062 rpy=0 0 0
- joint l_sole_skin_2_fixed_joint: origin xyz=0.06047679999999998 0.02541059999999999 0.007500000000000062 rpy=0 0 0 -> xyz=0.07252739999999999 -0.031282799999999986 0.007500000000000062 rpy=0 0 0
- joint l_sole_skin_3_fixed_joint: origin xyz=0.04611922999999998 0.012482499999999994 0.007500000000000062 rpy=0 0 0 -> xyz=0.09090179999999999 -0.03725379999999999 0.007500000000000062 rpy=0 0 0
- joint l_sole_skin_4_fixed_joint: origin xyz=0.05013608999999999 -0.006414799999999998 0.007500000000000062 rpy=0 0 0 -> xyz=0.10525929999999997 -0.024325399999999983 0.007500000000000062 rpy=0 0 0
- joint l_sole_skin_8_fixed_joint: origin xyz=0.07252739999999999 -0.031282799999999986 0.007500000000000062 rpy=0 0 0 -> xyz=0.11559999999999998 0.007499500000000006 0.007500000000000062 rpy=0 0 0
- joint l_sole_skin_9_fixed_joint: origin xyz=0.09090179999999999 -0.03725379999999999 0.007500000000000062 rpy=0 0 0 -> xyz=0.11158319999999997 0.02639729999999999 0.007500000000000062 rpy=0 0 0
- joint r_sole_skin_0_fixed_joint: origin xyz=0.060476699999999994 -0.0254106 0.007500000000000062 rpy=0 0 0 -> xyz=0.11559999999999998 -0.007499999999999993 0.007500000000000062 rpy=0 0 0
- joint r_sole_skin_10_fixed_joint: origin xyz=0.07252729999999998 0.03128289999999999 0.007500000000000062 rpy=0 0 0 -> xyz=0.060476699999999994 -0.0254106 0.007500000000000062 rpy=0 0 0
- joint r_sole_skin_11_fixed_joint: origin xyz=0.06851049999999997 0.012385000000000007 0.007500000000000062 rpy=0 0 0 -> xyz=0.07885119999999998 -0.019440400000000004 0.007500000000000062 rpy=0 0 0
- joint r_sole_skin_13_fixed_joint: origin xyz=0.10124239999999998 0.005427600000000005 0.007500000000000062 rpy=0 0 0 -> xyz=0.06851049999999997 0.012385000000000007 0.007500000000000062 rpy=0 0 0
- joint r_sole_skin_14_fixed_joint: origin xyz=0.050136039999999986 0.006414799999999998 0.007500000000000062 rpy=0 0 0 -> xyz=0.09320869999999999 -0.032368 0.007500000000000062 rpy=0 0 0
- joint r_sole_skin_15_fixed_joint: origin xyz=0.04611918999999999 -0.012483000000000008 0.007500000000000062 rpy=0 0 0 -> xyz=0.11158309999999998 -0.0263978 0.007500000000000062 rpy=0 0 0
- joint r_sole_skin_1_fixed_joint: origin xyz=0.07885119999999998 -0.019440400000000004 0.007500000000000062 rpy=0 0 0 -> xyz=0.10124239999999998 0.005427600000000005 0.007500000000000062 rpy=0 0 0
- joint r_sole_skin_2_fixed_joint: origin xyz=0.09320869999999999 -0.032368 0.007500000000000062 rpy=0 0 0 -> xyz=0.10525929999999997 0.024325399999999997 0.007500000000000062 rpy=0 0 0
- joint r_sole_skin_3_fixed_joint: origin xyz=0.11158309999999998 -0.0263978 0.007500000000000062 rpy=0 0 0 -> xyz=0.09090169999999997 0.03725289999999999 0.007500000000000062 rpy=0 0 0
- joint r_sole_skin_4_fixed_joint: origin xyz=0.11559999999999998 -0.007499999999999993 0.007500000000000062 rpy=0 0 0 -> xyz=0.07252729999999998 0.03128289999999999 0.007500000000000062 rpy=0 0 0
- joint r_sole_skin_8_fixed_joint: origin xyz=0.10525929999999997 0.024325399999999997 0.007500000000000062 rpy=0 0 0 -> xyz=0.050136039999999986 0.006414799999999998 0.007500000000000062 rpy=0 0 0
- joint r_sole_skin_9_fixed_joint: origin xyz=0.09090169999999997 0.03725289999999999 0.007500000000000062 rpy=0 0 0 -> xyz=0.04611918999999999 -0.012483000000000008 0.007500000000000062 rpy=0 0 0

File: iCub/robots/iCubGazeboV2_5/model.urdf (robot description, URDF)
Before this commit: robot iCub, 210 links, 209 joints
Joints:
- joint l_sole_skin_0_fixed_joint: origin xyz=0.09320879999999998 0.032367999999999994 0.007500000000000062 rpy=0 0 0 -> xyz=0.05013608999999999 -0.006414799999999998 0.007500000000000062 rpy=0 0 0
- joint l_sole_skin_10_fixed_joint: origin xyz=0.10525929999999997 -0.024325399999999983 0.007500000000000062 rpy=0 0 0 -> xyz=0.09320879999999998 0.032367999999999994 0.007500000000000062 rpy=0 0 0
- joint l_sole_skin_11_fixed_joint: origin xyz=0.10124249999999999 -0.005428100000000005 0.007500000000000062 rpy=0 0 0 -> xyz=0.07885119999999998 0.019439899999999996 0.007500000000000062 rpy=0 0 0
- joint l_sole_skin_13_fixed_joint: origin xyz=0.06851049999999999 -0.012385499999999994 0.007500000000000062 rpy=0 0 0 -> xyz=0.10124249999999999 -0.005428100000000005 0.007500000000000062 rpy=0 0 0
- joint l_sole_skin_14_fixed_joint: origin xyz=0.11559999999999998 0.007499500000000006 0.007500000000000062 rpy=0 0 0 -> xyz=0.06047679999999998 0.02541059999999999 0.007500000000000062 rpy=0 0 0
- joint l_sole_skin_15_fixed_joint: origin xyz=0.11158319999999997 0.02639729999999999 0.007500000000000062 rpy=0 0 0 -> xyz=0.04611922999999998 0.012482499999999994 0.007500000000000062 rpy=0 0 0
- joint l_sole_skin_1_fixed_joint: origin xyz=0.07885119999999998 0.019439899999999996 0.007500000000000062 rpy=0 0 0 -> xyz=0.06851049999999999 -0.012385499999999994 0.007500000000000062 rpy=0 0 0
- joint l_sole_skin_2_fixed_joint: origin xyz=0.06047679999999998 0.02541059999999999 0.007500000000000062 rpy=0 0 0 -> xyz=0.07252739999999999 -0.031282799999999986 0.007500000000000062 rpy=0 0 0
- joint l_sole_skin_3_fixed_joint: origin xyz=0.04611922999999998 0.012482499999999994 0.007500000000000062 rpy=0 0 0 -> xyz=0.09090179999999999 -0.03725379999999999 0.007500000000000062 rpy=0 0 0
- joint l_sole_skin_4_fixed_joint: origin xyz=0.05013608999999999 -0.006414799999999998 0.007500000000000062 rpy=0 0 0 -> xyz=0.10525929999999997 -0.024325399999999983 0.007500000000000062 rpy=0 0 0
- joint l_sole_skin_8_fixed_joint: origin xyz=0.07252739999999999 -0.031282799999999986 0.007500000000000062 rpy=0 0 0 -> xyz=0.11559999999999998 0.007499500000000006 0.007500000000000062 rpy=0 0 0
- joint l_sole_skin_9_fixed_joint: origin xyz=0.09090179999999999 -0.03725379999999999 0.007500000000000062 rpy=0 0 0 -> xyz=0.11158319999999997 0.02639729999999999 0.007500000000000062 rpy=0 0 0
- joint r_sole_skin_0_fixed_joint: origin xyz=0.060476699999999994 -0.0254106 0.007500000000000062 rpy=0 0 0 -> xyz=0.11559999999999998 -0.007499999999999993 0.007500000000000062 rpy=0 0 0
- joint r_sole_skin_10_fixed_joint: origin xyz=0.07252729999999998 0.03128289999999999 0.007500000000000062 rpy=0 0 0 -> xyz=0.060476699999999994 -0.0254106 0.007500000000000062 rpy=0 0 0
- joint r_sole_skin_11_fixed_joint: origin xyz=0.06851049999999997 0.012385000000000007 0.007500000000000062 rpy=0 0 0 -> xyz=0.07885119999999998 -0.019440400000000004 0.007500000000000062 rpy=0 0 0
- joint r_sole_skin_13_fixed_joint: origin xyz=0.10124239999999998 0.005427600000000005 0.007500000000000062 rpy=0 0 0 -> xyz=0.06851049999999997 0.012385000000000007 0.007500000000000062 rpy=0 0 0
- joint r_sole_skin_14_fixed_joint: origin xyz=0.050136039999999986 0.006414799999999998 0.007500000000000062 rpy=0 0 0 -> xyz=0.09320869999999999 -0.032368 0.007500000000000062 rpy=0 0 0
- joint r_sole_skin_15_fixed_joint: origin xyz=0.04611918999999999 -0.012483000000000008 0.007500000000000062 rpy=0 0 0 -> xyz=0.11158309999999998 -0.0263978 0.007500000000000062 rpy=0 0 0
- joint r_sole_skin_1_fixed_joint: origin xyz=0.07885119999999998 -0.019440400000000004 0.007500000000000062 rpy=0 0 0 -> xyz=0.10124239999999998 0.005427600000000005 0.007500000000000062 rpy=0 0 0
- joint r_sole_skin_2_fixed_joint: origin xyz=0.09320869999999999 -0.032368 0.007500000000000062 rpy=0 0 0 -> xyz=0.10525929999999997 0.024325399999999997 0.007500000000000062 rpy=0 0 0
- joint r_sole_skin_3_fixed_joint: origin xyz=0.11158309999999998 -0.0263978 0.007500000000000062 rpy=0 0 0 -> xyz=0.09090169999999997 0.03725289999999999 0.007500000000000062 rpy=0 0 0
- joint r_sole_skin_4_fixed_joint: origin xyz=0.11559999999999998 -0.007499999999999993 0.007500000000000062 rpy=0 0 0 -> xyz=0.07252729999999998 0.03128289999999999 0.007500000000000062 rpy=0 0 0
- joint r_sole_skin_8_fixed_joint: origin xyz=0.10525929999999997 0.024325399999999997 0.007500000000000062 rpy=0 0 0 -> xyz=0.050136039999999986 0.006414799999999998 0.007500000000000062 rpy=0 0 0
- joint r_sole_skin_9_fixed_joint: origin xyz=0.09090169999999997 0.03725289999999999 0.007500000000000062 rpy=0 0 0 -> xyz=0.04611918999999999 -0.012483000000000008 0.007500000000000062 rpy=0 0 0

File: iCub/robots/iCubGazeboV2_7/model.urdf (robot description, URDF)
Before this commit: robot iCub, 211 links, 210 joints
Joints:
- joint l_sole_skin_0_fixed_joint: origin xyz=0.09320879999999998 0.032367999999999994 0.007500000000000062 rpy=0 0 0 -> xyz=0.05013608999999999 -0.006414799999999998 0.007500000000000062 rpy=0 0 0
- joint l_sole_skin_10_fixed_joint: origin xyz=0.10525929999999997 -0.024325399999999983 0.007500000000000062 rpy=0 0 0 -> xyz=0.09320879999999998 0.032367999999999994 0.007500000000000062 rpy=0 0 0
- joint l_sole_skin_11_fixed_joint: origin xyz=0.10124249999999999 -0.005428100000000005 0.007500000000000062 rpy=0 0 0 -> xyz=0.07885119999999998 0.019439899999999996 0.007500000000000062 rpy=0 0 0
- joint l_sole_skin_13_fixed_joint: origin xyz=0.06851049999999999 -0.012385499999999994 0.007500000000000062 rpy=0 0 0 -> xyz=0.10124249999999999 -0.005428100000000005 0.007500000000000062 rpy=0 0 0
- joint l_sole_skin_14_fixed_joint: origin xyz=0.11559999999999998 0.007499500000000006 0.007500000000000062 rpy=0 0 0 -> xyz=0.06047679999999998 0.02541059999999999 0.007500000000000062 rpy=0 0 0
- joint l_sole_skin_15_fixed_joint: origin xyz=0.11158319999999997 0.02639729999999999 0.007500000000000062 rpy=0 0 0 -> xyz=0.04611922999999998 0.012482499999999994 0.007500000000000062 rpy=0 0 0
- joint l_sole_skin_1_fixed_joint: origin xyz=0.07885119999999998 0.019439899999999996 0.007500000000000062 rpy=0 0 0 -> xyz=0.06851049999999999 -0.012385499999999994 0.007500000000000062 rpy=0 0 0
- joint l_sole_skin_2_fixed_joint: origin xyz=0.06047679999999998 0.02541059999999999 0.007500000000000062 rpy=0 0 0 -> xyz=0.07252739999999999 -0.031282799999999986 0.007500000000000062 rpy=0 0 0
- joint l_sole_skin_3_fixed_joint: origin xyz=0.04611922999999998 0.012482499999999994 0.007500000000000062 rpy=0 0 0 -> xyz=0.09090179999999999 -0.03725379999999999 0.007500000000000062 rpy=0 0 0
- joint l_sole_skin_4_fixed_joint: origin xyz=0.05013608999999999 -0.006414799999999998 0.007500000000000062 rpy=0 0 0 -> xyz=0.10525929999999997 -0.024325399999999983 0.007500000000000062 rpy=0 0 0
- joint l_sole_skin_8_fixed_joint: origin xyz=0.07252739999999999 -0.031282799999999986 0.007500000000000062 rpy=0 0 0 -> xyz=0.11559999999999998 0.007499500000000006 0.007500000000000062 rpy=0 0 0
- joint l_sole_skin_9_fixed_joint: origin xyz=0.09090179999999999 -0.03725379999999999 0.007500000000000062 rpy=0 0 0 -> xyz=0.11158319999999997 0.02639729999999999 0.007500000000000062 rpy=0 0 0
- joint r_sole_skin_0_fixed_joint: origin xyz=0.060476699999999994 -0.0254106 0.007500000000000062 rpy=0 0 0 -> xyz=0.11559999999999998 -0.007499999999999993 0.007500000000000062 rpy=0 0 0
- joint r_sole_skin_10_fixed_joint: origin xyz=0.07252729999999998 0.03128289999999999 0.007500000000000062 rpy=0 0 0 -> xyz=0.060476699999999994 -0.0254106 0.007500000000000062 rpy=0 0 0
- joint r_sole_skin_11_fixed_joint: origin xyz=0.06851049999999997 0.012385000000000007 0.007500000000000062 rpy=0 0 0 -> xyz=0.07885119999999998 -0.019440400000000004 0.007500000000000062 rpy=0 0 0
- joint r_sole_skin_13_fixed_joint: origin xyz=0.10124239999999998 0.005427600000000005 0.007500000000000062 rpy=0 0 0 -> xyz=0.06851049999999997 0.012385000000000007 0.007500000000000062 rpy=0 0 0
- joint r_sole_skin_14_fixed_joint: origin xyz=0.050136039999999986 0.006414799999999998 0.007500000000000062 rpy=0 0 0 -> xyz=0.09320869999999999 -0.032368 0.007500000000000062 rpy=0 0 0
- joint r_sole_skin_15_fixed_joint: origin xyz=0.04611918999999999 -0.012483000000000008 0.007500000000000062 rpy=0 0 0 -> xyz=0.11158309999999998 -0.0263978 0.007500000000000062 rpy=0 0 0
- joint r_sole_skin_1_fixed_joint: origin xyz=0.07885119999999998 -0.019440400000000004 0.007500000000000062 rpy=0 0 0 -> xyz=0.10124239999999998 0.005427600000000005 0.007500000000000062 rpy=0 0 0
- joint r_sole_skin_2_fixed_joint: origin xyz=0.09320869999999999 -0.032368 0.007500000000000062 rpy=0 0 0 -> xyz=0.10525929999999997 0.024325399999999997 0.007500000000000062 rpy=0 0 0
- joint r_sole_skin_3_fixed_joint: origin xyz=0.11158309999999998 -0.0263978 0.007500000000000062 rpy=0 0 0 -> xyz=0.09090169999999997 0.03725289999999999 0.007500000000000062 rpy=0 0 0
- joint r_sole_skin_4_fixed_joint: origin xyz=0.11559999999999998 -0.007499999999999993 0.007500000000000062 rpy=0 0 0 -> xyz=0.07252729999999998 0.03128289999999999 0.007500000000000062 rpy=0 0 0
- joint r_sole_skin_8_fixed_joint: origin xyz=0.10525929999999997 0.024325399999999997 0.007500000000000062 rpy=0 0 0 -> xyz=0.050136039999999986 0.006414799999999998 0.007500000000000062 rpy=0 0 0
- joint r_sole_skin_9_fixed_joint: origin xyz=0.09090169999999997 0.03725289999999999 0.007500000000000062 rpy=0 0 0 -> xyz=0.04611918999999999 -0.012483000000000008 0.007500000000000062 rpy=0 0 0
