Commit message: Automatic build of models via icub-models-generator. icub-models-generator commit: robotology/icub-models-generator@e0020213eda652d4e72a8bb3ed0eafcba723fcb5 ### Dependencies information of dependencies installed manually: urdf_parser_py commit: ros/urdf_parser_py@31474b9baaf7c3845b40e5a9aa87d5900a2282c3 simmechanics-to-urdf commit: robotology/simmechanics-to-urdf@143fd8f5450d0f84611d35ea1611869e530b0623 ### Dependencies information via pixi list: Package                               Version       Build                  Size       Kind   Source _libgcc_mutex                         0.1           conda_forge            2.5 KiB    conda  _libgcc_mutex-0.1-conda_forge.tar.bz2 _openmp_mutex                         4.5           2_gnu                  23.1 KiB   conda  _openmp_mutex-4.5-2_gnu.tar.bz2 ace                                   7.1.3         h59595ed_2             5.2 MiB    conda  ace-7.1.3-h59595ed_2.conda alsa-lib                              1.2.11        hd590300_1             541.7 KiB  conda  alsa-lib-1.2.11-hd590300_1.conda ampl-mp                               3.1.0         h2cc385e_1006          1.1 MiB    conda  ampl-mp-3.1.0-h2cc385e_1006.tar.bz2 aom                                   3.8.2         h59595ed_0             2.6 MiB    conda  aom-3.8.2-h59595ed_0.conda assimp                                5.4.1         h8343317_0             3.3 MiB    conda  assimp-5.4.1-h8343317_0.conda attr                                  2.5.1         h166bdaf_1             69.4 KiB   conda  attr-2.5.1-h166bdaf_1.tar.bz2 binutils                              2.40          hdd6e379_0             29.8 KiB   conda  binutils-2.40-hdd6e379_0.conda binutils_impl_linux-64                2.40          hf600244_0             5.2 MiB    conda  binutils_impl_linux-64-2.40-hf600244_0.conda binutils_linux-64                     2.40          hdade7a5_3             28.2 KiB   conda  binutils_linux-64-2.40-hdade7a5_3.conda bzip2                                 1.0.8         hd590300_5             248.3 KiB  conda  bzip2-1.0.8-hd590300_5.conda c-ares                                1.28.1        hd590300_0             164.9 KiB  conda  c-ares-1.28.1-hd590300_0.conda c-compiler                            1.7.0         hd590300_0             6.1 KiB    conda  c-compiler-1.7.0-hd590300_0.conda ca-certificates                       2024.2.2      hbcca054_0             151.8 KiB  conda  ca-certificates-2024.2.2-hbcca054_0.conda cairo                                 1.18.0        h3faef2a_0             959.3 KiB  conda  cairo-1.18.0-h3faef2a_0.conda catkin_pkg                            1.0.0         pyhd8ed1ab_0           52.2 KiB   conda  catkin_pkg-1.0.0-pyhd8ed1ab_0.conda cmake                                 3.29.2        hcfe8598_0             18.1 MiB   conda  cmake-3.29.2-hcfe8598_0.conda cxx-compiler                          1.7.0         h00ab1b0_0             6.1 KiB    conda  cxx-compiler-1.7.0-h00ab1b0_0.conda dav1d                                 1.2.1         hd590300_0             742.4 KiB  conda  dav1d-1.2.1-hd590300_0.conda dbus                                  1.13.6        h5008d03_3             604.1 KiB  conda  dbus-1.13.6-h5008d03_3.tar.bz2 docutils                              0.20.1        py311h38be061_3        896.8 KiB  conda  docutils-0.20.1-py311h38be061_3.conda double-conversion                     3.3.0         h59595ed_0             76.8 KiB   conda  double-conversion-3.3.0-h59595ed_0.conda eigen                                 3.4.0         h00ab1b0_0             1 MiB      conda  eigen-3.4.0-h00ab1b0_0.conda expat                                 2.6.2         h59595ed_0             134.4 KiB  conda  expat-2.6.2-h59595ed_0.conda ffmpeg                                6.1.1         gpl_h38e077a_106       9.3 MiB    conda  ffmpeg-6.1.1-gpl_h38e077a_106.conda font-ttf-dejavu-sans-mono             2.37          hab24e00_0             388.1 KiB  conda  font-ttf-dejavu-sans-mono-2.37-hab24e00_0.tar.bz2 font-ttf-inconsolata                  3.000         h77eed37_0             94.3 KiB   conda  font-ttf-inconsolata-3.000-h77eed37_0.tar.bz2 font-ttf-source-code-pro              2.038         h77eed37_0             684.4 KiB  conda  font-ttf-source-code-pro-2.038-h77eed37_0.tar.bz2 font-ttf-ubuntu                       0.83          h77eed37_1             1.5 MiB    conda  font-ttf-ubuntu-0.83-h77eed37_1.conda fontconfig                            2.14.2        h14ed4e7_0             265.6 KiB  conda  fontconfig-2.14.2-h14ed4e7_0.conda fonts-conda-ecosystem                 1             0                      3.6 KiB    conda  fonts-conda-ecosystem-1-0.tar.bz2 fonts-conda-forge                     1             0                      4 KiB      conda  fonts-conda-forge-1-0.tar.bz2 freeglut                              3.2.2         hac7e632_2             139.6 KiB  conda  freeglut-3.2.2-hac7e632_2.conda freetype                              2.12.1        h267a509_2             620.1 KiB  conda  freetype-2.12.1-h267a509_2.conda fribidi                               1.0.10        h36c2ea0_0             111.7 KiB  conda  fribidi-1.0.10-h36c2ea0_0.tar.bz2 gcc                                   12.3.0        h95e488c_3             27.1 KiB   conda  gcc-12.3.0-h95e488c_3.conda gcc_impl_linux-64                     12.3.0        he2b93b0_5             49.5 MiB   conda  gcc_impl_linux-64-12.3.0-he2b93b0_5.conda gcc_linux-64                          12.3.0        h6477408_3             30.3 KiB   conda  gcc_linux-64-12.3.0-h6477408_3.conda gdbm                                  1.18          h0a1914f_2             190.2 KiB  conda  gdbm-1.18-h0a1914f_2.tar.bz2 gettext                               0.21.1        h27087fc_0             4.1 MiB    conda  gettext-0.21.1-h27087fc_0.tar.bz2 glfw                                  3.4           hd590300_0             163.5 KiB  conda  glfw-3.4-hd590300_0.conda glib                                  2.80.0        hf2295e7_1             492 KiB    conda  glib-2.80.0-hf2295e7_1.conda glib-tools                            2.80.0        hde27a5a_1             110.2 KiB  conda  glib-tools-2.80.0-hde27a5a_1.conda gmp                                   6.3.0         h59595ed_1             556.5 KiB  conda  gmp-6.3.0-h59595ed_1.conda gnutls                                3.7.9         hb077bed_0             1.9 MiB    conda  gnutls-3.7.9-hb077bed_0.conda graphite2                             1.3.13        h59595ed_1003          94.6 KiB   conda  graphite2-1.3.13-h59595ed_1003.conda gst-plugins-base                      1.22.9        hfa15dee_1             2.6 MiB    conda  gst-plugins-base-1.22.9-hfa15dee_1.conda gstreamer                             1.22.9        h98fc4e7_1             1.9 MiB    conda  gstreamer-1.22.9-h98fc4e7_1.conda gxx                                   12.3.0        h95e488c_3             26.6 KiB   conda  gxx-12.3.0-h95e488c_3.conda gxx_impl_linux-64                     12.3.0        he2b93b0_5             12.2 MiB   conda  gxx_impl_linux-64-12.3.0-he2b93b0_5.conda gxx_linux-64                          12.3.0        h4a1b8e8_3             28.6 KiB   conda  gxx_linux-64-12.3.0-h4a1b8e8_3.conda harfbuzz                              8.3.0         h3d44ed6_0             1.5 MiB    conda  harfbuzz-8.3.0-h3d44ed6_0.conda hdf5                                  1.14.3        nompi_h4f84152_100     3.7 MiB    conda  hdf5-1.14.3-nompi_h4f84152_100.conda icu                                   73.2          h59595ed_0             11.5 MiB   conda  icu-73.2-h59595ed_0.conda idyntree                              12.3.3        py311ha0a6677_0        2.4 MiB    conda  idyntree-12.3.3-py311ha0a6677_0.conda imath                                 3.1.11        hfc55251_0             158.7 KiB  conda  imath-3.1.11-hfc55251_0.conda ipopt                                 3.14.16       h3696c94_4             998 KiB    conda  ipopt-3.14.16-h3696c94_4.conda irrlicht                              1.8.5         h2a6caf8_4             1.9 MiB    conda  irrlicht-1.8.5-h2a6caf8_4.conda jasper                                4.2.3         he6dfbbe_0             659.3 KiB  conda  jasper-4.2.3-he6dfbbe_0.conda kernel-headers_linux-64               2.6.32        he073ed8_17            694 KiB    conda  kernel-headers_linux-64-2.6.32-he073ed8_17.conda keyutils                              1.6.1         h166bdaf_0             115.1 KiB  conda  keyutils-1.6.1-h166bdaf_0.tar.bz2 krb5                                  1.21.2        h659d440_0             1.3 MiB    conda  krb5-1.21.2-h659d440_0.conda lame                                  3.100         h166bdaf_1003          496.3 KiB  conda  lame-3.100-h166bdaf_1003.tar.bz2 ld_impl_linux-64                      2.40          h41732ed_0             688.2 KiB  conda  ld_impl_linux-64-2.40-h41732ed_0.conda lerc                                  4.0.0         h27087fc_0             275.2 KiB  conda  lerc-4.0.0-h27087fc_0.tar.bz2 libabseil                             20240116.1    cxx17_h59595ed_2       1.2 MiB    conda  libabseil-20240116.1-cxx17_h59595ed_2.conda libaec                                1.1.3         h59595ed_0             34.6 KiB   conda  libaec-1.1.3-h59595ed_0.conda libass                                0.17.1        h8fe9dca_1             123.9 KiB  conda  libass-0.17.1-h8fe9dca_1.conda libblas                               3.9.0         21_linux64_openblas    14.3 KiB   conda  libblas-3.9.0-21_linux64_openblas.conda libboost                              1.84.0        h8013b2b_2             2.7 MiB    conda  libboost-1.84.0-h8013b2b_2.conda libcap                                2.69          h0f662aa_0             98.2 KiB   conda  libcap-2.69-h0f662aa_0.conda libcblas                              3.9.0         21_linux64_openblas    14.3 KiB   conda  libcblas-3.9.0-21_linux64_openblas.conda libclang-cpp15                        15.0.7        default_h127d8a8_5     16.4 MiB   conda  libclang-cpp15-15.0.7-default_h127d8a8_5.conda libclang-cpp18.1                      18.1.2        default_h127d8a8_1     18.4 MiB   conda  libclang-cpp18.1-18.1.2-default_h127d8a8_1.conda libclang13                            18.1.2        default_h5d6823c_1     10.6 MiB   conda  libclang13-18.1.2-default_h5d6823c_1.conda libcups                               2.3.3         h4637d8d_4             4.3 MiB    conda  libcups-2.3.3-h4637d8d_4.conda libcurl                               8.7.1         hca28451_0             389 KiB    conda  libcurl-8.7.1-hca28451_0.conda libdeflate                            1.20          hd590300_0             69.8 KiB   conda  libdeflate-1.20-hd590300_0.conda libdrm                                2.4.120       hd590300_0             296 KiB    conda  libdrm-2.4.120-hd590300_0.conda libedit                               3.1.20191231  he28a2e2_2             121 KiB    conda  libedit-3.1.20191231-he28a2e2_2.tar.bz2 libev                                 4.33          hd590300_2             110.1 KiB  conda  libev-4.33-hd590300_2.conda libevent                              2.1.12        hf998b51_1             417.4 KiB  conda  libevent-2.1.12-hf998b51_1.conda libexpat                              2.6.2         h59595ed_0             72 KiB     conda  libexpat-2.6.2-h59595ed_0.conda libffi                                3.4.2         h7f98852_5             56.9 KiB   conda  libffi-3.4.2-h7f98852_5.tar.bz2 libflac                               1.4.3         h59595ed_0             385.1 KiB  conda  libflac-1.4.3-h59595ed_0.conda libgcc-devel_linux-64                 12.3.0        h8bca6fd_105           2.4 MiB    conda  libgcc-devel_linux-64-12.3.0-h8bca6fd_105.conda libgcc-ng                             13.2.0        h807b86a_5             752.4 KiB  conda  libgcc-ng-13.2.0-h807b86a_5.conda libgcrypt                             1.10.3        hd590300_0             620 KiB    conda  libgcrypt-1.10.3-hd590300_0.conda libgfortran-ng                        13.2.0        h69a702a_5             23.3 KiB   conda  libgfortran-ng-13.2.0-h69a702a_5.conda libgfortran5                          13.2.0        ha4646dd_5             1.4 MiB    conda  libgfortran5-13.2.0-ha4646dd_5.conda libglib                               2.80.0        hf2295e7_1             2.8 MiB    conda  libglib-2.80.0-hf2295e7_1.conda libglu                                9.0.0         hac7e632_1003          323.5 KiB  conda  libglu-9.0.0-hac7e632_1003.conda libgomp                               13.2.0        h807b86a_5             409.9 KiB  conda  libgomp-13.2.0-h807b86a_5.conda libgpg-error                          1.48          h71f35ed_0             260.2 KiB  conda  libgpg-error-1.48-h71f35ed_0.conda libhwloc                              2.10.0        default_h5622ce7_1001  2.3 MiB    conda  libhwloc-2.10.0-default_h5622ce7_1001.conda libi2c                                4.3           hcb278e6_2             18.2 KiB   conda  libi2c-4.3-hcb278e6_2.conda libiconv                              1.17          hd590300_2             689.2 KiB  conda  libiconv-1.17-hd590300_2.conda libidn2                               2.3.7         hd590300_0             123.5 KiB  conda  libidn2-2.3.7-hd590300_0.conda libjpeg-turbo                         3.0.0         hd590300_1             604.1 KiB  conda  libjpeg-turbo-3.0.0-hd590300_1.conda liblapack                             3.9.0         21_linux64_openblas    14.3 KiB   conda  liblapack-3.9.0-21_linux64_openblas.conda liblapacke                            3.9.0         21_linux64_openblas    14.3 KiB   conda  liblapacke-3.9.0-21_linux64_openblas.conda libllvm15                             15.0.7        hb3ce162_4             31.8 MiB   conda  libllvm15-15.0.7-hb3ce162_4.conda libllvm18                             18.1.2        h2448989_0             36.6 MiB   conda  libllvm18-18.1.2-h2448989_0.conda libnghttp2                            1.58.0        h47da74e_1             617.1 KiB  conda  libnghttp2-1.58.0-h47da74e_1.conda libnsl                                2.0.1         hd590300_0             32.6 KiB   conda  libnsl-2.0.1-hd590300_0.conda libogg                                1.3.4         h7f98852_1             205.6 KiB  conda  libogg-1.3.4-h7f98852_1.tar.bz2 libopenblas                           0.3.26        pthreads_h413a1c8_0    5.3 MiB    conda  libopenblas-0.3.26-pthreads_h413a1c8_0.conda libopencv                             4.9.0         qt6_py39h8add8c0_612   28.8 MiB   conda  libopencv-4.9.0-qt6_py39h8add8c0_612.conda libopenvino                           2024.0.0      h2e90f83_4             4.9 MiB    conda  libopenvino-2024.0.0-h2e90f83_4.conda libopenvino-auto-batch-plugin         2024.0.0      hd5fc58b_4             107.6 KiB  conda  libopenvino-auto-batch-plugin-2024.0.0-hd5fc58b_4.conda libopenvino-auto-plugin               2024.0.0      hd5fc58b_4             224.1 KiB  conda  libopenvino-auto-plugin-2024.0.0-hd5fc58b_4.conda libopenvino-hetero-plugin             2024.0.0      h3ecfda7_4             176 KiB    conda  libopenvino-hetero-plugin-2024.0.0-h3ecfda7_4.conda libopenvino-intel-cpu-plugin          2024.0.0      h2e90f83_4             10.1 MiB   conda  libopenvino-intel-cpu-plugin-2024.0.0-h2e90f83_4.conda libopenvino-intel-gpu-plugin          2024.0.0      h2e90f83_4             8 MiB      conda  libopenvino-intel-gpu-plugin-2024.0.0-h2e90f83_4.conda libopenvino-ir-frontend               2024.0.0      h3ecfda7_4             196.5 KiB  conda  libopenvino-ir-frontend-2024.0.0-h3ecfda7_4.conda libopenvino-onnx-frontend             2024.0.0      h757c851_4             1.5 MiB    conda  libopenvino-onnx-frontend-2024.0.0-h757c851_4.conda libopenvino-paddle-frontend           2024.0.0      h757c851_4             679.3 KiB  conda  libopenvino-paddle-frontend-2024.0.0-h757c851_4.conda libopenvino-pytorch-frontend          2024.0.0      h59595ed_4             1 MiB      conda  libopenvino-pytorch-frontend-2024.0.0-h59595ed_4.conda libopenvino-tensorflow-frontend       2024.0.0      hca94c1a_4             1.2 MiB    conda  libopenvino-tensorflow-frontend-2024.0.0-hca94c1a_4.conda libopenvino-tensorflow-lite-frontend  2024.0.0      h59595ed_4             466.2 KiB  conda  libopenvino-tensorflow-lite-frontend-2024.0.0-h59595ed_4.conda libopus                               1.3.1         h7f98852_1             254.5 KiB  conda  libopus-1.3.1-h7f98852_1.tar.bz2 libosqp                               0.6.3         h59595ed_0             70.4 KiB   conda  libosqp-0.6.3-h59595ed_0.conda libpciaccess                          0.18          hd590300_0             27.7 KiB   conda  libpciaccess-0.18-hd590300_0.conda libpng                                1.6.43        h2797004_0             281.5 KiB  conda  libpng-1.6.43-h2797004_0.conda libpq                                 16.2          h33b98f1_1             2.5 MiB    conda  libpq-16.2-h33b98f1_1.conda libprotobuf                           4.25.3        h08a7969_0             2.7 MiB    conda  libprotobuf-4.25.3-h08a7969_0.conda libqdldl                              0.1.5         h27087fc_1             16.5 KiB   conda  libqdldl-0.1.5-h27087fc_1.tar.bz2 libsanitizer                          12.3.0        h0f45ef3_5             3.7 MiB    conda  libsanitizer-12.3.0-h0f45ef3_5.conda libscotch                             7.0.4         h91e35bf_1             331.7 KiB  conda  libscotch-7.0.4-h91e35bf_1.conda libsndfile                            1.2.2         hc60ed4a_1             346.1 KiB  conda  libsndfile-1.2.2-hc60ed4a_1.conda libspral                              2024.05.08    h1b93dcb_1             347.4 KiB  conda  libspral-2024.05.08-h1b93dcb_1.conda libsqlite                             3.45.2        h2797004_0             837.4 KiB  conda  libsqlite-3.45.2-h2797004_0.conda libssh2                               1.11.0        h0841786_0             264.8 KiB  conda  libssh2-1.11.0-h0841786_0.conda libstdcxx-devel_linux-64              12.3.0        h8bca6fd_105           11.1 MiB   conda  libstdcxx-devel_linux-64-12.3.0-h8bca6fd_105.conda libstdcxx-ng                          13.2.0        h7e041cc_5             3.7 MiB    conda  libstdcxx-ng-13.2.0-h7e041cc_5.conda libsystemd0                           255           h3516f8a_1             393.2 KiB  conda  libsystemd0-255-h3516f8a_1.conda libtasn1                              4.19.0        h166bdaf_0             114.1 KiB  conda  libtasn1-4.19.0-h166bdaf_0.tar.bz2 libtiff                               4.6.0         h1dd3fc0_3             276.1 KiB  conda  libtiff-4.6.0-h1dd3fc0_3.conda libunistring                          0.9.10        h7f98852_0             1.4 MiB    conda  libunistring-0.9.10-h7f98852_0.tar.bz2 libuuid                               2.38.1        h0b41bf4_0             32.8 KiB   conda  libuuid-2.38.1-h0b41bf4_0.conda libuv                                 1.48.0        hd590300_0             878.9 KiB  conda  libuv-1.48.0-hd590300_0.conda libva                                 2.21.0        hd590300_0             184.9 KiB  conda  libva-2.21.0-hd590300_0.conda libvorbis                             1.3.7         h9c3ff4c_0             279.6 KiB  conda  libvorbis-1.3.7-h9c3ff4c_0.tar.bz2 libvpx                                1.14.0        h59595ed_0             995.7 KiB  conda  libvpx-1.14.0-h59595ed_0.conda libwebp-base                          1.3.2         hd590300_0             392.4 KiB  conda  libwebp-base-1.3.2-hd590300_0.conda libxcb                                1.15          h0b41bf4_0             375.2 KiB  conda  libxcb-1.15-h0b41bf4_0.conda libxcrypt                             4.4.36        hd590300_1             98 KiB     conda  libxcrypt-4.4.36-hd590300_1.conda libxkbcommon                          1.7.0         h662e7e4_0             579.6 KiB  conda  libxkbcommon-1.7.0-h662e7e4_0.conda libxml2                               2.12.7        hc051c1a_1             688.5 KiB  conda  libxml2-2.12.7-hc051c1a_1.conda libxslt                               1.1.39        h76b75d6_0

File: iCub/robots/iCubGazeboV2_5_KIT_007/model.urdf (robot description, URDF)
Before this commit: robot iCub, 157 links, 156 joints
Links:
- added link imu_frame
- added link l_arm_ft
- added link r_arm_ft
- added link root_link_imu_frame
Joints:
- added joint imu_frame_fixed_joint: type fixed, parent head, child imu_frame, origin xyz=0.009500000190735 0.133444 0.009299999999999996 rpy=-1.5707963267948961 1.570796326794896 0
- added joint l_arm_ft_fixed_joint: type fixed, parent l_shoulder_3, child l_arm_ft, origin xyz=0.05093014324520106 0 0.029175829465900395 rpy=0 -1.3089970069677395 3.1415926535897927
- added joint r_arm_ft_fixed_joint: type fixed, parent r_shoulder_3, child r_arm_ft, origin xyz=-0.05089730176650909 0 0.029167029620599215 rpy=0 -1.3089970069677397 0
- added joint root_link_imu_frame_fixed_joint: type fixed, parent root_link, child root_link_imu_frame, origin xyz=0.08515499999999998 -0.011000000000000022 -0.11230899999999999 rpy=-2.0943952105869323 0 -1.5707963267948963

File: iCub/robots/iCubGazeboV2_6/model.urdf (robot description, URDF)
Before this commit: robot iCub, 210 links, 209 joints
Links:
- added link imu_frame
- added link l_arm_ft
- added link r_arm_ft
Joints:
- added joint imu_frame_fixed_joint: type fixed, parent head, child imu_frame, origin xyz=0.023453700190734995 0.20544400000000002 -0.023077900000000023 rpy=-1.5707963267948997 0 -3.141592653589793
- added joint l_arm_ft_fixed_joint: type fixed, parent l_shoulder_3, child l_arm_ft, origin xyz=0.05093014324520106 0 0.029175829465900395 rpy=0 -1.3089970069677395 3.1415926535897927
- added joint r_arm_ft_fixed_joint: type fixed, parent r_shoulder_3, child r_arm_ft, origin xyz=-0.05089730176650909 0 0.029167029620599215 rpy=0 -1.3089970069677397 0

File: iCub/robots/iCubGazeboV2_7/model.urdf (robot description, URDF)
Before this commit: robot iCub, 211 links, 210 joints
Links:
- added link imu_frame
- added link l_arm_ft
- added link r_arm_ft
Joints:
- added joint imu_frame_fixed_joint: type fixed, parent head, child imu_frame, origin xyz=0.023453700190734995 0.20544400000000002 -0.023077900000000023 rpy=-1.5707963267948997 0 -3.141592653589793
- added joint l_arm_ft_fixed_joint: type fixed, parent l_shoulder_3, child l_arm_ft, origin xyz=0.05093014324520106 0 0.029175829465900395 rpy=0 -1.3089970069677395 3.1415926535897927
- added joint r_arm_ft_fixed_joint: type fixed, parent r_shoulder_3, child r_arm_ft, origin xyz=-0.05089730176650909 0 0.029167029620599215 rpy=0 -1.3089970069677397 0

File: iCub/robots/iCubGazeboV3/model.urdf (robot description, URDF)
Before this commit: robot iCub, 56 links, 55 joints
Links:
- added link chest_depth_frame
- added link imu_frame
Joints:
- added joint chest_depth_frame_fixed_joint: type fixed, parent chest, child chest_depth_frame, origin xyz=0.0894115 0.0175 0.09929950000000001 rpy=-1.5707963267948968 0 -1.5707963267948968
- added joint imu_frame_fixed_joint: type fixed, parent head, child imu_frame, origin xyz=0.0035000000000000005 0.0055 0.10133400000000001 rpy=3.141592653589793 0 -1.5707963267948966
