Commit message: Renamed iCub_models into iCub_creo2urdf

File: iCub_creo2urdf/robots/iCubGazeboV2_10/model.urdf (robot description, URDF)
Before this commit: robot iCub, 221 links, 220 joints
Links:
- link chest: geometry collision mesh filename=package://iCub/meshes_creo2urdf/simmechanics/sim_ibbbbeba_c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 scale=0.001 0.001 0.001; visual mesh filename=package://iCub/meshes_creo2urdf/simmechanics/sim_ibbbbeba_c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 scale=0.001 0.001 0.001
- link eyes_tilt_frame: geometry collision mesh filename=package://iCub/meshes_creo2urdf/simmechanics/sim_ibbbbeba_e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 scale=0.001 0.001 0.001; visual mesh filename=package://iCub/meshes_creo2urdf/simmechanics/sim_ibbbbeba_e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 scale=0.001 0.001 0.001
- link head: geometry collision mesh filename=package://iCub/meshes_creo2urdf/simmechanics/sim_ibbbbeba_h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 scale=0.001 0.001 0.001; visual mesh filename=package://iCub/meshes_creo2urdf/simmechanics/sim_ibbbbeba_h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 scale=0.001 0.001 0.001
- link l_ankle_1: geometry collision mesh filename=package://iCub/meshes_creo2urdf/simmechanics/sim_sea_2-5_l_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 scale=0.001 0.001 0.001; visual mesh filename=package://iCub/meshes_creo2urdf/simmechanics/sim_sea_2-5_l_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 scale=0.001 0.001 0.001
- link l_ankle_2: geometry collision mesh filename=package://iCub/meshes_creo2urdf/simmechanics/sim_sea_2-5_l_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 scale=0.001 0.001 0.001; visual mesh filename=package://iCub/meshes_creo2urdf/simmechanics/sim_sea_2-5_l_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 scale=0.001 0.001 0.001
- link l_elbow_1: geometry collision mesh filename=package://iCub/meshes_creo2urdf/simmechanics/sim_sea_2-5_l_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 scale=0.001 0.001 0.001; visual mesh filename=package://iCub/meshes_creo2urdf/simmechanics/sim_sea_2-5_l_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 scale=0.001 0.001 0.001
- link l_eye: geometry collision mesh filename=package://iCub/meshes_creo2urdf/simmechanics/sim_ibbbbeba_l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 scale=0.001 0.001 0.001; visual mesh filename=package://iCub/meshes_creo2urdf/simmechanics/sim_ibbbbeba_l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 scale=0.001 0.001 0.001
- link l_foot: geometry collision box size=0.16 0.072 0.001; visual mesh filename=package://iCub/meshes_creo2urdf/simmechanics/sim_sea_2-5_l_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 scale=0.001 0.001 0.001
- link l_forearm: geometry collision mesh filename=package://iCub/meshes_creo2urdf/simmechanics/sim_sea_2-5_l_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 scale=0.001 0.001 0.001; visual mesh filename=package://iCub/meshes_creo2urdf/simmechanics/sim_sea_2-5_l_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 scale=0.001 0.001 0.001
- link l_hand: geometry collision mesh filename=package://iCub/meshes_creo2urdf/simmechanics/sim_sea_2-5_l_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 scale=0.001 0.001 0.001; visual mesh filename=package://iCub/meshes_creo2urdf/simmechanics/sim_sea_2-5_l_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 scale=0.001 0.001 0.001
- link l_hip_1: geometry collision mesh filename=package://iCub/meshes_creo2urdf/simmechanics/sim_sea_2-5_l_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 scale=0.001 0.001 0.001; visual mesh filename=package://iCub/meshes_creo2urdf/simmechanics/sim_sea_2-5_l_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 scale=0.001 0.001 0.001
- link l_hip_2: geometry collision mesh filename=package://iCub/meshes_creo2urdf/simmechanics/sim_sea_2-5_l_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 scale=0.001 0.001 0.001; visual mesh filename=package://iCub/meshes_creo2urdf/simmechanics/sim_sea_2-5_l_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 scale=0.001 0.001 0.001
- link l_hip_3: geometry collision mesh filename=package://iCub/meshes_creo2urdf/simmechanics/sim_sea_2-5_l_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 scale=0.001 0.001 0.001; visual mesh filename=package://iCub/meshes_creo2urdf/simmechanics/sim_sea_2-5_l_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 scale=0.001 0.001 0.001
- link l_lower_leg: geometry collision mesh filename=package://iCub/meshes_creo2urdf/simmechanics/sim_sea_2-5_l_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 scale=0.001 0.001 0.001; visual mesh filename=package://iCub/meshes_creo2urdf/simmechanics/sim_sea_2-5_l_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 scale=0.001 0.001 0.001
- link l_shoulder_1: geometry collision mesh filename=package://iCub/meshes_creo2urdf/simmechanics/sim_sea_2-5_l_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 scale=0.001 0.001 0.001; visual mesh filename=package://iCub/meshes_creo2urdf/simmechanics/sim_sea_2-5_l_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 scale=0.001 0.001 0.001
- link l_shoulder_2: geometry collision mesh filename=package://iCub/meshes_creo2urdf/simmechanics/sim_sea_2-5_l_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 scale=0.001 0.001 0.001; visual mesh filename=package://iCub/meshes_creo2urdf/simmechanics/sim_sea_2-5_l_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 scale=0.001 0.001 0.001
- link l_shoulder_3: geometry collision mesh filename=package://iCub/meshes_creo2urdf/simmechanics/sim_sea_2-5_l_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 scale=0.001 0.001 0.001; visual mesh filename=package://iCub/meshes_creo2urdf/simmechanics/sim_sea_2-5_l_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 scale=0.001 0.001 0.001
- link l_upper_arm: geometry collision mesh filename=package://iCub/meshes_creo2urdf/simmechanics/sim_sea_2-5_l_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 scale=0.001 0.001 0.001; visual mesh filename=package://iCub/meshes_creo2urdf/simmechanics/sim_sea_2-5_l_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 scale=0.001 0.001 0.001
- link l_upper_leg: geometry collision mesh filename=package://iCub/meshes_creo2urdf/simmechanics/sim_sea_2-5_l_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 scale=0.001 0.001 0.001; visual mesh filename=package://iCub/meshes_creo2urdf/simmechanics/sim_sea_2-5_l_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 scale=0.001 0.001 0.001
- link l_wrist_1: geometry collision mesh filename=package://iCub/meshes_creo2urdf/simmechanics/sim_sea_2-5_l_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 scale=0.001 0.001 0.001; visual mesh filename=package://iCub/meshes_creo2urdf/simmechanics/sim_sea_2-5_l_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 scale=0.001 0.001 0.001
- link neck_1: geometry collision mesh filename=package://iCub/meshes_creo2urdf/simmechanics/sim_ibbbbeba_n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 scale=0.001 0.001 0.001; visual mesh filename=package://iCub/meshes_creo2urdf/simmechanics/sim_ibbbbeba_n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 scale=0.001 0.001 0.001
- link neck_2: geometry collision mesh filename=package://iCub/meshes_creo2urdf/simmechanics/sim_ibbbbeba_n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 scale=0.001 0.001 0.001; visual mesh filename=package://iCub/meshes_creo2urdf/simmechanics/sim_ibbbbeba_n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 scale=0.001 0.001 0.001
- link neck_3: geometry collision mesh filename=package://iCub/meshes_creo2urdf/simmechanics/sim_ibbbbeba_n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 scale=0.001 0.001 0.001; visual mesh filename=package://iCub/meshes_creo2urdf/simmechanics/sim_ibbbbeba_n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 scale=0.001 0.001 0.001
- link r_ankle_1: geometry collision mesh filename=package://iCub/meshes_creo2urdf/simmechanics/sim_sea_2-5_r_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 scale=0.001 0.001 0.001; visual mesh filename=package://iCub/meshes_creo2urdf/simmechanics/sim_sea_2-5_r_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 scale=0.001 0.001 0.001
- link r_ankle_2: geometry collision mesh filename=package://iCub/meshes_creo2urdf/simmechanics/sim_sea_2-5_r_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 scale=0.001 0.001 0.001; visual mesh filename=package://iCub/meshes_creo2urdf/simmechanics/sim_sea_2-5_r_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 scale=0.001 0.001 0.001
- link r_elbow_1: geometry collision mesh filename=package://iCub/meshes_creo2urdf/simmechanics/sim_sea_2-5_r_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 scale=0.001 0.001 0.001; visual mesh filename=package://iCub/meshes_creo2urdf/simmechanics/sim_sea_2-5_r_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 scale=0.001 0.001 0.001
- link r_eye: geometry collision mesh filename=package://iCub/meshes_creo2urdf/simmechanics/sim_ibbbbeba_r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 scale=0.001 0.001 0.001; visual mesh filename=package://iCub/meshes_creo2urdf/simmechanics/sim_ibbbbeba_r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 scale=0.001 0.001 0.001
- link r_foot: geometry collision box size=0.16 0.072 0.001; visual mesh filename=package://iCub/meshes_creo2urdf/simmechanics/sim_sea_2-5_r_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 scale=0.001 0.001 0.001
- link r_forearm: geometry collision mesh filename=package://iCub/meshes_creo2urdf/simmechanics/sim_sea_2-5_r_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 scale=0.001 0.001 0.001; visual mesh filename=package://iCub/meshes_creo2urdf/simmechanics/sim_sea_2-5_r_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 scale=0.001 0.001 0.001
- link r_hand: geometry collision mesh filename=package://iCub/meshes_creo2urdf/simmechanics/sim_sea_2-5_r_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 scale=0.001 0.001 0.001; visual mesh filename=package://iCub/meshes_creo2urdf/simmechanics/sim_sea_2-5_r_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 scale=0.001 0.001 0.001
- link r_hip_1: geometry collision mesh filename=package://iCub/meshes_creo2urdf/simmechanics/sim_sea_2-5_r_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 scale=0.001 0.001 0.001; visual mesh filename=package://iCub/meshes_creo2urdf/simmechanics/sim_sea_2-5_r_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 scale=0.001 0.001 0.001
- link r_hip_2: geometry collision mesh filename=package://iCub/meshes_creo2urdf/simmechanics/sim_sea_2-5_r_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 scale=0.001 0.001 0.001; visual mesh filename=package://iCub/meshes_creo2urdf/simmechanics/sim_sea_2-5_r_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 scale=0.001 0.001 0.001
- link r_hip_3: geometry collision mesh filename=package://iCub/meshes_creo2urdf/simmechanics/sim_sea_2-5_r_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 scale=0.001 0.001 0.001; visual mesh filename=package://iCub/meshes_creo2urdf/simmechanics/sim_sea_2-5_r_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 scale=0.001 0.001 0.001
- link r_lower_leg: geometry collision mesh filename=package://iCub/meshes_creo2urdf/simmechanics/sim_sea_2-5_r_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 scale=0.001 0.001 0.001; visual mesh filename=package://iCub/meshes_creo2urdf/simmechanics/sim_sea_2-5_r_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 scale=0.001 0.001 0.001
- link r_shoulder_1: geometry collision mesh filename=package://iCub/meshes_creo2urdf/simmechanics/sim_sea_2-5_r_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 scale=0.001 0.001 0.001; visual mesh filename=package://iCub/meshes_creo2urdf/simmechanics/sim_sea_2-5_r_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 scale=0.001 0.001 0.001
- link r_shoulder_2: geometry collision mesh filename=package://iCub/meshes_creo2urdf/simmechanics/sim_sea_2-5_r_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 scale=0.001 0.001 0.001; visual mesh filename=package://iCub/meshes_creo2urdf/simmechanics/sim_sea_2-5_r_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 scale=0.001 0.001 0.001
- link r_shoulder_3: geometry collision mesh filename=package://iCub/meshes_creo2urdf/simmechanics/sim_sea_2-5_r_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 scale=0.001 0.001 0.001; visual mesh filename=package://iCub/meshes_creo2urdf/simmechanics/sim_sea_2-5_r_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 scale=0.001 0.001 0.001
- link r_upper_arm: geometry collision mesh filename=package://iCub/meshes_creo2urdf/simmechanics/sim_sea_2-5_r_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 scale=0.001 0.001 0.001; visual mesh filename=package://iCub/meshes_creo2urdf/simmechanics/sim_sea_2-5_r_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 scale=0.001 0.001 0.001
- link r_upper_leg: geometry collision mesh filename=package://iCub/meshes_creo2urdf/simmechanics/sim_sea_2-5_r_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 scale=0.001 0.001 0.001; visual mesh filename=package://iCub/meshes_creo2urdf/simmechanics/sim_sea_2-5_r_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 scale=0.001 0.001 0.001
- link r_wrist_1: geometry collision mesh filename=package://iCub/meshes_creo2urdf/simmechanics/sim_sea_2-5_r_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 scale=0.001 0.001 0.001; visual mesh filename=package://iCub/meshes_creo2urdf/simmechanics/sim_sea_2-5_r_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 scale=0.001 0.001 0.001
- link root_link: geometry collision mesh filename=package://iCub/meshes_creo2urdf/simmechanics/sim_sea_2-5_ro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 scale=0.001 0.001 0.001; visual mesh filename=package://iCub/meshes_creo2urdf/simmechanics/sim_sea_2-5_ro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 scale=0.001 0.001 0.001
- link torso_1: geometry collision mesh filename=package://iCub/meshes_creo2urdf/simmechanics/sim_ibbbbeba_t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 scale=0.001 0.001 0.001; visual mesh filename=package://iCub/meshes_creo2urdf/simmechanics/sim_ibbbbeba_t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 scale=0.001 0.001 0.001
- link torso_2: geometry collision mesh filename=package://iCub/meshes_creo2urdf/simmechanics/sim_ibbbbeba_t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 scale=0.001 0.001 0.001; visual mesh filename=package://iCub/meshes_creo2urdf/simmechanics/sim_ibbbbeba_t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 scale=0.001 0.001 0.001

Commit message: Remove eyes_tilt exported frame

File: iCub_creo2urdf/robots/iCubGazeboV2_10/model.urdf (robot description, URDF)
Before this commit: robot iCub, 221 links, 220 joints
Links:
- removed link eyes_tilt
Joints:
- removed joint eyes_tilt_fixed_joint

Commit message: Update iCubGazeboV2_10 without gazebo classic

File: iCub_creo2urdf/robots/iCubGazeboV2_10/model.urdf (robot description, URDF)
Before this commit: robot iCub, 221 links, 220 joints
Joints:
- joint root_link_ems_gyro_eb5_fixed_joint: child root_link -> root_link_ems_gyro_eb5; parent root_link_ems_gyro_eb5 -> root_link

Commit message: [iCubGazeboV2_10] Fix reverse rotation axis

File: iCub_creo2urdf/robots/iCubGazeboV2_10/model.urdf (robot description, URDF)
Before this commit: robot iCub, 220 links, 219 joints
Joints:
- joint l_ankle_pitch: axis 1.7552765002815832e-14 -1 7.973463690438263e-14 -> -1.7552765002815832e-14 1 -7.973463690438263e-14; limit lower=0.03490658503988659 upper=0.03490658503988659 effort=1e+9 velocity=1e+9 -> lower=-0.8726646259971648 upper=0.3490658503988659 effort=1e+9 velocity=1e+9
- joint l_ankle_roll: axis -0.9999999999999983 1.9663419506723466e-14 -2.225885610944277e-14 -> 0.9999999999999983 -1.9663419506723466e-14 2.225885610944277e-14
- joint l_hip_roll: axis -0.999999999999998 2.906647793090718e-14 1.1696369637952586e-14 -> 0.999999999999998 -2.906647793090718e-14 -1.1696369637952586e-14
- joint l_hip_yaw: axis -7.749471415023418e-16 2.0406078820946993e-14 -0.9999999999999943 -> 7.749471415023418e-16 -2.0406078820946993e-14 0.9999999999999943
- joint l_knee: axis -1.7019517803789784e-14 1 -1.0624352005446662e-13 -> 1.7019517803789784e-14 -1 1.0624352005446662e-13
- joint r_ankle_pitch: axis 1.6922193422825768e-14 -1 -1.5473390515819732e-14 -> -1.6922193422825768e-14 1 1.5473390515819732e-14; limit lower=0.03490658503988659 upper=0.03490658503988659 effort=1e+9 velocity=1e+9 -> lower=-0.8726646259971648 upper=0.3490658503988659 effort=1e+9 velocity=1e+9
- joint r_ankle_roll: axis 1 -1.0494425887568333e-14 3.142167137936615e-14 -> -1 1.0494425887568333e-14 -3.142167137936615e-14
- joint r_hip_roll: axis 1 -2.6163525606402277e-14 -3.3084227166665015e-14 -> -1 2.6163525606402277e-14 3.3084227166665015e-14
- joint r_hip_yaw: axis -2.080649515309335e-14 1.5268127249500356e-14 1 -> 2.080649515309335e-14 -1.5268127249500356e-14 -1
- joint r_knee: axis -1.4934554061540765e-14 1 1.5350925835905035e-14 -> 1.4934554061540765e-14 -1 -1.5350925835905035e-14
